Commit message: Apply review feedback to the blueboat packages
Assisted-by: Claude Fable 5 <noreply@anthropic.com>
Signed-off-by: Carlos Aguero <caguero@honurobotics.com>

File: blueboat_description/urdf/thruster.xacro (robot description, xacro)
@@ -16,7 +16,9 @@
     <link name="motor_${side}_link">
       <inertial>
-        <mass value="0.2"/>
-        <inertia ixx="0.1" ixy="0.0" ixz="0.0"
-                 iyy="0.1" iyz="0.0" izz="0.1"/>
+        <!-- T200 in air ~0.344 kg; short-cylinder inertia (r~38 mm, h~40 mm).
+             Note izz <= ixx + iyy must hold or sdformat rejects the link. -->
+        <mass value="0.344"/>
+        <inertia ixx="1.7e-4" ixy="0.0" ixz="0.0"
+                 iyy="1.7e-4" iyz="0.0" izz="2.5e-4"/>
       </inertial>
       <visual>
