Commit message: Propagate the PR 1 review fixes to the blueboat packages
Assisted-by: Claude Fable 5 <noreply@anthropic.com>
Signed-off-by: Carlos Aguero <caguero@honurobotics.com>

File: blueboat_description/urdf/accessories.xacro (robot description, xacro)
@@ -8,9 +8,14 @@
 <robot xmlns:xacro="http://ros.org/wiki/xacro">
   <!-- ===== helpers ===== -->
+  <!-- Inertia tensors follow from the primitive geometry and the mass, so they
+       track the placeholder dimensions automatically. -->
   <xacro:macro name="_box_accessory" params="name xyz rpy parent size mass:=0.3">
+    <xacro:property name="d" value="${[float(v) for v in size.split()]}"/>
     <link name="${name}">
       <inertial>
         <mass value="${mass}"/>
-        <inertia ixx="0.001" ixy="0" ixz="0" iyy="0.001" iyz="0" izz="0.001"/>
+        <inertia ixx="${float(mass)/12.0 * (d[1]**2 + d[2]**2)}" ixy="0" ixz="0"
+                 iyy="${float(mass)/12.0 * (d[0]**2 + d[2]**2)}" iyz="0"
+                 izz="${float(mass)/12.0 * (d[0]**2 + d[1]**2)}"/>
       </inertial>
       <visual>
@@ -28,5 +33,7 @@
       <inertial>
         <mass value="${mass}"/>
-        <inertia ixx="0.001" ixy="0" ixz="0" iyy="0.001" iyz="0" izz="0.001"/>
+        <inertia ixx="${float(mass)/12.0 * (3*float(radius)**2 + float(length)**2)}" ixy="0" ixz="0"
+                 iyy="${float(mass)/12.0 * (3*float(radius)**2 + float(length)**2)}" iyz="0"
+                 izz="${float(mass)/2.0 * float(radius)**2}"/>
       </inertial>
       <visual>
@@ -45,6 +52,11 @@
     <link name="${name}">
       <inertial>
+        <origin xyz="0 0 0.15" rpy="0 0 0"/>
         <mass value="0.05"/>
-        <inertia ixx="0.0001" ixy="0" ixz="0" iyy="0.0001" iyz="0" izz="0.0001"/>
+        <!-- Slender pole (r 6 mm, l 0.30 m) about its centre; the cloth is
+             negligible. -->
+        <inertia ixx="${0.05/12.0 * (3*0.006**2 + 0.30**2)}" ixy="0" ixz="0"
+                 iyy="${0.05/12.0 * (3*0.006**2 + 0.30**2)}" iyz="0"
+                 izz="${0.05/2.0 * 0.006**2}"/>
       </inertial>
       <visual>
@@ -92,17 +104,12 @@
                           size="0.191 0.091 0.057" mass="0.6"/>
   </xacro:macro>
-  <!-- ===== recursive dispatcher: mount each config accessory by type ===== -->
+  <!-- ===== recursive dispatcher: mount each config accessory by type =====
+       The config `type` IS the macro name, invoked directly; an unknown type
+       fails the build loudly instead of silently mounting nothing. -->
   <xacro:macro name="mount_accessories" params="items parent:=base_link">
     <xacro:if value="${len(items) > 0}">
       <xacro:property name="a" value="${items[0]}"/>
-      <xacro:property name="t" value="${a['type']}"/>
-      <xacro:if value="${t == 'flag'}">               <xacro:flag                name="${a['name']}" xyz="${a['xyz']}" rpy="${a['rpy']}" parent="${parent}"/></xacro:if>
-      <xacro:if value="${t == 'antenna_mast'}">       <xacro:antenna_mast        name="${a['name']}" xyz="${a['xyz']}" rpy="${a['rpy']}" parent="${parent}"/></xacro:if>
-      <xacro:if value="${t == 'basestation_antenna'}"><xacro:basestation_antenna name="${a['name']}" xyz="${a['xyz']}" rpy="${a['rpy']}" parent="${parent}"/></xacro:if>
-      <xacro:if value="${t == 'ping_sonar'}">         <xacro:ping_sonar          name="${a['name']}" xyz="${a['xyz']}" rpy="${a['rpy']}" parent="${parent}"/></xacro:if>
-      <xacro:if value="${t == 'ping_mount'}">         <xacro:ping_mount          name="${a['name']}" xyz="${a['xyz']}" rpy="${a['rpy']}" parent="${parent}"/></xacro:if>
-      <xacro:if value="${t == 'payload_bracket'}">    <xacro:payload_bracket     name="${a['name']}" xyz="${a['xyz']}" rpy="${a['rpy']}" parent="${parent}"/></xacro:if>
-      <xacro:if value="${t == 'omniscan_450'}">       <xacro:omniscan_450        name="${a['name']}" xyz="${a['xyz']}" rpy="${a['rpy']}" parent="${parent}"/></xacro:if>
-      <xacro:if value="${t == 'surveyor_multibeam'}"> <xacro:surveyor_multibeam  name="${a['name']}" xyz="${a['xyz']}" rpy="${a['rpy']}" parent="${parent}"/></xacro:if>
+      <xacro:call macro="${a['type']}" name="${a['name']}"
+                  xyz="${a['xyz']}" rpy="${a['rpy']}" parent="${parent}"/>
       <xacro:mount_accessories items="${items[1:]}" parent="${parent}"/>
     </xacro:if>

File: blueboat_description/urdf/blueboat.urdf.xacro (robot description, xacro)
@@ -21,4 +21,5 @@
        for the waterline you want (verify the float on a GPU). Dims/offsets approx.
        the two pontoons from the hull collision mesh (~1.19 m long, centres y~0.3). -->
+  <xacro:property name="thruster_mass" value="0.344"/>
   <xacro:property name="pontoon_length" value="1.1"/>
   <xacro:property name="pontoon_width"  value="0.19"/>

File: blueboat_description/urdf/thruster.xacro (robot description, xacro)
@@ -18,5 +18,5 @@
         <!-- T200 in air ~0.344 kg; short-cylinder inertia (r~38 mm, h~40 mm).
              Note izz <= ixx + iyy must hold or sdformat rejects the link. -->
-        <mass value="0.344"/>
+        <mass value="${thruster_mass}"/>
         <inertia ixx="1.7e-4" ixy="0.0" ixz="0.0"
                  iyy="1.7e-4" iyz="0.0" izz="2.5e-4"/>

File: blueboat_gazebo/model.sdf.xacro (robot description, xacro)
@@ -48,8 +48,8 @@
       <pose relative_to="base_link">${pose}</pose>
       <inertial>
-        <mass>0.001</mass>
+        <mass>1e-5</mass>
         <inertia>
-          <ixx>1e-6</ixx><ixy>0</ixy><ixz>0</ixz>
-          <iyy>1e-6</iyy><iyz>0</iyz><izz>1e-6</izz>
+          <ixx>1e-8</ixx><ixy>0</ixy><ixz>0</ixz>
+          <iyy>1e-8</iyy><iyz>0</iyz><izz>1e-8</izz>
         </inertia>
       </inertial>

Commit message: Apply the PR 2 review feedback and propagate the merged PR 1 improvements
Assisted-by: Claude Fable 5 <noreply@anthropic.com>
Signed-off-by: Carlos Aguero <caguero@honurobotics.com>

File: blueboat_description/urdf/accessories.xacro (robot description, xacro)
@@ -10,15 +10,15 @@
   <!-- Inertia tensors follow from the primitive geometry and the mass, so they
        track the placeholder dimensions automatically. -->
-  <xacro:macro name="_box_accessory" params="name xyz rpy parent size mass:=0.3">
-    <xacro:property name="d" value="${[float(v) for v in size.split()]}"/>
+  <!-- One shared skeleton (link + fixed joint + visual); the box/cyl wrappers
+       below compute the matching inertia tensor from geometry and mass, so the
+       two never drift apart. -->
+  <xacro:macro name="_accessory" params="name xyz rpy parent mass ixx iyy izz *geometry">
     <link name="${name}">
       <inertial>
         <mass value="${mass}"/>
-        <inertia ixx="${float(mass)/12.0 * (d[1]**2 + d[2]**2)}" ixy="0" ixz="0"
-                 iyy="${float(mass)/12.0 * (d[0]**2 + d[2]**2)}" iyz="0"
-                 izz="${float(mass)/12.0 * (d[0]**2 + d[1]**2)}"/>
+        <inertia ixx="${ixx}" ixy="0" ixz="0" iyy="${iyy}" iyz="0" izz="${izz}"/>
       </inertial>
       <visual>
-        <geometry><box size="${size}"/></geometry>
+        <xacro:insert_block name="geometry"/>
         <material name="${name}_mat"><color rgba="0.5 0.5 0.55 1"/></material>
       </visual>
@@ -29,24 +29,25 @@
     </joint>
   </xacro:macro>
+  <xacro:macro name="_box_accessory" params="name xyz rpy parent size mass:=0.3">
+    <xacro:property name="d" value="${[float(v) for v in size.split()]}"/>
+    <xacro:_accessory name="${name}" xyz="${xyz}" rpy="${rpy}" parent="${parent}"
+                      mass="${mass}"
+                      ixx="${float(mass)/12.0 * (d[1]**2 + d[2]**2)}"
+                      iyy="${float(mass)/12.0 * (d[0]**2 + d[2]**2)}"
+                      izz="${float(mass)/12.0 * (d[0]**2 + d[1]**2)}">
+      <geometry><box size="${size}"/></geometry>
+    </xacro:_accessory>
+  </xacro:macro>
   <xacro:macro name="_cyl_accessory" params="name xyz rpy parent radius length mass:=0.3">
-    <link name="${name}">
-      <inertial>
-        <mass value="${mass}"/>
-        <inertia ixx="${float(mass)/12.0 * (3*float(radius)**2 + float(length)**2)}" ixy="0" ixz="0"
-                 iyy="${float(mass)/12.0 * (3*float(radius)**2 + float(length)**2)}" iyz="0"
-                 izz="${float(mass)/2.0 * float(radius)**2}"/>
-      </inertial>
-      <visual>
-        <geometry><cylinder radius="${radius}" length="${length}"/></geometry>
-        <material name="${name}_mat"><color rgba="0.5 0.5 0.55 1"/></material>
-      </visual>
-    </link>
-    <joint name="${name}_joint" type="fixed">
-      <parent link="${parent}"/><child link="${name}"/>
-      <origin xyz="${xyz}" rpy="${rpy}"/>
-    </joint>
+    <xacro:_accessory name="${name}" xyz="${xyz}" rpy="${rpy}" parent="${parent}"
+                      mass="${mass}"
+                      ixx="${float(mass)/12.0 * (3*float(radius)**2 + float(length)**2)}"
+                      iyy="${float(mass)/12.0 * (3*float(radius)**2 + float(length)**2)}"
+                      izz="${float(mass)/2.0 * float(radius)**2}">
+      <geometry><cylinder radius="${radius}" length="${length}"/></geometry>
+    </xacro:_accessory>
   </xacro:macro>
   <!-- ===== accessories ===== -->
-  <!-- Flag: reuses the existing base flag mesh, split out so it can be toggled. -->
+  <!-- Flag: pole + banner primitives; a separate accessory so it can be toggled. -->
   <xacro:macro name="flag" params="name xyz rpy parent:=base_link">
     <link name="${name}">

File: blueboat_description/urdf/blueboat.urdf.xacro (robot description, xacro)
@@ -94,4 +94,4 @@
   <xacro:blueboat_thruster side="stbd" xyz="-0.488 -0.295 -0.272"/>
   <!-- ===================== Accessories (from config) ===================== -->
-  <xacro:mount_accessories items="${cfg.get('accessories', [])}"/>
+  <xacro:mount_accessories items="${cfg.get('accessories') or []}"/>
 </robot>

File: blueboat_gazebo/model.sdf.xacro (robot description, xacro)
@@ -27,10 +27,11 @@
        /model/blueboat/joint/motor_<side>_joint/cmd_thrust. -->
   <xacro:macro name="thruster" params="side coeff">
+    <!-- No <namespace>: the plugin defaults to the model name, so the command
+         topics track the instance name and multiple vehicles stay distinct. -->
     <plugin filename="gz-sim-thruster-system" name="gz::sim::systems::Thruster">
-      <namespace>blueboat</namespace>
       <joint_name>motor_${side}_joint</joint_name>
       <thrust_coefficient>${coeff}</thrust_coefficient>
       <fluid_density>1025.0</fluid_density>
-      <propeller_diameter>0.1</propeller_diameter>
+      <propeller_diameter>0.076</propeller_diameter>  <!-- T200 prop -->
       <velocity_control>true</velocity_control>
       <max_thrust_cmd>${t200_max_thrust}</max_thrust_cmd>
@@ -66,4 +67,9 @@
     <xacro:sensor_link name="${name}" pose="${pose}">
       <sensor name="${name}" type="gpu_lidar">
+        <!-- Pin frame_id to the accessory's own URDF link: that is the only
+             name TF carries (robot_state_publisher publishes the URDF links;
+             the ${name}_sensor wrapper link exists only here, and gz's derived
+             id is in neither). Body frame convention. -->
+        <frame_id>${name}</frame_id>
         <topic>${topic_base}/range</topic>
         <update_rate>10</update_rate>
@@ -115,9 +121,15 @@
       <nRabsR>-30</nRabsR>
     </plugin>
+    <!-- Joint states for the motor joints, so robot_state_publisher can
+         animate the props in RViz. Bridged to /joint_states. -->
+    <plugin filename="gz-sim-joint-state-publisher-system"
+            name="gz::sim::systems::JointStatePublisher">
+      <topic>${topic_ns}/joint_states</topic>
+    </plugin>
     <!-- Twin outboards (counter-rotating). -->
     <xacro:thruster side="port" coeff="0.02"/>
     <xacro:thruster side="stbd" coeff="-0.02"/>
     <!-- Sensors: one per sensor-type accessory in config/blueboat.yaml. -->
-    <xacro:mount_sensors items="${cfg.get('accessories', [])}"/>
+    <xacro:mount_sensors items="${cfg.get('accessories') or []}"/>
   </model>
 </sdf>
