Commit message: added the blueboat and a few mesh accessories; also, a first attempt to added the collision converting SDF to URDF

File: blueboat_description/urdf/blueboat.urdf.xacro (robot description, xacro)
@@ -89,4 +89,250 @@
     <xacro:hull_visuals/>
   </link>
+  <!-- ===================== Pulled from SDF Export for Blueboat ===================== -->
+  <!--
+  <link name="Blueboat_link">
+    <visual name="Blueboat_visual">
+      <geometry>
+        <mesh>
+          <uri>/meshes/blueboat.visual.glb</uri>
+        </mesh>
+      </geometry>
+    </visual>
+    <collision name="blue usv_collider_box">
+      <pose>-0.104158 -0.295896 -0.043697 0.0 0.0 0.0</pose>
+      <geometry>
+        <box>
+          <size>0.696765 0.018217 0.370259</size>
+        </box>
+      </geometry>
+    </collision>
+    <collision name="blue usv_collider_box.002">
+      <pose>-0.012113 -0.363698 0.083833 0.0 0.0 0.0</pose>
+      <geometry>
+        <box>
+          <size>0.872756 0.125557 0.116921</size>
+        </box>
+      </geometry>
+    </collision>
+    <collision name="blue usv_collider_cylinder">
+      <pose>-0.017902 -0.360024 0.01984 0.0 0.0 0.0</pose>
+      <geometry>
+        <cylinder>
+          <radius>0.411411</radius>
+          <length>0.135532</length>
+        </cylinder>
+      </geometry>
+    </collision>
+    <collision name="blue usv_collider_box.006">
+      <pose>-0.522288 -0.295896 -0.211583 0.0 0.0 0.0</pose>
+      <geometry>
+        <box>
+          <size>0.150178 0.018217 0.034487</size>
+        </box>
+      </geometry>
+    </collision>
+    <collision name="blue usv_collider_cylinder.001">
+      <pose>-0.033923 -0.323371 -0.052308 0.0 0.0 0.0</pose>
+      <geometry>
+        <cylinder>
+          <radius>0.421063</radius>
+          <length>0.056977</length>
+        </cylinder>
+      </geometry>
+    </collision>
+    <collision name="blue usv_collider_box.004">
+      <pose>-0.467242 -0.314934 0.038698 0.0 0.0 0.0</pose>
+      <geometry>
+        <box>
+          <size>0.127101 0.074541 0.20022</size>
+        </box>
+      </geometry>
+    </collision>
+    <collision name="blue usv_collider_box.008">
+      <pose>0.488345 -0.302387 0.086141 0.0 0.0 0.0</pose>
+      <geometry>
+        <box>
+          <size>0.197621 0.049447 0.105333</size>
+        </box>
+      </geometry>
+    </collision>
+    <collision name="blue usv_collider_cylinder.002">
+      <pose>0.406722 -0.321877 0.030426 0.0 0.0 0.0</pose>
+      <geometry>
+        <cylinder>
+          <radius>0.111828</radius>
+          <length>0.223656</length>
+        </cylinder>
+      </geometry>
+    </collision>
+    <collision name="blue usv_collider_cylinder.003">
+      <pose>0.283564 -0.295886 -0.045978 0.0 0.0 0.0</pose>
+      <geometry>
+        <cylinder>
+          <radius>0.132203</radius>
+          <length>0.264407</length>
+        </cylinder>
+      </geometry>
+    </collision>
+    <collision name="blue usv_collider_cylinder.004">
+      <pose>-0.447734 -0.30143 -0.126513 0.0 0.0 0.0</pose>
+      <geometry>
+        <cylinder>
+          <radius>0.040196</radius>
+          <length>0.040861</length>
+        </cylinder>
+      </geometry>
+    </collision>
+    <collision name="blue usv_collider_box.001">
+      <pose>0.488345 0.302388 0.086141 0.0 0.0 0.0</pose>
+      <geometry>
+        <box>
+          <size>0.197621 0.049447 0.105333</size>
+        </box>
+      </geometry>
+    </collision>
+    <collision name="blue usv_collider_cylinder.005">
+      <pose>0.406722 0.321876 0.030426 0.0 0.0 0.0</pose>
+      <geometry>
+        <cylinder>
+          <radius>0.111828</radius>
+          <length>0.223656</length>
+        </cylinder>
+      </geometry>
+    </collision>
+    <collision name="blue usv_collider_cylinder.006">
+      <pose>-0.017902 0.360024 0.01984 0.0 0.0 0.0</pose>
+      <geometry>
+        <cylinder>
+          <radius>0.411411</radius>
+          <length>0.135532</length>
+        </cylinder>
+      </geometry>
+    </collision>
+    <collision name="blue usv_collider_box.003">
+      <pose>-0.012113 0.363698 0.083833 0.0 0.0 0.0</pose>
+      <geometry>
+        <box>
+          <size>0.872756 0.125557 0.116921</size>
+        </box>
+      </geometry>
+    </collision>
+    <collision name="blue usv_collider_cylinder.007">
+      <pose>0.283564 0.295886 -0.045978 0.0 0.0 0.0</pose>
+      <geometry>
+        <cylinder>
+          <radius>0.132203</radius>
+          <length>0.264407</length>
+        </cylinder>
+      </geometry>
+    </collision>
+    <collision name="blue usv_collider_box.005">
+      <pose>-0.104158 0.295896 -0.043697 0.0 0.0 0.0</pose>
+      <geometry>
+        <box>
+          <size>0.696765 0.018217 0.370259</size>
+        </box>
+      </geometry>
+    </collision>
+    <collision name="blue usv_collider_cylinder.008">
+      <pose>-0.447734 0.30143 -0.126513 0.0 0.0 0.0</pose>
+      <geometry>
+        <cylinder>
+          <radius>0.040196</radius>
+          <length>0.040861</length>
+        </cylinder>
+      </geometry>
+    </collision>
+    <collision name="blue usv_collider_box.007">
+      <pose>0.299059 -0.0 0.142501 0.0 0.0 0.0</pose>
+      <geometry>
+        <box>
+          <size>0.0257 0.500356 0.037959</size>
+        </box>
+      </geometry>
+    </collision>
+    <collision name="blue usv_collider_box.009">
+      <pose>-0.300152 0.0 0.142501 0.0 0.0 0.0</pose>
+      <geometry>
+        <box>
+          <size>0.0257 0.500356 0.037959</size>
+        </box>
+      </geometry>
+    </collision>
+    <collision name="blue usv_collider_box.010">
+      <pose>0.298121 -0.317568 0.130778 0.0 0.0 0.0</pose>
+      <geometry>
+        <box>
+          <size>0.043582 0.183315 0.063965</size>
+        </box>
+      </geometry>
+    </collision>
+    <collision name="blue usv_collider_box.011">
+      <pose>-0.29897 -0.317568 0.130778 0.0 0.0 0.0</pose>
+      <geometry>
+        <box>
+          <size>0.043582 0.183315 0.063965</size>
+        </box>
+      </geometry>
+    </collision>
+    <collision name="blue usv_collider_box.012">
+      <pose>-0.29897 0.317568 0.130778 0.0 0.0 0.0</pose>
+      <geometry>
+        <box>
+          <size>0.043582 0.183315 0.063965</size>
+        </box>
+      </geometry>
+    </collision>
+    <collision name="blue usv_collider_box.013">
+      <pose>0.298121 0.317568 0.130778 0.0 0.0 0.0</pose>
+      <geometry>
+        <box>
+          <size>0.043582 0.183315 0.063965</size>
+        </box>
+      </geometry>
+    </collision>
+    <collision name="blue usv_collider_cylinder.009">
+      <pose>-0.253322 -0.00144 0.117093 0.0 0.0 0.0</pose>
+      <geometry>
+        <cylinder>
+          <radius>0.016745</radius>
+          <length>0.03349</length>
+        </cylinder>
+      </geometry>
+    </collision>
+    <collision name="blue usv_collider_box.014">
+      <pose>0.003337 -0.36614 0.160429 0.0 0.0 0.0</pose>
+      <geometry>
+        <box>
+          <size>0.415567 0.151904 0.045952</size>
+        </box>
+      </geometry>
+    </collision>
+    <collision name="blue usv_collider_box.015">
+      <pose>0.003337 0.36614 0.160429 0.0 0.0 0.0</pose>
+      <geometry>
+        <box>
+          <size>0.415567 0.151904 0.045952</size>
+        </box>
+      </geometry>
+    </collision>
+    <collision name="blue usv_collider_box.016">
+      <pose>-0.467242 0.314935 0.038698 0.0 0.0 0.0</pose>
+      <geometry>
+        <box>
+          <size>0.127101 0.074541 0.20022</size>
+        </box>
+      </geometry>
+    </collision>
+    <collision name="blue usv_collider_box.017">
+      <pose>-0.522288 0.295896 -0.211583 0.0 0.0 0.0</pose>
+      <geometry>
+        <box>
+          <size>0.150178 0.018217 0.034487</size>
+        </box>
+      </geometry>
+    </collision>
+  </link>
+  -->
   <!-- ===================== Thrusters (props) ===================== -->
   <xacro:blueboat_thruster side="port" xyz="-0.488 0.295 -0.272"/>

Commit message: added visual and collision code but commented out until I figure out if I'm doing this correctly

File: blueboat_description/urdf/blueboat.urdf.xacro (robot description, xacro)
@@ -89,4 +89,252 @@
     <xacro:pontoon side="stbd" y="${-pontoon_y}" n="${pontoon_segments}"/>
     <xacro:hull_visuals/>
+    <!-- TODO: Verify I'm doing this right -->
+    <!-- Can I remove the line above and replace it with this reference to the visual?  -->
+    <!-- Also, how does the path reference work?  -->
+    <!-- Visual for the blueboat
+    <visual name="Blueboat_visual">
+      <geometry>
+        <mesh>
+          <uri>blueboat.visual.glb</uri>
+        </mesh>
+      </geometry>
+    </visual> -->
+    <!-- Collision exported from SDF Gen -->
+    <!--
+    <collision name="blue usv_collider_box">
+        <pose>-0.104158 -0.295896 -0.043697 0.0 0.0 0.0</pose>
+        <geometry>
+          <box>
+            <size>0.696765 0.018217 0.370259</size>
+          </box>
+        </geometry>
+      </collision>
+      <collision name="blue usv_collider_box.002">
+        <pose>-0.012113 -0.363698 0.083833 0.0 0.0 0.0</pose>
+        <geometry>
+          <box>
+            <size>0.872756 0.125557 0.116921</size>
+          </box>
+        </geometry>
+      </collision>
+      <collision name="blue usv_collider_cylinder">
+        <pose>-0.017902 -0.360024 0.01984 0.0 0.0 0.0</pose>
+        <geometry>
+          <cylinder>
+            <radius>0.411411</radius>
+            <length>0.135532</length>
+          </cylinder>
+        </geometry>
+      </collision>
+      <collision name="blue usv_collider_box.006">
+        <pose>-0.522288 -0.295896 -0.211583 0.0 0.0 0.0</pose>
+        <geometry>
+          <box>
+            <size>0.150178 0.018217 0.034487</size>
+          </box>
+        </geometry>
+      </collision>
+      <collision name="blue usv_collider_cylinder.001">
+        <pose>-0.033923 -0.323371 -0.052308 0.0 0.0 0.0</pose>
+        <geometry>
+          <cylinder>
+            <radius>0.421063</radius>
+            <length>0.056977</length>
+          </cylinder>
+        </geometry>
+      </collision>
+      <collision name="blue usv_collider_box.004">
+        <pose>-0.467242 -0.314934 0.038698 0.0 0.0 0.0</pose>
+        <geometry>
+          <box>
+            <size>0.127101 0.074541 0.20022</size>
+          </box>
+        </geometry>
+      </collision>
+      <collision name="blue usv_collider_box.008">
+        <pose>0.488345 -0.302387 0.086141 0.0 0.0 0.0</pose>
+        <geometry>
+          <box>
+            <size>0.197621 0.049447 0.105333</size>
+          </box>
+        </geometry>
+      </collision>
+      <collision name="blue usv_collider_cylinder.002">
+        <pose>0.406722 -0.321877 0.030426 0.0 0.0 0.0</pose>
+        <geometry>
+          <cylinder>
+            <radius>0.111828</radius>
+            <length>0.223656</length>
+          </cylinder>
+        </geometry>
+      </collision>
+      <collision name="blue usv_collider_cylinder.003">
+        <pose>0.283564 -0.295886 -0.045978 0.0 0.0 0.0</pose>
+        <geometry>
+          <cylinder>
+            <radius>0.132203</radius>
+            <length>0.264407</length>
+          </cylinder>
+        </geometry>
+      </collision>
+      <collision name="blue usv_collider_cylinder.004">
+        <pose>-0.447734 -0.30143 -0.126513 0.0 0.0 0.0</pose>
+        <geometry>
+          <cylinder>
+            <radius>0.040196</radius>
+            <length>0.040861</length>
+          </cylinder>
+        </geometry>
+      </collision>
+      <collision name="blue usv_collider_box.001">
+        <pose>0.488345 0.302388 0.086141 0.0 0.0 0.0</pose>
+        <geometry>
+          <box>
+            <size>0.197621 0.049447 0.105333</size>
+          </box>
+        </geometry>
+      </collision>
+      <collision name="blue usv_collider_cylinder.005">
+        <pose>0.406722 0.321876 0.030426 0.0 0.0 0.0</pose>
+        <geometry>
+          <cylinder>
+            <radius>0.111828</radius>
+            <length>0.223656</length>
+          </cylinder>
+        </geometry>
+      </collision>
+      <collision name="blue usv_collider_cylinder.006">
+        <pose>-0.017902 0.360024 0.01984 0.0 0.0 0.0</pose>
+        <geometry>
+          <cylinder>
+            <radius>0.411411</radius>
+            <length>0.135532</length>
+          </cylinder>
+        </geometry>
+      </collision>
+      <collision name="blue usv_collider_box.003">
+        <pose>-0.012113 0.363698 0.083833 0.0 0.0 0.0</pose>
+        <geometry>
+          <box>
+            <size>0.872756 0.125557 0.116921</size>
+          </box>
+        </geometry>
+      </collision>
+      <collision name="blue usv_collider_cylinder.007">
+        <pose>0.283564 0.295886 -0.045978 0.0 0.0 0.0</pose>
+        <geometry>
+          <cylinder>
+            <radius>0.132203</radius>
+            <length>0.264407</length>
+          </cylinder>
+        </geometry>
+      </collision>
+      <collision name="blue usv_collider_box.005">
+        <pose>-0.104158 0.295896 -0.043697 0.0 0.0 0.0</pose>
+        <geometry>
+          <box>
+            <size>0.696765 0.018217 0.370259</size>
+          </box>
+        </geometry>
+      </collision>
+      <collision name="blue usv_collider_cylinder.008">
+        <pose>-0.447734 0.30143 -0.126513 0.0 0.0 0.0</pose>
+        <geometry>
+          <cylinder>
+            <radius>0.040196</radius>
+            <length>0.040861</length>
+          </cylinder>
+        </geometry>
+      </collision>
+      <collision name="blue usv_collider_box.007">
+        <pose>0.299059 -0.0 0.142501 0.0 0.0 0.0</pose>
+        <geometry>
+          <box>
+            <size>0.0257 0.500356 0.037959</size>
+          </box>
+        </geometry>
+      </collision>
+      <collision name="blue usv_collider_box.009">
+        <pose>-0.300152 0.0 0.142501 0.0 0.0 0.0</pose>
+        <geometry>
+          <box>
+            <size>0.0257 0.500356 0.037959</size>
+          </box>
+        </geometry>
+      </collision>
+      <collision name="blue usv_collider_box.010">
+        <pose>0.298121 -0.317568 0.130778 0.0 0.0 0.0</pose>
+        <geometry>
+          <box>
+            <size>0.043582 0.183315 0.063965</size>
+          </box>
+        </geometry>
+      </collision>
+      <collision name="blue usv_collider_box.011">
+        <pose>-0.29897 -0.317568 0.130778 0.0 0.0 0.0</pose>
+        <geometry>
+          <box>
+            <size>0.043582 0.183315 0.063965</size>
+          </box>
+        </geometry>
+      </collision>
+      <collision name="blue usv_collider_box.012">
+        <pose>-0.29897 0.317568 0.130778 0.0 0.0 0.0</pose>
+        <geometry>
+          <box>
+            <size>0.043582 0.183315 0.063965</size>
+          </box>
+        </geometry>
+      </collision>
+      <collision name="blue usv_collider_box.013">
+        <pose>0.298121 0.317568 0.130778 0.0 0.0 0.0</pose>
+        <geometry>
+          <box>
+            <size>0.043582 0.183315 0.063965</size>
+          </box>
+        </geometry>
+      </collision>
+      <collision name="blue usv_collider_cylinder.009">
+        <pose>-0.253322 -0.00144 0.117093 0.0 0.0 0.0</pose>
+        <geometry>
+          <cylinder>
+            <radius>0.016745</radius>
+            <length>0.03349</length>
+          </cylinder>
+        </geometry>
+      </collision>
+      <collision name="blue usv_collider_box.014">
+        <pose>0.003337 -0.36614 0.160429 0.0 0.0 0.0</pose>
+        <geometry>
+          <box>
+            <size>0.415567 0.151904 0.045952</size>
+          </box>
+        </geometry>
+      </collision>
+      <collision name="blue usv_collider_box.015">
+        <pose>0.003337 0.36614 0.160429 0.0 0.0 0.0</pose>
+        <geometry>
+          <box>
+            <size>0.415567 0.151904 0.045952</size>
+          </box>
+        </geometry>
+      </collision>
+      <collision name="blue usv_collider_box.016">
+        <pose>-0.467242 0.314935 0.038698 0.0 0.0 0.0</pose>
+        <geometry>
+          <box>
+            <size>0.127101 0.074541 0.20022</size>
+          </box>
+        </geometry>
+      </collision>
+      <collision name="blue usv_collider_box.017">
+        <pose>-0.522288 0.295896 -0.211583 0.0 0.0 0.0</pose>
+        <geometry>
+          <box>
+            <size>0.150178 0.018217 0.034487</size>
+          </box>
+        </geometry>
+      </collision>
+      -->
   </link>
   <!-- ===================== Thrusters (props) ===================== -->
