Commit message: Account for accessory collision volumes in the buoyancy sizing
Assisted-by: Claude Fable 5 <noreply@anthropic.com>
Signed-off-by: Carlos Aguero <caguero@honurobotics.com>

File: bluerov2_description/urdf/accessories.xacro (robot description, xacro)
@@ -14,4 +14,11 @@
   <xacro:property name="accessory_mass"
     value="${dict(ping360=0.5, payload_skid=3.0, roof_rack=0.2, sonoptix_echo=0.75, omniscan_450_fs=0.44, marinesitu_c3=0.43, explorehd_camera=0.08, dvl_a50=0.17, newton_gripper=0.5, sediment_sampler=0.5)}"/>
+  <!-- Displaced volume (m^3) of each accessory's COLLISION geometry. The
+       Buoyancy plugin sums every collision in the model, so the analytic hull
+       box in bluerov2.urdf.xacro must shrink by this amount to keep the total
+       displacement on target. Only the claws carry collisions; keep these in
+       sync with the collision boxes below. -->
+  <xacro:property name="accessory_volume"
+    value="${dict(ping360=0.0, payload_skid=0.0, roof_rack=0.0, sonoptix_echo=0.0, omniscan_450_fs=0.0, marinesitu_c3=0.0, explorehd_camera=0.0, dvl_a50=0.0, newton_gripper=0.05*0.06*0.06 + 2*0.06*0.012*0.03, sediment_sampler=0.05*0.06*0.06 + 2*0.09*0.02*0.026)}"/>
   <!-- ===== helpers ===== -->
   <xacro:macro name="_box_accessory" params="name xyz rpy parent size mass:=0.3">

File: bluerov2_description/urdf/bluerov2.urdf.xacro (robot description, xacro)
@@ -37,6 +37,11 @@
   <xacro:property name="total_mass"
     value="${base_mass + n_thrusters * thruster_mass + acc_mass_total}"/>
+  <!-- The Buoyancy plugin sums EVERY collision in the model, so accessories
+       that carry collisions (the claws) already displace water; shrink the
+       hull box by their volume to keep total displacement on target. -->
+  <xacro:property name="acc_volume_total"
+    value="${fsum([accessory_volume[a['type']] for a in cfg.get('accessories', [])])}"/>
   <xacro:property name="buoyancy_volume"
-    value="${total_mass * (1.0 + buoyancy_margin) / water_density}"/>
+    value="${total_mass * (1.0 + buoyancy_margin) / water_density - acc_volume_total}"/>
   <xacro:property name="buoyancy_height"
     value="${buoyancy_volume / (footprint_x * footprint_y)}"/>

Commit message: Compute accessory inertias from geometry, dispatch types as macros, fix ament hook
Assisted-by: Claude Fable 5 <noreply@anthropic.com>
Signed-off-by: Carlos Aguero <caguero@honurobotics.com>

File: bluerov2_description/urdf/accessories.xacro (robot description, xacro)
@@ -22,9 +22,14 @@
     value="${dict(ping360=0.0, payload_skid=0.0, roof_rack=0.0, sonoptix_echo=0.0, omniscan_450_fs=0.0, marinesitu_c3=0.0, explorehd_camera=0.0, dvl_a50=0.0, newton_gripper=0.05*0.06*0.06 + 2*0.06*0.012*0.03, sediment_sampler=0.05*0.06*0.06 + 2*0.09*0.02*0.026)}"/>
   <!-- ===== helpers ===== -->
+  <!-- Inertia tensors follow from the primitive geometry and the mass, so they
+       track the mass table and the placeholder dimensions automatically. -->
   <xacro:macro name="_box_accessory" params="name xyz rpy parent size mass:=0.3">
+    <xacro:property name="d" value="${[float(v) for v in size.split()]}"/>
     <link name="${name}">
       <inertial>
         <mass value="${mass}"/>
-        <inertia ixx="0.001" ixy="0" ixz="0" iyy="0.001" iyz="0" izz="0.001"/>
+        <inertia ixx="${float(mass)/12.0 * (d[1]**2 + d[2]**2)}" ixy="0" ixz="0"
+                 iyy="${float(mass)/12.0 * (d[0]**2 + d[2]**2)}" iyz="0"
+                 izz="${float(mass)/12.0 * (d[0]**2 + d[1]**2)}"/>
       </inertial>
       <visual>
@@ -42,5 +47,7 @@
       <inertial>
         <mass value="${mass}"/>
-        <inertia ixx="0.001" ixy="0" ixz="0" iyy="0.001" iyz="0" izz="0.001"/>
+        <inertia ixx="${float(mass)/12.0 * (3*float(radius)**2 + float(length)**2)}" ixy="0" ixz="0"
+                 iyy="${float(mass)/12.0 * (3*float(radius)**2 + float(length)**2)}" iyz="0"
+                 izz="${float(mass)/2.0 * float(radius)**2}"/>
       </inertial>
       <visual>
@@ -60,5 +67,8 @@
       <inertial>
         <mass value="${accessory_mass['ping360']}"/>
-        <inertia ixx="0.001" ixy="0" ixz="0" iyy="0.001" iyz="0" izz="0.001"/>
+        <!-- Solid cylinder over the device envelope (r 38 mm, h 117 mm). -->
+        <inertia ixx="${accessory_mass['ping360']/12.0 * (3*0.038**2 + 0.117**2)}" ixy="0" ixz="0"
+                 iyy="${accessory_mass['ping360']/12.0 * (3*0.038**2 + 0.117**2)}" iyz="0"
+                 izz="${accessory_mass['ping360']/2.0 * 0.038**2}"/>
       </inertial>
       <visual>
@@ -112,6 +122,10 @@
     <link name="${name}_jaw_${side}">
       <inertial>
+        <origin xyz="0.03 0 0" rpy="0 0 0"/>
         <mass value="0.1"/>
-        <inertia ixx="0.0001" ixy="0" ixz="0" iyy="0.0001" iyz="0" izz="0.0001"/>
+        <!-- Box 0.06 x 0.012 x 0.03, about its own centre (the visual pose). -->
+        <inertia ixx="${0.1/12.0 * (0.012**2 + 0.03**2)}" ixy="0" ixz="0"
+                 iyy="${0.1/12.0 * (0.06**2 + 0.03**2)}" iyz="0"
+                 izz="${0.1/12.0 * (0.06**2 + 0.012**2)}"/>
       </inertial>
       <visual>
@@ -137,5 +151,8 @@
       <inertial>
         <mass value="0.3"/>
-        <inertia ixx="0.0005" ixy="0" ixz="0" iyy="0.0005" iyz="0" izz="0.0005"/>
+        <!-- Box 0.05 x 0.06 x 0.06 (the housing collision/visual). -->
+        <inertia ixx="${0.3/12.0 * (0.06**2 + 0.06**2)}" ixy="0" ixz="0"
+                 iyy="${0.3/12.0 * (0.05**2 + 0.06**2)}" iyz="0"
+                 izz="${0.3/12.0 * (0.05**2 + 0.06**2)}"/>
       </inertial>
       <visual>
@@ -160,6 +177,10 @@
     <link name="${name}_cup_${side}">
       <inertial>
+        <origin xyz="0.028 0 0" rpy="0 0 0"/>
         <mass value="0.1"/>
-        <inertia ixx="0.0001" ixy="0" ixz="0" iyy="0.0001" iyz="0" izz="0.0001"/>
+        <!-- Dominant arm box 0.055 x 0.01 x 0.012, about its own centre. -->
+        <inertia ixx="${0.1/12.0 * (0.01**2 + 0.012**2)}" ixy="0" ixz="0"
+                 iyy="${0.1/12.0 * (0.055**2 + 0.012**2)}" iyz="0"
+                 izz="${0.1/12.0 * (0.055**2 + 0.01**2)}"/>
       </inertial>
       <visual>
@@ -190,19 +211,12 @@
     <xacro:_sampler_cup name="${name}" side="right" y="-0.02" axis="0 0 -1"/>
   </xacro:macro>
-  <!-- ===== recursive dispatcher: mount each config accessory by type ===== -->
+  <!-- ===== recursive dispatcher: mount each config accessory by type =====
+       The config `type` IS the macro name, invoked directly; an unknown type
+       fails the build loudly instead of silently mounting nothing. -->
   <xacro:macro name="mount_accessories" params="items parent:=base_link">
     <xacro:if value="${len(items) > 0}">
       <xacro:property name="a" value="${items[0]}"/>
-      <xacro:property name="t" value="${a['type']}"/>
-      <xacro:if value="${t == 'ping360'}">         <xacro:ping360         name="${a['name']}" xyz="${a['xyz']}" rpy="${a['rpy']}" parent="${parent}"/></xacro:if>
-      <xacro:if value="${t == 'payload_skid'}">    <xacro:payload_skid    name="${a['name']}" xyz="${a['xyz']}" rpy="${a['rpy']}" parent="${parent}"/></xacro:if>
-      <xacro:if value="${t == 'roof_rack'}">       <xacro:roof_rack       name="${a['name']}" xyz="${a['xyz']}" rpy="${a['rpy']}" parent="${parent}"/></xacro:if>
-      <xacro:if value="${t == 'sonoptix_echo'}">   <xacro:sonoptix_echo   name="${a['name']}" xyz="${a['xyz']}" rpy="${a['rpy']}" parent="${parent}"/></xacro:if>
-      <xacro:if value="${t == 'omniscan_450_fs'}"> <xacro:omniscan_450_fs name="${a['name']}" xyz="${a['xyz']}" rpy="${a['rpy']}" parent="${parent}"/></xacro:if>
-      <xacro:if value="${t == 'marinesitu_c3'}">   <xacro:marinesitu_c3   name="${a['name']}" xyz="${a['xyz']}" rpy="${a['rpy']}" parent="${parent}"/></xacro:if>
-      <xacro:if value="${t == 'explorehd_camera'}"><xacro:explorehd_camera name="${a['name']}" xyz="${a['xyz']}" rpy="${a['rpy']}" parent="${parent}"/></xacro:if>
-      <xacro:if value="${t == 'dvl_a50'}">         <xacro:dvl_a50         name="${a['name']}" xyz="${a['xyz']}" rpy="${a['rpy']}" parent="${parent}"/></xacro:if>
-      <xacro:if value="${t == 'newton_gripper'}"> <xacro:newton_gripper  name="${a['name']}" xyz="${a['xyz']}" rpy="${a['rpy']}" parent="${parent}"/></xacro:if>
-      <xacro:if value="${t == 'sediment_sampler'}"><xacro:sediment_sampler name="${a['name']}" xyz="${a['xyz']}" rpy="${a['rpy']}" parent="${parent}"/></xacro:if>
+      <xacro:call macro="${a['type']}" name="${a['name']}"
+                  xyz="${a['xyz']}" rpy="${a['rpy']}" parent="${parent}"/>
       <xacro:mount_accessories items="${items[1:]}" parent="${parent}"/>
     </xacro:if>

File: bluerov2_description/urdf/bluerov2.urdf.xacro (robot description, xacro)
@@ -60,4 +60,8 @@
                izz="${base_mass/12.0 * (footprint_x**2 + footprint_y**2)}"/>
     </inertial>
+    <!-- The DAVE hull meshes are authored in 25 mm units with a +90-deg-about-Y
+     node transform, so 0.025 puts them in metres: 0.450 x 0.339 x 0.250 m,
+     matching the real 457 x 338 x 254 mm and footprint_x/footprint_y above.
+     Both variant meshes share the scale. -->
     <visual>
       <origin xyz="0 0 0" rpy="0 0 0"/>

File: bluerov2_description/urdf/thruster.xacro (robot description, xacro)
@@ -19,7 +19,8 @@
     <link name="thruster${number}">
       <inertial>
-        <!-- T200 in air ~0.344 kg; short-cylinder inertia (r~38 mm, h~40 mm).
-             Note izz <= ixx + iyy must hold or sdformat rejects the link. -->
-        <mass value="0.344"/>
+        <!-- T200 in air (thruster_mass, set in bluerov2.urdf.xacro); short
+             cylinder inertia (r~38 mm, h~40 mm). Note izz <= ixx + iyy must
+             hold or sdformat rejects the link. -->
+        <mass value="${thruster_mass}"/>
         <inertia ixx="1.7e-4" ixy="0.0" ixz="0.0"
                  iyy="1.7e-4" iyz="0.0" izz="2.5e-4"/>
