Commit message: Address review feedback on the part macro prototype
Point by point against caguero's review.

1. mount_parts removed rather than wired to the probe. The dispatcher is
   ahead of where we are — there are no assemblies to exercise it against —
   so it comes back with the assembly work. Recording the trap found while
   testing it, so it does not have to be found twice: an inline list of
   dicts fails, because xacro closes the ${...} on the first } inside the
   dict ("error: '{' was never closed"). Building them with dict() instead
   of braces works:

       <xacro:property name="items" value="${[
           dict(type=part, name='probe',        xyz='0 0 0'),
           dict(type=part, name='probe_nocol',  xyz='2 0 0', collision=False),
           dict(type=part, name='probe_stacked', xyz='0 0 0.5', parent='probe')]}"/>

2. part_probe no longer declares <xacro:arg name="part">. Omitting part:=
   now fails with "Undefined substitution argument part" instead of the
   confusing "unknown macro name: xacro:". Note xacro:arg requires a
   default attribute, so dropping the declaration is the only way to get
   the good error.

3. The "order matters" claim is gone. It was wrong — URDF only needs the
   link to exist somewhere in the document, and a child listed before its
   parent parses fine. It lived only in the mount_parts doc block.

4. Origin convention stated once. The origin is the centroid of the mesh,
   equivalently its center of mass at uniform density, with the frame per
   REP 103. The conflicting "in the place the part would sensibly be
   mounted from" is removed from the acceptance checklist. Also notes that
   the mesh centroid is not the part's center of gravity, which is the
   other half of the terminology overload.

5. Acceptance step 5 gains a mesh-existence check. check_urdf validates
   XML but does not resolve package://, so a part passed acceptance with
   no .glb in the package at all.

6. The part macro contract — name, parent, xyz, rpy, collision — is now
   stated in parts.xacro. A macro that drops one fails with
   'Invalid parameter "collision"'.

7. "Source of truth" dropped throughout. It appeared six times naming
   three different things. Replaced with who authors what and what reads
   what: the modeler works in SDF, ROS and Gazebo read the xacro, and the
   import script is the seam. SDF is not interim and model.sdf is not
   deleted — it stays as the record of what was delivered.

Also: US spelling throughout the package, and a note on the mast's
placeholder inertial origin, which assumes a base-origin mesh and needs
revisiting when the corrected mesh lands.

Co-Authored-By: Claude Opus 5 <noreply@anthropic.com>

File: bluerobotics_parts/models/blueboat_antenna_mast/blueboat_antenna_mast.collision.xacro (robot description, xacro)
@@ -3,7 +3,8 @@
   GENERATED FILE — DO NOT EDIT.
   Written by scripts/import_part.py from model.sdf, and overwritten on every
-  re-import. Any hand edit here is lost the next time the modeller redelivers.
+  re-import. Any hand edit here is lost the next time the modeler redelivers.
   To change this collision geometry, edit model.sdf and re-run the import.
-  model.sdf is the source of physical truth for the collision geometry.
+  model.sdf is the modeler's work product; this file is what ROS and Gazebo
+  actually read.
   The macro is called from blueboat_antenna_mast.urdf.xacro, which is the
   hand-authored half and is never touched by the import.

File: bluerobotics_parts/models/blueboat_antenna_mast/blueboat_antenna_mast.urdf.xacro (robot description, xacro)
@@ -2,15 +2,16 @@
 <!--
   blueboat_antenna_mast — part macro.
-  This file is HAND-AUTHORED and is never written by tooling. It is the SOURCE
-  OF TRUTH for this part's mass, inertia tensor and center-of-gravity pose.
-  Nothing downstream re-derives them: assemblies compose what is written here.
-  See AUR_BUOYANCY_DESIGN.md.
+  This file is HAND-AUTHORED and is never written by tooling. This part's mass,
+  inertia tensor and center-of-gravity pose are stated here and nowhere else;
+  nothing downstream re-derives them, and assemblies compose what is written
+  here. See AUR_BUOYANCY_DESIGN.md.
   The generated half lives in its own file, so the two never share a file and
   a re-import cannot touch anything written by hand:
     blueboat_antenna_mast.collision.xacro   GENERATED by scripts/import_part.py
                                             from model.sdf, overwritten on every
-                                            re-import. model.sdf is the source of
-                                            physical truth for the collision
-                                            geometry.
+                                            re-import. model.sdf is the
+                                            modeler's work product; the
+                                            generated xacro is what ROS and
+                                            Gazebo read.
   This collision is tied to the part. When assembled into a vehicle the
   collision geometry can be ignored — see collision:=false in the macro call.
@@ -32,5 +33,9 @@
     <link name="${name}">
       <inertial>
-        <!-- TODO: Update.  Just using rough numbers for prototype -->
+        <!-- TODO: Update. Rough numbers for the prototype — a slender rod.
+             These also assume a mesh whose origin is at the base of the mast.
+             The delivered mesh currently is, but that violates rule 2 (origin
+             at the centroid of the mesh) and is back with the modeler. Revisit
+             this origin when the corrected mesh lands. -->
         <origin xyz="0 0 0.5" rpy="0 0 0"/>
         <mass value="1.0"/>
@@ -42,5 +47,5 @@
         <origin xyz="0 0 0" rpy="0 0 0"/>
         <geometry>
-          <!-- Delivered by the modeller; PBR materials ride inside the .glb. -->
+          <!-- Delivered by the modeler; PBR materials ride inside the .glb. -->
           <mesh filename="package://bluerobotics_parts/models/blueboat_antenna_mast/blueboat_antenna_mast.visual.glb"/>
         </geometry>

File: bluerobotics_parts/urdf/part_probe.urdf.xacro (robot description, xacro)
@@ -12,7 +12,10 @@
 <robot name="part_probe" xmlns:xacro="http://ros.org/wiki/xacro">
   <xacro:include filename="$(find bluerobotics_parts)/urdf/parts.xacro"/>
-  <!-- Part name = macro name = directory name. No default: forgetting the
-       argument should fail loudly rather than probe nothing. -->
-  <xacro:arg name="part" default=""/>
+  <!-- Part name = macro name = directory name. Deliberately NOT declared with
+       <xacro:arg>: omitting part:= then fails with "Undefined substitution
+       argument part", which names what is missing. Declaring it with an empty
+       default instead expands to nothing and reports the useless "unknown
+       macro name: xacro:". Note that xacro:arg requires a default attribute,
+       so leaving the declaration out is the only way to get the good error. -->
   <xacro:property name="part" value="$(arg part)"/>
   <link name="base_link"/>

File: bluerobotics_parts/urdf/parts.xacro (robot description, xacro)
@@ -3,16 +3,27 @@
   bluerobotics_parts — the parts-level macro library.
   PROTOTYPE. One part is wired up (blueboat_antenna_mast); the rest of the
-  catalog follows the same two lines once each part has a macro.
-  Include this once and you have every part available as a macro, plus the
-  dispatcher that mounts a list of them. An assembly should not include
-  individual part files directly — that is what this file is for.
+  catalog follows the same one line once each part has a macro.
+  Include this once and every part is available as a macro. An assembly should
+  not include individual part files directly — that is what this file is for.
       <xacro:include filename="$(find bluerobotics_parts)/urdf/parts.xacro"/>
-      <xacro:mount_parts items="${parts}" parent="base_link"/>
-  Generalized from bluerov2_description/urdf/accessories.xacro, with one
-  deliberate difference. There, a central accessory_mass dict fed helper macros
-  that DERIVED inertia from primitive dimensions. Here each part carries its own
-  measured mass, inertia tensor and center-of-gravity pose in its own file, so
-  there is no table here and nothing central to keep in sync. The part is the
-  source of truth. See AUR_BUOYANCY_DESIGN.md.
+      <xacro:blueboat_antenna_mast name="mast" parent="base_link" xyz="0 0 0.2"/>
+  ===== the part macro contract =====
+  Every macro included below takes exactly these parameters, in this order:
+      name       link name for this instance; the fixed joint is <name>_joint
+      parent     link to attach to
+      xyz / rpy  mount pose relative to parent (meters / radians)
+      collision  false to instantiate the part with no contact geometry
+  This is a contract, not a convention. A dispatcher that mounts parts from a
+  config list forwards exactly this set to whichever macro a `type` names, so a
+  macro that drops or renames one fails with `Invalid parameter "collision"`
+  instead of doing something surprising. The vessel macros will have to honor
+  it too.
+  That dispatcher (`mount_parts`, generalized from accessories.xacro) is not
+  here yet. It belongs with the assembly work, where it can be exercised
+  against a real vehicle rather than against itself.
+  Mass, inertia tensor and center-of-gravity pose are carried by each part in
+  its own file, hand-authored from measurement or the vendor. There is no
+  central mass table here and so nothing to keep in sync. See
+  AUR_BUOYANCY_DESIGN.md.
 -->
 <robot xmlns:xacro="http://ros.org/wiki/xacro">
@@ -21,29 +32,3 @@
        name and the macro name are all the part name from models/parts.csv. -->
   <xacro:include filename="$(find bluerobotics_parts)/models/blueboat_antenna_mast/blueboat_antenna_mast.urdf.xacro"/>
-  <!-- ===== dispatcher =====
-       Mounts each entry of `items` by calling the macro its `type` names, so an
-       unknown type fails the build loudly instead of silently mounting nothing.
-       Recursion rather than iteration because xacro has no loop construct.
-       Each item is a dict:
-         type       part name — must match a macro included above  (required)
-         name       link name for this instance                    (required)
-         xyz / rpy  mount pose relative to parent, default zero    (optional)
-         parent     override the dispatcher's parent               (optional)
-         collision  false to mount the part without contact geometry (optional)
-       `parent` per item is what lets a part hang off another part rather than
-       off the chassis — a sensor on the mast rather than on the hull. Order
-       matters when it is used: the parent must already be mounted.
-  -->
-  <xacro:macro name="mount_parts" params="items parent:=base_link">
-    <xacro:if value="${len(items) > 0}">
-      <xacro:property name="p" value="${items[0]}"/>
-      <xacro:call macro="${p['type']}"
-                  name="${p['name']}"
-                  parent="${p.get('parent', parent)}"
-                  xyz="${p.get('xyz', '0 0 0')}"
-                  rpy="${p.get('rpy', '0 0 0')}"
-                  collision="${p.get('collision', True)}"/>
-      <xacro:mount_parts items="${items[1:]}" parent="${parent}"/>
-    </xacro:if>
-  </xacro:macro>
 </robot>
