Commit message: BlueBoat: chassis frame orientation per the glTF axes convention, verified
The main result of this increment: base_link's frame is verified to follow
ISO 9787 / REP 103 (x forward, y left, z up) against the PR #83 chassis
geometry in Gazebo. The check was visual, in a visuals only spike world
(~/maritime_ws/spike/blueboat_frames, not in the repo) generated from the
real Gazebo flavoured expansion: one link, one visual, an ISO reference
triad beside the boat, View > Frames showing just the link and glTF frames
as in gltf-robotics docs/walkthroughs/coordinate_orientation_demo.md.

- parts.xacro: part_visual takes axes:=gltf for deliveries in the Honu glTF
  Asset Profile's axes (+x left, +y up, +z forward): rpy 1.5708 0 1.5708 for
  Gazebo, 0 0 1.5708 for RViz from Lyrical on (it adds the roll itself), as
  the walkthrough sets. axes:=legacy (default) keeps the old rotation for
  the earlier exports.
- blueboat_chassis, m200_weedless_prop_ccw/_cw opt in with axes="gltf".
  Rotated into base_link, the chassis mesh is 1.19 m along x and 0.93 m
  along y, on the colliders. Prop slot poses are unchanged.
- The two tests that pinned one visual rotation per flavour accept both.
- worlds/parts_check.sdf regenerated: the three parts' visual poses only.

Co-Authored-By: Claude Opus 5.5 <noreply@anthropic.com>

File: bluerobotics_parts/urdf/blueboat_chassis.urdf.xacro (robot description, xacro)
@@ -49,5 +49,5 @@
                  izz="3.23"/>
       </inertial>
-      <xacro:part_visual mesh="package://bluerobotics_parts/models/blueboat_chassis/blueboat_chassis_visual.glb"/>
+      <xacro:part_visual mesh="package://bluerobotics_parts/models/blueboat_chassis/blueboat_chassis_visual.glb" axes="gltf"/>
       <xacro:if value="${collision}">
         <collision>

File: bluerobotics_parts/urdf/m200_weedless_prop_ccw.urdf.xacro (robot description, xacro)
@@ -30,5 +30,5 @@
                  izz="3.11438e-05"/>
       </inertial>
-      <xacro:part_visual mesh="package://bluerobotics_parts/models/m200_weedless_prop_ccw/m200_weedless_prop_ccw_visual.glb"/>
+      <xacro:part_visual mesh="package://bluerobotics_parts/models/m200_weedless_prop_ccw/m200_weedless_prop_ccw_visual.glb" axes="gltf"/>
       <xacro:if value="${collision}">
         <collision>

File: bluerobotics_parts/urdf/m200_weedless_prop_cw.urdf.xacro (robot description, xacro)
@@ -32,5 +32,5 @@
                  izz="3.11438e-05"/>
       </inertial>
-      <xacro:part_visual mesh="package://bluerobotics_parts/models/m200_weedless_prop_cw/m200_weedless_prop_cw_visual.glb"/>
+      <xacro:part_visual mesh="package://bluerobotics_parts/models/m200_weedless_prop_cw/m200_weedless_prop_cw_visual.glb" axes="gltf"/>
       <xacro:if value="${collision}">
         <collision>

File: bluerobotics_parts/urdf/parts.xacro (robot description, xacro)
@@ -67,8 +67,10 @@
   <xacro:arg name="gltf_up" default="y"/>
   <xacro:property name="gltf_visual_rpy" value="${'1.5708 0 0' if '$(arg gltf_up)' == 'z' else '0 0 0'}"/>
-  <!-- A part's visual mesh, with the glTF up axis handling above. -->
-  <xacro:macro name="part_visual" params="mesh xyz:='0 0 0'">
+  <!-- axes="gltf": a delivery in the Honu glTF Asset Profile's axes (+x left, +y up, +z forward; profile Axes section), rotated into ISO 9787 / REP 103 as in gltf-robotics docs/walkthroughs/coordinate_orientation_demo.md: roll 90 then yaw 90 for Gazebo (and RViz before Lyrical), which add nothing on load; yaw 90 only for RViz from Lyrical on, which adds the roll itself. New deliveries use it; axes="legacy" (the default) keeps the rotation above for the earlier exports. -->
+  <xacro:property name="gltf_profile_rpy" value="${'1.5708 0 1.5708' if '$(arg gltf_up)' == 'z' else '0 0 1.5708'}"/>
+  <!-- A part's visual mesh, with the glTF axes handling above. -->
+  <xacro:macro name="part_visual" params="mesh xyz:='0 0 0' axes:='legacy'">
     <visual>
-      <origin xyz="${xyz}" rpy="${gltf_visual_rpy}"/>
+      <origin xyz="${xyz}" rpy="${gltf_profile_rpy if axes == 'gltf' else gltf_visual_rpy}"/>
       <geometry>
         <mesh filename="${mesh}"/>
