Commit message: Fit T200 bodies on chassis body slots by default and lay the camera placeholder along its sensing axis
Assisted-by: Claude Fable 5 <noreply@anthropic.com>
Signed-off-by: Carlos Agüero <caguero@honurobotics.com>

File: bluerobotics_parts/urdf/bluerov2_chassis.urdf.xacro (robot description, xacro)
@@ -6,6 +6,6 @@
   it by hand from here on.
   The chassis is the standard (6 thruster) BlueROV2 hull as one rigid body,
-  T200 thruster bodies included; only the propellers are separate parts, on
-  the thruster slots. Mass is the hull plus six T200 bodies (9.4 + 6 x
+  with T200 bodies and propellers as parts on the thruster_body_N and
+  thruster_N slots (all fitted by default). Mass is the hull plus six T200 bodies (9.4 + 6 x
   0.3049 kg, the T200 in air mass minus its prop part), so the default
   loadout totals the reference ~11.5 kg in air. Inertia: tensor shape
@@ -43,4 +43,10 @@
             payload=dict(xyz='0 0 -0.17', rpy='0 0 0', accepts=['payload_skid'], default='none'),
             rack=dict(xyz='0 0 0.17', rpy='0 0 0', accepts=['roof_rack'], default='none'),
+            thruster_body_1=dict(xyz='0.14 -0.092 0.0', rpy='0 0 -2.3562', accepts=['t200_thruster'], default='t200_thruster', collision=False),
+            thruster_body_2=dict(xyz='0.14 0.092 0.0', rpy='0 0 2.3562', accepts=['t200_thruster'], default='t200_thruster', collision=False),
+            thruster_body_3=dict(xyz='-0.15 -0.092 0.0', rpy='0 0 -0.7854', accepts=['t200_thruster'], default='t200_thruster', collision=False),
+            thruster_body_4=dict(xyz='-0.15 0.092 0.0', rpy='0 0 0.7854', accepts=['t200_thruster'], default='t200_thruster', collision=False),
+            thruster_body_5=dict(xyz='0.0 -0.109 0.077', rpy='0 1.5708 0', accepts=['t200_thruster'], default='t200_thruster', collision=False),
+            thruster_body_6=dict(xyz='0.0 0.109 0.077', rpy='0 1.5708 0', accepts=['t200_thruster'], default='t200_thruster', collision=False),
         ),
         frames=dict(
@@ -57,8 +63,10 @@
              volumes put it 3 cm low, which made surge climb. -->
         <origin xyz="0.00979373 -0.000225576 0.011" rpy="0 0 0"/>
-        <mass value="11.2297"/>
-        <inertia ixx="0.167167" ixy="-6.77391e-06" ixz="-0.000601754"
-                 iyy="0.208312" iyz="2.46933e-05"
-                 izz="0.263922"/>
+        <mass value="9.4"/>
+        <!-- Bare hull: the T200 bodies and props are parts on the
+             thruster_body / thruster slots. Tensor scaled to this mass. -->
+        <inertia ixx="1.399298e-01" ixy="-5.670210e-06" ixz="-5.037078e-04"
+                 iyy="1.743709e-01" iyz="2.066992e-05"
+                 izz="2.209201e-01"/>
       </inertial>
       <xacro:part_visual mesh="package://bluerobotics_parts/models/bluerov2_chassis/bluerov2_chassis.visual.glb"/>

File: bluerobotics_parts/urdf/bluerov2_heavy_chassis.urdf.xacro (robot description, xacro)
@@ -3,6 +3,6 @@
   bluerov2_heavy_chassis part macro.
   Hand derived from the bluerov2_chassis part: the Heavy kit hull (wider
-  frame, 8 thrusters) as one rigid body, T200 bodies included; only the
-  propellers are separate parts. The visual is the DAVE heavy mesh, a
+  frame, 8 thrusters) as one rigid body, with T200 bodies and propellers
+  as parts on their slots. The visual is the DAVE heavy mesh, a
   PLACEHOLDER until the artist delivers the heavy shell; collisions are the
   standard chassis set (approximate for the wider hull). Mass is the heavy
@@ -44,4 +44,12 @@
             payload=dict(xyz='0 0 -0.17', rpy='0 0 0', accepts=['payload_skid'], default='none'),
             rack=dict(xyz='0 0 0.17', rpy='0 0 0', accepts=['roof_rack'], default='none'),
+            thruster_body_1=dict(xyz='0.14 -0.092 0.0', rpy='0 0 -2.3562', accepts=['t200_thruster'], default='t200_thruster', collision=False),
+            thruster_body_2=dict(xyz='0.14 0.092 0.0', rpy='0 0 2.3562', accepts=['t200_thruster'], default='t200_thruster', collision=False),
+            thruster_body_3=dict(xyz='-0.15 -0.092 0.0', rpy='0 0 -0.7854', accepts=['t200_thruster'], default='t200_thruster', collision=False),
+            thruster_body_4=dict(xyz='-0.15 0.092 0.0', rpy='0 0 0.7854', accepts=['t200_thruster'], default='t200_thruster', collision=False),
+            thruster_body_5=dict(xyz='0.118 -0.215 0.064', rpy='0 1.5708 0', accepts=['t200_thruster'], default='t200_thruster', collision=False),
+            thruster_body_6=dict(xyz='0.118 0.215 0.064', rpy='0 1.5708 0', accepts=['t200_thruster'], default='t200_thruster', collision=False),
+            thruster_body_7=dict(xyz='-0.118 -0.215 0.064', rpy='0 1.5708 0', accepts=['t200_thruster'], default='t200_thruster', collision=False),
+            thruster_body_8=dict(xyz='-0.118 0.215 0.064', rpy='0 1.5708 0', accepts=['t200_thruster'], default='t200_thruster', collision=False),
         ),
         frames=dict(
@@ -58,10 +66,10 @@
              volumes put it 3 cm low, which made surge climb. -->
         <origin xyz="0.00979373 -0.000225576 0.011" rpy="0 0 0"/>
-        <mass value="15.1896"/>
-        <!-- Standard chassis tensor scaled to the heavy mass; refine when
-             the heavy shell arrives. -->
-        <inertia ixx="0.226119" ixy="-9.16233e-06" ixz="-0.000813946"
-                 iyy="0.281774" iyz="3.34021e-05"
-                 izz="0.357013"/>
+        <mass value="12.75"/>
+        <!-- Bare hull: the T200 bodies and props are parts on the
+             thruster_body / thruster slots. Tensor scaled to this mass. -->
+        <inertia ixx="1.898021e-01" ixy="-7.690769e-06" ixz="-6.832182e-04"
+                 iyy="2.365183e-01" iyz="2.803739e-05"
+                 izz="2.996732e-01"/>
       </inertial>
       <!-- DAVE heavy hull, authored in 25 mm units (0.025 scales to metres). -->

File: bluerobotics_parts/urdf/explorehd_camera.urdf.xacro (robot description, xacro)
@@ -32,4 +32,7 @@
       </inertial>
       <visual>
+        <!-- The cylinder primitive's axis is z; the camera points along +x
+             (the sensing direction), so lay the visual on its side. -->
+        <origin xyz="0 0 0" rpy="0 1.5708 0"/>
         <geometry><cylinder radius="${_r}" length="${_l}"/></geometry>
         <material name="${name}_mat"><color rgba="0.5 0.5 0.55 1"/></material>

File: bluerobotics_parts/urdf/t200_thruster.urdf.xacro (robot description, xacro)
@@ -24,8 +24,11 @@
       <inertial>
         <origin xyz="-0.00688307 0.00285552 -0.000166273" rpy="0 0 0"/>
-        <mass value="0.344"/>
-        <inertia ixx="0.00031312" ixy="-1.30503e-08" ixz="-2.56102e-07"
-                 iyy="0.00029151" iyz="-3.50359e-10"
-                 izz="0.000291503"/>
+        <!-- Body only: the full T200 is 0.344 kg in air; its propeller is
+             the separate t200_prop part (0.0391 kg), so body + prop sum to
+             the real thruster. -->
+        <mass value="0.3049466"/>
+        <inertia ixx="2.775723e-04" ixy="-1.156873e-08" ixz="-2.270274e-07"
+                 iyy="2.584156e-04" iyz="-3.105837e-10"
+                 izz="2.584094e-04"/>
       </inertial>
       <xacro:part_visual mesh="package://bluerobotics_parts/models/t200_thruster/t200_thruster.visual.glb"/>

Commit message: BlueROV2: name the datum frame base_footprint, per REP 105
Part frames are named <instance>_<frame>, which made the chassis datum
base_link_footprint. A frame entry may now give `link`, the exact link
name, used only when the part is the assembly root (part_frames
root:=True), so a part instantiated twice cannot clash; the chassis passes
root for parent "". The parts contract comment and docs/design/parts.md
describe the key. worlds/parts_check.sdf regenerated.

Tests: bluerobotics_parts 51, bluerov2_description 29, bluerov2_gazebo 79,
all pass.

Co-Authored-By: Claude Opus 5.5 <noreply@anthropic.com>

File: bluerobotics_parts/urdf/bluerov2_chassis.urdf.xacro (robot description, xacro)
@@ -28,5 +28,5 @@
 -->
 <robot xmlns:xacro="http://ros.org/wiki/xacro">
-  <!-- The delivered chassis mesh has its origin on the commissioned datum (commissions/commission-bluerov2.yaml): the center of the frame's footprint on its bottom plane, the base_footprint of REP 105. That point is the footprint frame. base_link stays at the main tube's center, (-0.013605, 0, 0.187846) from the datum, so the visual is placed by the opposite offset: gz-sim's Hydrodynamics samples the link origin's velocity but applies its wrench at the CoM, and with base_link on the datum, 0.19 m below the CoM, roll couples into sway (the axis test measured sway 31 degrees off axis).
+  <!-- The delivered chassis mesh has its origin on the commissioned datum (commissions/commission-bluerov2.yaml): the center of the frame's footprint on its bottom plane, the base_footprint of REP 105. That point is the base_footprint frame. base_link stays at the main tube's center, (-0.013605, 0, 0.187846) from the datum, so the visual is placed by the opposite offset: gz-sim's Hydrodynamics samples the link origin's velocity but applies its wrench at the CoM, and with base_link on the datum, 0.19 m below the CoM, roll couples into sway (the axis test measured sway 31 degrees off axis).
        The thruster_N and thruster_body_N poses are taken from the Blender assembly bluerov2_chassis.blend (the chassis file with t200_thruster, t200_prop_cw and t200_prop_ccw linked in): each instance's translation and rotation relative to the untransformed chassis, mapped from Blender axes to these (x = -Blender y, y = Blender x, z = Blender z) and moved by the datum offset above. A body and its prop share one pose, as their datums are the same point.
        Two corrections keep each thruster's positive thrust where ArduSub's Vectored frame puts it (AP_Motors6DOF.cpp, SUB_FRAME_VECTORED). The four horizontals are turned 90 degrees about z from the assembly, so +x lies along ArduSub's direction for that motor (1 aft starboard, 2 aft port, 3 fore starboard, 4 fore port); in the assembly they face the other diagonal, which is open with the modeler. The two verticals face up in the assembly, so their prop slots spin the occupant about -1 0 0 and positive thrust pushes down, as ArduSub's throttle factor of -1 expects.
@@ -63,5 +63,5 @@
         frames=dict(
             imu=dict(xyz='0 0 0', rpy='0 0 0'),
-            footprint=dict(xyz='0.013605 0 -0.187846', rpy='0 0 0'),
+            footprint=dict(xyz='0.013605 0 -0.187846', rpy='0 0 0', link='base_footprint'),
         ))}"/>
   </xacro:macro>
@@ -146,5 +146,6 @@
                       joint="${joint}" axis="${axis}" attach="${part_info['attach']}"/>
     <xacro:part_slots name="${name}" items="${list(part_info['slots'].items())}"/>
-    <xacro:part_frames name="${name}" items="${list(part_info['frames'].items())}"/>
+    <xacro:part_frames name="${name}" items="${list(part_info['frames'].items())}"
+                       root="${parent == ''}"/>
   </xacro:macro>
 </robot>

File: bluerobotics_parts/urdf/parts.xacro (robot description, xacro)
@@ -52,6 +52,8 @@
      collision), the mounting joint (part_joint), and its slots and frames as
      massless links named <name>_<slot> / <name>_<frame> (part_slots,
-     part_frames). They show up in TF and are lumped away in Gazebo, where
-     they survive as frames of the same name.
+     part_frames), or the entry's `link` where a frame needs a conventional
+     name (the chassis's base_footprint, REP 105), used only when the part is
+     the assembly root (root:=True), so a second instance cannot clash. They show up in TF and are
+     lumped away in Gazebo, where they survive as frames of the same name.
   The URDF xacro is the part. It may be bootstrapped from a modeler's SDF
   with scripts/sdf_to_part.py or written by hand; nothing downstream knows
@@ -122,13 +124,13 @@
   <!-- All of a part's slots (or frames: same thing to the URDF) from its
        part_info table (xacro has no loop; recurse over list(table.items())). -->
-  <xacro:macro name="part_slots" params="name items">
+  <xacro:macro name="part_slots" params="name items root:=False">
     <xacro:if value="${len(items) > 0}">
-      <xacro:part_slot name="${name}_${items[0][0]}" parent="${name}"
+      <xacro:part_slot name="${items[0][1]['link'] if root and 'link' in items[0][1] else name + '_' + items[0][0]}" parent="${name}"
                        xyz="${items[0][1]['xyz']}" rpy="${items[0][1].get('rpy', '0 0 0')}"/>
-      <xacro:part_slots name="${name}" items="${items[1:]}"/>
+      <xacro:part_slots name="${name}" items="${items[1:]}" root="${root}"/>
     </xacro:if>
   </xacro:macro>
-  <xacro:macro name="part_frames" params="name items">
-    <xacro:part_slots name="${name}" items="${items}"/>
+  <xacro:macro name="part_frames" params="name items root:=False">
+    <xacro:part_slots name="${name}" items="${items}" root="${root}"/>
   </xacro:macro>
   <!-- ===== catalog =====

Commit message: BlueROV2: sensors without visuals; accessories and gripper out of scope
Accessory visuals are out of scope while the work focuses on the
functional parts. The explorehd_camera, dvl_a50 and ping360 parts lose
their visuals (placeholder cylinders and the older ping360 .dae, which
stays in the package unused) and keep their link, inertia and frame, so
bluerov2_gazebo still hangs each sensor on that frame: topics unchanged.
Subsea manipulation is out of scope too; the gripper slot stays empty.

The chassis comment records that the collisions were checked against the
new chassis in Gazebo. The parts catalog and the BlueROV2 sensors and
configuration pages say the same in one line each.

Tests: bluerobotics_parts 51, bluerov2_description 29, bluerov2_gazebo 79,
all pass.

Co-Authored-By: Claude Opus 5.5 <noreply@anthropic.com>

File: bluerobotics_parts/urdf/bluerov2_chassis.urdf.xacro (robot description, xacro)
@@ -31,5 +31,5 @@
        The thruster_N and thruster_body_N poses are taken from the Blender assembly bluerov2_chassis.blend (the chassis file with t200_thruster, t200_prop_cw and t200_prop_ccw linked in): each instance's translation and rotation relative to the untransformed chassis, mapped from Blender axes to these (x = -Blender y, y = Blender x, z = Blender z) and moved by the datum offset above. A body and its prop share one pose, as their datums are the same point.
        Two corrections keep each thruster's positive thrust where ArduSub's Vectored frame puts it (AP_Motors6DOF.cpp, SUB_FRAME_VECTORED). The four horizontals are turned 90 degrees about z from the assembly, so +x lies along ArduSub's direction for that motor (1 aft starboard, 2 aft port, 3 fore starboard, 4 fore port); in the assembly they face the other diagonal, which is open with the modeler. The two verticals face up in the assembly, so their prop slots spin the occupant about -1 0 0 and positive thrust pushes down, as ArduSub's throttle factor of -1 expects.
-       The camera, sonar, dvl, gripper, payload and rack positions, the inertial origin and the collisions predate the assembly; they are refit in a later increment.
+       The camera, sonar, dvl, gripper, payload and rack positions and the inertial origin predate the assembly. The collisions were checked against the new chassis in Gazebo. Accessory visuals are out of scope: the camera, sonar and dvl parts carry no visual and work from their frames, and the gripper (subsea manipulation) is not yet in scope.
        The imu frame is where the flight controller senses attitude. Declared
        as a frame rather than a part because nothing about its mass or

File: bluerobotics_parts/urdf/dvl_a50.urdf.xacro (robot description, xacro)
@@ -2,7 +2,5 @@
 <!--
   dvl_a50 part macro: a Water Linked DVL A50 doppler velocity log.
-  Ported from the BlueROV2 accessory macros; a sized cylinder placeholder until a
-  real mesh is delivered. Visual only, like the accessory it replaces (the
-  chassis carries the vehicle's contact geometry).
+  Ported from the BlueROV2 accessory macros. No visual: accessory visuals are out of scope until a glTF part is commissioned, so the part is its link, inertia and frame, and bluerov2_gazebo hangs the sensor on that frame. Mass and inertia are a cylinder over the device envelope; the chassis carries the vehicle's contact geometry.
   Contract (see parts.xacro): <part>_info exports the metadata (attach,
   slots, frames, drive); <part> instantiates the link, its mounting joint
@@ -31,8 +29,4 @@
                  izz="${_m/2.0 * _r**2}"/>
       </inertial>
-      <visual>
-        <geometry><cylinder radius="${_r}" length="${_l}"/></geometry>
-        <material name="${name}_mat"><color rgba="0.5 0.5 0.55 1"/></material>
-      </visual>
     </link>
     <xacro:part_joint name="${name}" parent="${parent}" xyz="${xyz}" rpy="${rpy}"

File: bluerobotics_parts/urdf/explorehd_camera.urdf.xacro (robot description, xacro)
@@ -2,7 +2,5 @@
 <!--
   explorehd_camera part macro: a DWE exploreHD underwater camera.
-  Ported from the BlueROV2 accessory macros; a sized cylinder placeholder until a
-  real mesh is delivered. Visual only, like the accessory it replaces (the
-  chassis carries the vehicle's contact geometry).
+  Ported from the BlueROV2 accessory macros. No visual: accessory visuals are out of scope until a glTF part is commissioned, so the part is its link, inertia and frame, and bluerov2_gazebo hangs the sensor on that frame. Mass and inertia are a cylinder over the device envelope; the chassis carries the vehicle's contact geometry.
   Contract (see parts.xacro): <part>_info exports the metadata (attach,
   slots, frames, drive); <part> instantiates the link, its mounting joint
@@ -31,11 +29,4 @@
                  izz="${_m/2.0 * _r**2}"/>
       </inertial>
-      <visual>
-        <!-- The cylinder primitive's axis is z; the camera points along +x
-             (the sensing direction), so lay the visual on its side. -->
-        <origin xyz="0 0 0" rpy="0 1.5708 0"/>
-        <geometry><cylinder radius="${_r}" length="${_l}"/></geometry>
-        <material name="${name}_mat"><color rgba="0.5 0.5 0.55 1"/></material>
-      </visual>
     </link>
     <xacro:part_joint name="${name}" parent="${parent}" xyz="${xyz}" rpy="${rpy}"

File: bluerobotics_parts/urdf/ping360.urdf.xacro (robot description, xacro)
@@ -2,8 +2,5 @@
 <!--
   ping360 part macro: a Blue Robotics Ping360 scanning imaging sonar.
-  Mesh reused from CentraleNantes (Apache 2.0), ~100x oversized as authored
-  (no COLLADA unit element); the 0.01 scale matches upstream usage. Visual
-  only, like the accessory it replaces. Simulated as a planar gpu_lidar
-  (geometry/range, no acoustics) by bluerov2_gazebo.
+  No visual: accessory visuals are out of scope until a glTF part is commissioned, so the part is its link, inertia and frame, and bluerov2_gazebo hangs the sensor on that frame. Simulated as a planar gpu_lidar (geometry/range, no acoustics) by bluerov2_gazebo. The earlier visual, models/ping360/ping360.dae from CentraleNantes (Apache 2.0), stays in the package but is not used.
   Contract (see parts.xacro): <part>_info exports the metadata (attach,
   slots, frames, drive); <part> instantiates the link, its mounting joint
@@ -31,10 +28,4 @@
                  izz="${_m/2.0 * 0.038**2}"/>
       </inertial>
-      <visual>
-        <geometry>
-          <mesh filename="package://bluerobotics_parts/models/ping360/ping360.dae"
-                scale="0.01 0.01 0.01"/>
-        </geometry>
-      </visual>
     </link>
     <xacro:part_joint name="${name}" parent="${parent}" xyz="${xyz}" rpy="${rpy}"
