Commit message: Make the part meshes spec compliant Y-up glTF and merge a Gazebo flavoured URDF that pre-rotates them
Assisted-by: Claude Fable 5 <noreply@anthropic.com>
Signed-off-by: Carlos Agüero <caguero@honurobotics.com>

File: blueboat_gazebo/model.sdf.xacro (robot description, xacro)
@@ -17,8 +17,9 @@
              default="$(find blueboat_description)/config/blueboat.yaml"/>
   <xacro:property name="cfg" value="${xacro.load_yaml('$(arg config_file)')}"/>
-  <!-- The URDF to merge: the installed default, or (configure_vehicle.py,
-       launch time loadouts) a file:// URI of a URDF generated from the same
-       config. -->
-  <xacro:arg name="urdf_uri" default="package://blueboat_description/urdf/blueboat.urdf"/>
+  <!-- The URDF to merge: the Gazebo flavoured expansion (gltf_up:=z, glTF
+       visuals pre-rotated because Gazebo does not convert the glTF up axis)
+       installed next to this model, or (configure_vehicle.py, launch time
+       loadouts) a file:// URI of one generated from the same config. -->
+  <xacro:arg name="urdf_uri" default="model://blueboat/blueboat.urdf"/>
   <!-- Topic namespace for sensor topics: /<topic_namespace>/<part name>/...
        Per part, `gz_topic` / `topic` override the gz-side base (the bridge

File: bluerobotics_parts/urdf/basestation_antenna.urdf.xacro (robot description, xacro)
@@ -30,10 +30,5 @@
                  izz="0.00173301"/>
       </inertial>
-      <visual>
-        <origin xyz="0 0 0" rpy="0 0 0"/>
-        <geometry>
-          <mesh filename="package://bluerobotics_parts/models/basestation_antenna/basestation_antenna.visual.glb"/>
-        </geometry>
-      </visual>
+      <xacro:part_visual mesh="package://bluerobotics_parts/models/basestation_antenna/basestation_antenna.visual.glb"/>
       <xacro:if value="${collision}">
         <collision>

File: bluerobotics_parts/urdf/blueboat_antenna_mast.urdf.xacro (robot description, xacro)
@@ -30,10 +30,5 @@
                  izz="1.85026e-05"/>
       </inertial>
-      <visual>
-        <origin xyz="0 0 0" rpy="0 0 0"/>
-        <geometry>
-          <mesh filename="package://bluerobotics_parts/models/blueboat_antenna_mast/blueboat_antenna_mast.visual.glb"/>
-        </geometry>
-      </visual>
+      <xacro:part_visual mesh="package://bluerobotics_parts/models/blueboat_antenna_mast/blueboat_antenna_mast.visual.glb"/>
       <xacro:if value="${collision}">
         <collision>

File: bluerobotics_parts/urdf/blueboat_chassis.urdf.xacro (robot description, xacro)
@@ -43,10 +43,5 @@
                  izz="2.53089"/>
       </inertial>
-      <visual>
-        <origin xyz="0 0 0" rpy="0 0 0"/>
-        <geometry>
-          <mesh filename="package://bluerobotics_parts/models/blueboat_chassis/blueboat_chassis.visual.glb"/>
-        </geometry>
-      </visual>
+      <xacro:part_visual mesh="package://bluerobotics_parts/models/blueboat_chassis/blueboat_chassis.visual.glb"/>
       <xacro:if value="${collision}">
         <collision>

File: bluerobotics_parts/urdf/blueboat_flag.urdf.xacro (robot description, xacro)
@@ -30,10 +30,5 @@
                  izz="7.53318e-08"/>
       </inertial>
-      <visual>
-        <origin xyz="0 0 0" rpy="0 0 0"/>
-        <geometry>
-          <mesh filename="package://bluerobotics_parts/models/blueboat_flag/blueboat_flag.visual.glb"/>
-        </geometry>
-      </visual>
+      <xacro:part_visual mesh="package://bluerobotics_parts/models/blueboat_flag/blueboat_flag.visual.glb"/>
       <xacro:if value="${collision}">
         <collision>

File: bluerobotics_parts/urdf/blueboat_payload_bracket.urdf.xacro (robot description, xacro)
@@ -30,10 +30,5 @@
                  izz="0.000415846"/>
       </inertial>
-      <visual>
-        <origin xyz="0 0 0" rpy="0 0 0"/>
-        <geometry>
-          <mesh filename="package://bluerobotics_parts/models/blueboat_payload_bracket/blueboat_payload_bracket.visual.glb"/>
-        </geometry>
-      </visual>
+      <xacro:part_visual mesh="package://bluerobotics_parts/models/blueboat_payload_bracket/blueboat_payload_bracket.visual.glb"/>
       <xacro:if value="${collision}">
         <collision>

File: bluerobotics_parts/urdf/blueboat_ping_singlebeam_mount.urdf.xacro (robot description, xacro)
@@ -33,10 +33,5 @@
                  izz="0.000301922"/>
       </inertial>
-      <visual>
-        <origin xyz="0 0 0" rpy="0 0 0"/>
-        <geometry>
-          <mesh filename="package://bluerobotics_parts/models/blueboat_ping_singlebeam_mount/blueboat_ping_singlebeam_mount.visual.glb"/>
-        </geometry>
-      </visual>
+      <xacro:part_visual mesh="package://bluerobotics_parts/models/blueboat_ping_singlebeam_mount/blueboat_ping_singlebeam_mount.visual.glb"/>
       <xacro:if value="${collision}">
         <collision>

File: bluerobotics_parts/urdf/m200_weedless_prop_ccw.urdf.xacro (robot description, xacro)
@@ -30,10 +30,5 @@
                  izz="3.11438e-05"/>
       </inertial>
-      <visual>
-        <origin xyz="0 0 0" rpy="0 0 0"/>
-        <geometry>
-          <mesh filename="package://bluerobotics_parts/models/m200_weedless_prop_ccw/m200_weedless_prop_ccw.visual.glb"/>
-        </geometry>
-      </visual>
+      <xacro:part_visual mesh="package://bluerobotics_parts/models/m200_weedless_prop_ccw/m200_weedless_prop_ccw.visual.glb"/>
       <xacro:if value="${collision}">
         <collision>

File: bluerobotics_parts/urdf/m200_weedless_prop_cw.urdf.xacro (robot description, xacro)
@@ -30,10 +30,5 @@
                  izz="3.11438e-05"/>
       </inertial>
-      <visual>
-        <origin xyz="0 0 0" rpy="0 0 0"/>
-        <geometry>
-          <mesh filename="package://bluerobotics_parts/models/m200_weedless_prop_cw/m200_weedless_prop_cw.visual.glb"/>
-        </geometry>
-      </visual>
+      <xacro:part_visual mesh="package://bluerobotics_parts/models/m200_weedless_prop_cw/m200_weedless_prop_cw.visual.glb"/>
       <xacro:if value="${collision}">
         <collision>

File: bluerobotics_parts/urdf/omniscan_450_sidescan.urdf.xacro (robot description, xacro)
@@ -30,10 +30,5 @@
                  izz="0.00378588"/>
       </inertial>
-      <visual>
-        <origin xyz="0 0 0" rpy="0 0 0"/>
-        <geometry>
-          <mesh filename="package://bluerobotics_parts/models/omniscan_450_sidescan/omniscan_450_sidescan.visual.glb"/>
-        </geometry>
-      </visual>
+      <xacro:part_visual mesh="package://bluerobotics_parts/models/omniscan_450_sidescan/omniscan_450_sidescan.visual.glb"/>
       <xacro:if value="${collision}">
         <collision>

File: bluerobotics_parts/urdf/parts.xacro (robot description, xacro)
@@ -30,6 +30,6 @@
          joint      fixed (default), or continuous / revolute for parts that spin
          axis       joint axis in the part frame, used when joint is not fixed
-     and emitting one link (inertia, visual, optional collision), the
-     mounting joint (part_joint), and its slots and frames as massless links
+     and emitting one link (inertia, visual via part_visual, optional
+     collision), the mounting joint (part_joint), and its slots and frames as massless links
      named <name>_<slot> / <name>_<frame> (part_slots, part_frames). They
      show up in TF and are lumped away in Gazebo, where they survive as
@@ -42,4 +42,20 @@
 <robot xmlns:xacro="http://ros.org/wiki/xacro">
   <!-- ===== helpers used by every part macro ===== -->
+  <!-- glTF meshes are Y-up by specification and the delivered .glb files
+       conform. RViz and other ROS tools rotate them to Z-up on load; Gazebo
+       does not (it shows the data as is), so the URDF Gazebo merges is
+       expanded with gltf_up:=z, which pre-rotates every glTF visual by +90
+       degrees about x. The installed ROS URDF keeps gltf_up=y (no rotation). -->
+  <xacro:arg name="gltf_up" default="y"/>
+  <xacro:property name="gltf_visual_rpy" value="${'1.5708 0 0' if '$(arg gltf_up)' == 'z' else '0 0 0'}"/>
+  <!-- A part's visual mesh, with the glTF up axis handling above. -->
+  <xacro:macro name="part_visual" params="mesh xyz:='0 0 0'">
+    <visual>
+      <origin xyz="${xyz}" rpy="${gltf_visual_rpy}"/>
+      <geometry>
+        <mesh filename="${mesh}"/>
+      </geometry>
+    </visual>
+  </xacro:macro>
   <!-- The mounting joint. attach is the bolt on point in the part frame:
        the child frame is placed at xyz/rpy minus the rotated attach offset,

File: bluerobotics_parts/urdf/ping_singlebeam.urdf.xacro (robot description, xacro)
@@ -32,10 +32,5 @@
                  izz="2.02698e-05"/>
       </inertial>
-      <visual>
-        <origin xyz="0 0 0" rpy="0 0 0"/>
-        <geometry>
-          <mesh filename="package://bluerobotics_parts/models/ping_singlebeam/ping_singlebeam.visual.glb"/>
-        </geometry>
-      </visual>
+      <xacro:part_visual mesh="package://bluerobotics_parts/models/ping_singlebeam/ping_singlebeam.visual.glb"/>
       <xacro:if value="${collision}">
         <collision>

File: bluerobotics_parts/urdf/surveyor_multibeam.urdf.xacro (robot description, xacro)
@@ -30,10 +30,5 @@
                  izz="0.00170839"/>
       </inertial>
-      <visual>
-        <origin xyz="0 0 0" rpy="0 0 0"/>
-        <geometry>
-          <mesh filename="package://bluerobotics_parts/models/surveyor_multibeam/surveyor_multibeam.visual.glb"/>
-        </geometry>
-      </visual>
+      <xacro:part_visual mesh="package://bluerobotics_parts/models/surveyor_multibeam/surveyor_multibeam.visual.glb"/>
       <xacro:if value="${collision}">
         <collision>

File: bluerobotics_parts/urdf/t200_prop_ccw.urdf.xacro (robot description, xacro)
@@ -30,10 +30,5 @@
                  izz="7.07841e-06"/>
       </inertial>
-      <visual>
-        <origin xyz="0 0 0" rpy="0 0 0"/>
-        <geometry>
-          <mesh filename="package://bluerobotics_parts/models/t200_prop_ccw/t200_prop_ccw.visual.glb"/>
-        </geometry>
-      </visual>
+      <xacro:part_visual mesh="package://bluerobotics_parts/models/t200_prop_ccw/t200_prop_ccw.visual.glb"/>
       <xacro:if value="${collision}">
         <collision>

File: bluerobotics_parts/urdf/t200_prop_cw.urdf.xacro (robot description, xacro)
@@ -30,10 +30,5 @@
                  izz="7.07841e-06"/>
       </inertial>
-      <visual>
-        <origin xyz="0 0 0" rpy="0 0 0"/>
-        <geometry>
-          <mesh filename="package://bluerobotics_parts/models/t200_prop_cw/t200_prop_cw.visual.glb"/>
-        </geometry>
-      </visual>
+      <xacro:part_visual mesh="package://bluerobotics_parts/models/t200_prop_cw/t200_prop_cw.visual.glb"/>
       <xacro:if value="${collision}">
         <collision>

File: bluerobotics_parts/urdf/t200_thruster.urdf.xacro (robot description, xacro)
@@ -30,10 +30,5 @@
                  izz="0.000291503"/>
       </inertial>
-      <visual>
-        <origin xyz="0 0 0" rpy="0 0 0"/>
-        <geometry>
-          <mesh filename="package://bluerobotics_parts/models/t200_thruster/t200_thruster.visual.glb"/>
-        </geometry>
-      </visual>
+      <xacro:part_visual mesh="package://bluerobotics_parts/models/t200_thruster/t200_thruster.visual.glb"/>
       <xacro:if value="${collision}">
         <collision>
