Commit message: Fix the generation audit findings: of: instead of the YAML boolean on:, config driven thrusters, manifest backed config check, base name plumbing, no dead axis metadata
Assisted-by: Claude Fable 5 <noreply@anthropic.com>
Signed-off-by: Carlos Agüero <caguero@honurobotics.com>

File: blueboat_gazebo/model.sdf.xacro (robot description, xacro)
@@ -4,6 +4,7 @@
   time. It merge-includes the blueboat_description geometry (assembled from
   bluerobotics_parts) and adds the Gazebo plugins: hydrodynamics, one Thruster
-  per outboard motor, and one <sensor> per sensor part. Buoyancy is a world plugin (graded, in the playground
-  world), not here.
+  per propeller part, one <sensor> per sensor part, both placed by the same
+  assembly resolution the URDF went through. Buoyancy is a world plugin
+  (graded, in the playground world), not here.
   In a world:  <include><uri>model://blueboat</uri></include>
 -->
@@ -11,6 +12,7 @@
      xmlns:gz="http://gazebosim.org/schema">
   <!-- The assembly dispatcher, run here with Gazebo side emitters: the same
-       resolution of slots and defaults the URDF went through, emitting one
-       <sensor> per sensor part instead of links. -->
+       resolution of slots and defaults the URDF went through, emitting a
+       <sensor> per sensor part and a Thruster per propeller instead of
+       links. -->
   <xacro:include filename="$(find bluerobotics_parts)/urdf/assembly.xacro"/>
   <xacro:arg name="config_file"
@@ -22,36 +24,43 @@
        loadouts) a file:// URI of one generated from the same config. -->
   <xacro:arg name="urdf_uri" default="model://blueboat/blueboat.urdf"/>
-  <!-- Topic namespace for sensor topics: /<topic_namespace>/<part name>/...
-       Per part, `gz_topic` / `topic` override the gz-side base (the bridge
-       config is generated from the same yaml, so gz and ROS sides stay in sync). -->
+  <!-- Topic namespace: every part topic is /<topic_namespace>/<part name>/...
+       on both sides (a propeller's /thrust, the Ping's /range). Per part,
+       `gz_topic` / `topic` override the gz side base; the bridge config is
+       generated from the same yaml, so gz and ROS sides stay in sync. -->
   <xacro:property name="topic_ns" value="${cfg.get('topic_namespace', 'blueboat')}"/>
-  <!-- T200 thrust saturation (same motors as the BlueROV2), 16 V full-throttle
-       endpoints; tune per bus voltage. Curve/datasheet:
-       https://bluerobotics.com/store/rov/bluerov2-components-spares/t200-thruster-brov2-spare-r1-vp/ -->
-  <xacro:property name="t200_max_thrust" value="51.5"/>   <!-- N, forward -->
-  <xacro:property name="t200_min_thrust" value="-40.2"/>  <!-- N, reverse -->
-  <!-- One Thruster plugin per outboard motor. Twin-screw differential drive: the
-       props counter-rotate (opposite coeff sign) so their reaction yaw cancels in
-       straight-line running. Command thrust (N) on
-       /model/blueboat/joint/motor_<side>_joint/cmd_thrust. -->
-  <xacro:macro name="thruster" params="side coeff">
-    <!-- No <namespace>: the plugin defaults to the model name, so the command
-         topics track the instance name. NOTE: the shipped bridge config and the
-         playground world's buoyancy <enable> still bake the default instance
-         name (blueboat); per instance parameterization is the multi vehicle
-         PR. -->
+  <!-- The root link the assembly names (the config's base.name). -->
+  <xacro:property name="base_name" value="${cfg['base'].get('name', 'base_link')}"/>
+  <!-- Config entry that fitted an instance, or {} (slot entries default their
+       name to the slot). -->
+  <xacro:macro name="part_entry" params="name">
+    <xacro:property name="ovr"
+                    value="${[e for e in (cfg.get('parts') or []) if e.get('name', e.get('slot')) == name]}"/>
+    <xacro:property name="entry" scope="parent" value="${ovr[0] if ovr else dict()}"/>
+  </xacro:macro>
+  <!-- A propeller part drives its mounting joint: one Thruster plugin per
+       propeller instance, with the limits and diameter the part declares in
+       its `drive` table. Counter rotating pairs (ccw to port, cw to
+       starboard in the default loadout) get opposite coefficient signs so
+       their reaction yaw cancels in straight line running. Thrust commands
+       (N) on <topic_base>/thrust, speed feedback on <topic_base>/thrust/ang_vel:
+       the plugin prefixes a custom <topic> with its <namespace> (the model
+       name unless given), so the namespace is emptied and the topic follows
+       the config like every other part topic, not the spawn name. -->
+  <xacro:macro name="thruster" params="name drive topic_base">
     <plugin filename="gz-sim-thruster-system" name="gz::sim::systems::Thruster">
-      <joint_name>motor_${side}_joint</joint_name>
-      <thrust_coefficient>${coeff}</thrust_coefficient>
+      <joint_name>${name}_joint</joint_name>
+      <namespace></namespace>
+      <topic>${topic_base}/thrust</topic>
+      <thrust_coefficient>${0.02 if drive['rotation'] == 'ccw' else -0.02}</thrust_coefficient>
       <fluid_density>1025.0</fluid_density>
-      <propeller_diameter>0.076</propeller_diameter>  <!-- T200 prop -->
+      <propeller_diameter>${drive['diameter']}</propeller_diameter>
       <velocity_control>true</velocity_control>
-      <max_thrust_cmd>${t200_max_thrust}</max_thrust_cmd>
-      <min_thrust_cmd>${t200_min_thrust}</min_thrust_cmd>
+      <max_thrust_cmd>${drive['max_thrust']}</max_thrust_cmd>
+      <min_thrust_cmd>${drive['min_thrust']}</min_thrust_cmd>
     </plugin>
   </xacro:macro>
   <!-- ===================== Sensors (config-driven) =====================
-       One <sensor> per sensor part, as a massless link fixed to base_link at
-       the part's frame (keeps the description Gazebo-free). Needs
+       One <sensor> per sensor part, as a massless link fixed to the root link
+       at the part's frame (keeps the description Gazebo-free). Needs
        gz-sim-sensors-system in the world (GPU). The two imaging sonars
        (omniscan_450 side-scan, surveyor_multibeam) are PARKED - no acoustic model
@@ -61,6 +70,6 @@
       <!-- Posed at the frame the part declares for its sensing origin (its
            `beam`, `lens`, ...): the URDF conversion lumps the part into
-           base_link but keeps every frame by name, so the sensor follows the
-           part wherever the config mounted it. -->
+           the root link but keeps every frame by name, so the sensor follows
+           the part wherever the config mounted it. -->
       <pose relative_to="${frame}">0 0 0 0 0 0</pose>
       <inertial>
@@ -74,5 +83,5 @@
     </link>
     <joint name="${name}_sensor_joint" type="fixed">
-      <parent>base_link</parent>
+      <parent>${base_name}</parent>
       <child>${name}_sensor</child>
     </joint>
@@ -104,16 +113,21 @@
     </xacro:sensor_link>
   </xacro:macro>
-  <!-- Emitters for the assembly dispatcher. Per resolved part instance:
+  <!-- Emitters for the assembly dispatcher. Per resolved part instance: a
+       propeller (a part with a `drive` table) gets a Thruster on its joint,
        the Ping2 echosounder gets its sensor, every other part is geometry
        only and emits nothing here. Topic overrides come from the config
-       entry that fitted the instance (slot entries default their name to
-       the slot). Ad hoc slots are URDF frames; nothing to emit. -->
-  <xacro:macro name="gz_part" params="ptype name parent xyz rpy collision joint axis">
+       entry that fitted the instance. Ad hoc slots are URDF frames; nothing
+       to emit. -->
+  <xacro:macro name="gz_part" params="ptype name parent xyz rpy collision joint axis info">
+    <xacro:part_entry name="${name}"/>
+    <xacro:property name="topic_base"
+                    value="${entry.get('gz_topic', entry.get('topic', topic_ns + '/' + name))}"/>
+    <!-- A propeller on a fixed joint (a spare, say) is lumped away and
+         drives nothing. -->
+    <xacro:if value="${'drive' in info and joint != 'fixed'}">
+      <xacro:thruster name="${name}" drive="${info['drive']}" topic_base="${topic_base}"/>
+    </xacro:if>
     <xacro:if value="${ptype == 'ping_singlebeam'}">
-      <xacro:property name="ovr"
-                      value="${[e for e in (cfg.get('parts') or []) if e.get('name', e.get('slot')) == name]}"/>
-      <xacro:property name="o" value="${ovr[0] if ovr else dict()}"/>
-      <xacro:echosounder_sensor name="${name}" frame="${name}_beam"
-                                topic_base="${o.get('gz_topic', o.get('topic', topic_ns + '/' + name))}"/>
+      <xacro:echosounder_sensor name="${name}" frame="${name}_beam" topic_base="${topic_base}"/>
     </xacro:if>
   </xacro:macro>
@@ -128,5 +142,5 @@
        hubs). Segmented so each box responds to its own local depth and a
        pitched waterplane restores properly. The boxes also give contact.
-       Fixed jointed to base_link: physics sees one rigid body. -->
+       Fixed jointed to the root link: physics sees one rigid body. -->
   <xacro:macro name="pontoon" params="hull side y n i:=0">
     <xacro:if value="${i != n}">
@@ -143,5 +157,5 @@
   <xacro:macro name="hull_displacement" params="hull">
     <link name="hull_displacement">
-      <pose relative_to="base_link">0 0 0 0 0 0</pose>
+      <pose relative_to="${base_name}">0 0 0 0 0 0</pose>
       <inertial>
         <mass>1e-5</mass>
@@ -155,5 +169,5 @@
     </link>
     <joint name="hull_displacement_joint" type="fixed">
-      <parent>base_link</parent>
+      <parent>${base_name}</parent>
       <child>hull_displacement</child>
     </joint>
@@ -172,5 +186,5 @@
     <plugin filename="gz-sim-hydrodynamics-system"
             name="gz::sim::systems::Hydrodynamics">
-      <link_name>base_link</link_name>
+      <link_name>${base_name}</link_name>
       <water_density>1025.0</water_density>
       <xU>-20</xU>    <yV>-40</yV>    <zW>-30</zW>
@@ -183,5 +197,5 @@
       <nRabsR>-30</nRabsR>
     </plugin>
-    <!-- Joint states for the motor joints, so robot_state_publisher can
+    <!-- Joint states for the propeller joints, so robot_state_publisher can
          animate the props in RViz. Bridged to /joint_states. -->
     <plugin filename="gz-sim-joint-state-publisher-system"
@@ -189,10 +203,9 @@
       <topic>${topic_ns}/joint_states</topic>
     </plugin>
-    <!-- Twin outboards (counter-rotating). -->
-    <xacro:thruster side="port" coeff="0.02"/>
-    <xacro:thruster side="stbd" coeff="-0.02"/>
-    <!-- Sensors: one per sensor part the assembly resolves to. -->
+    <!-- Thrusters and sensors: one per propeller / sensor part the
+         assembly resolves to. No manifest: that lives in the merged URDF. -->
     <xacro:assemble base="${cfg['base']}" parts="${cfg.get('parts') or []}"
-                    slots="${cfg.get('slots') or []}" emit="gz_part" emit_slot="gz_no_slot"/>
+                    slots="${cfg.get('slots') or []}" emit="gz_part" emit_slot="gz_no_slot"
+                    manifest="false"/>
   </model>
 </sdf>

File: bluerobotics_parts/urdf/assembly.xacro (robot description, xacro)
@@ -13,8 +13,8 @@
         - {slot: ping_mount, type: none}                   # leave a slot empty
         - {slot: mast, type: blueboat_antenna_mast}        # fill a slot that has no default
-        - {slot: ping, on: ping_mount, type: ping_singlebeam, topic: sonar}   # a slot on another part
+        - {slot: ping, of: ping_mount, type: ping_singlebeam, topic: sonar}   # a slot of another part
         - {type: explorehd_camera, name: cam, xyz: "0.3 0 0.2", rpy: "0 0 0"}  # free placement
       slots:
-        - {on: base_link, name: gopro, xyz: "0.45 0 0.2", accepts: [explorehd_camera]}
+        - {of: base_link, name: gopro, xyz: "0.45 0 0.2", accepts: [explorehd_camera]}
   How it resolves:
   * The base part is the root (its link is the named root link, no joint).
@@ -23,22 +23,34 @@
     has an entry for that slot: `type:` picks another option (it must be in
     the slot's accepts list), `type: none` leaves it empty. An entry names
-    the slot, and `on:` the instance carrying it (default: the base). The
-    occupant's instance name defaults to the slot name.
+    the slot, and `of:` the instance carrying it (default: the base). The
+    occupant's instance name defaults to the slot name. (The key is `of`,
+    not `on`: a bare `on` is a YAML boolean and would read as `true`.)
   * Entries without slot: are free placements: type, name, xyz/rpy relative
     to parent (default: the base). Their slots fill too.
+  * The occupant's joint is the entry's `joint:`, else the slot's, else the
+    part's nature: a propeller (a part with a `drive` table) turns on a
+    continuous joint, anything else is fixed.
   * `slots:` declares ad hoc slots on any instance, usable like the part's
     own (accepts and default work the same).
-  * Mistakes fail the expansion loudly: an unknown slot on the base, a type
-    a slot does not accept, or a slot configured twice. An unknown part type
-    fails as "unknown macro name".
-  Every instance is also recorded as <assembly_part type name parent/>, a
-  URDF extension element urdfdom and Gazebo ignore, so tooling downstream
-  (the Gazebo composition, the bridge generator) knows the resolved parts
-  list without re-resolving anything.
+  * Mistakes the expansion can see fail it loudly: an unknown slot on the
+    base, a type a slot does not accept, a slot configured twice, a bare
+    `on:` key. An unknown part type fails as "unknown macro name". What
+    xacro cannot see across the recursion (an entry or ad hoc slot whose
+    `of:` or `slot:` matches nothing deeper down, two instances with the
+    same name, an unknown key) is caught by bluerobotics_parts.assembly.check
+    from the manifest below; the vehicle builds and launches run it.
+  The manifest: every instance is recorded as <assembly_part type name
+  parent/> and every slot visited as <assembly_slot of name/>, URDF
+  extension elements urdfdom and Gazebo ignore, so tooling downstream (the
+  Gazebo composition, the bridge generator, the config check) knows the
+  resolved assembly without re-resolving anything. `manifest:=false` turns
+  the records off for outputs that are not URDF.
   The emitter is pluggable: `emit` names the macro called per instance
-  (default emit_part: the part macro plus the manifest element), `emit_slot`
-  the one called per ad hoc slot (default part_slot). blueboat_gazebo runs
-  the same resolution with emitters that produce sensors, so the composed
-  model can never disagree with the URDF about which parts are fitted.
+  (default emit_part: the part macro), `emit_slot` the one called per ad hoc
+  slot (default part_slot). Emitters receive the part's `info` table, so a
+  simulator can place a sensor at a declared frame or drive a propeller.
+  blueboat_gazebo runs the same resolution with such emitters, so the
+  composed model can never disagree with the URDF about which parts are
+  fitted.
 -->
 <robot xmlns:xacro="http://ros.org/wiki/xacro">
@@ -55,7 +67,6 @@
     <xacro:property name="part_info" scope="parent" value="${part_info}"/>
   </xacro:macro>
-  <!-- Default emitter: manifest element plus the part macro itself. -->
-  <xacro:macro name="emit_part" params="ptype name parent xyz rpy collision joint axis">
-    <assembly_part type="${ptype}" name="${name}" parent="${parent}"/>
+  <!-- Default emitter: the part macro itself. -->
+  <xacro:macro name="emit_part" params="ptype name parent xyz rpy collision joint axis info">
     <xacro:if value="${axis == ''}">
       <xacro:call macro="${ptype}" name="${name}" parent="${parent}" xyz="${xyz}" rpy="${rpy}"
@@ -77,6 +88,9 @@
   <!-- One slot of one instance: config entry, else the slot default. -->
   <xacro:macro name="fill_slot" params="inst slot spec entries adhoc emit emit_slot">
+    <xacro:if value="${manifest}">
+      <assembly_slot of="${inst}" name="${slot}"/>
+    </xacro:if>
     <xacro:property name="matches"
-                    value="${[e for e in entries if e.get('slot') == slot and e.get('on', base_name) == inst]}"/>
+                    value="${[e for e in entries if e.get('slot') == slot and e.get('of', base_name) == inst]}"/>
     <xacro:if value="${len(matches) > 1}">
       <xacro:assembly_fail message="slot '${slot}' of '${inst}' is configured ${len(matches)} times"/>
@@ -91,5 +105,5 @@
                         xyz="${entry.get('xyz', '0 0 0')}" rpy="${entry.get('rpy', '0 0 0')}"
                         collision="${entry.get('collision', True)}"
-                        joint="${entry.get('joint', spec.get('joint', 'fixed'))}"
+                        joint="${entry.get('joint', spec.get('joint', ''))}"
                         axis="${entry.get('axis', '')}"
                         entries="${entries}" adhoc="${adhoc}" emit="${emit}" emit_slot="${emit_slot}"/>
@@ -105,11 +119,18 @@
   </xacro:macro>
   <!-- Instantiate a part, then its slots: the part's own and the ad hoc
-       ones the config put on this instance. -->
+       ones the config put on this instance. joint "" means unspecified by
+       the entry and the slot: a part that drives (a propeller) then turns
+       on a continuous joint, anything else is fixed. -->
   <xacro:macro name="place_part"
                params="ptype name parent xyz rpy collision joint axis entries adhoc emit emit_slot">
     <xacro:part_info_of ptype="${ptype}"/>
+    <xacro:property name="joint_type"
+                    value="${joint if joint != '' else ('continuous' if 'drive' in part_info else 'fixed')}"/>
+    <xacro:if value="${manifest}">
+      <assembly_part type="${ptype}" name="${name}" parent="${parent}"/>
+    </xacro:if>
     <xacro:call macro="${emit}" ptype="${ptype}" name="${name}" parent="${parent}" xyz="${xyz}" rpy="${rpy}"
-                collision="${collision}" joint="${joint}" axis="${axis}"/>
-    <xacro:property name="mine" value="${[s for s in adhoc if s.get('on', base_name) == name]}"/>
+                collision="${collision}" joint="${joint_type}" axis="${axis}" info="${part_info}"/>
+    <xacro:property name="mine" value="${[s for s in adhoc if s.get('of', base_name) == name]}"/>
     <xacro:adhoc_slots inst="${name}" items="${mine}" emit_slot="${emit_slot}"/>
     <xacro:fill_slots inst="${name}"
@@ -127,5 +148,5 @@
         <xacro:place_part ptype="${it['type']}" name="${it['name']}" parent="${it.get('parent', base_name)}"
                           xyz="${it['xyz']}" rpy="${it.get('rpy', '0 0 0')}"
-                          collision="${it.get('collision', True)}" joint="${it.get('joint', 'fixed')}"
+                          collision="${it.get('collision', True)}" joint="${it.get('joint', '')}"
                           axis="${it.get('axis', '')}"
                           entries="${entries}" adhoc="${adhoc}" emit="${emit}" emit_slot="${emit_slot}"/>
@@ -139,5 +160,5 @@
   <xacro:macro name="check_base_slots" params="items known">
     <xacro:if value="${len(items) > 0}">
-      <xacro:if value="${items[0].get('on', base_name) == base_name and items[0]['slot'] not in known}">
+      <xacro:if value="${items[0].get('of', base_name) == base_name and items[0]['slot'] not in known}">
         <xacro:assembly_fail message="unknown slot '${items[0]['slot']}' on '${base_name}' (known: ${known})"/>
       </xacro:if>
@@ -145,12 +166,17 @@
     </xacro:if>
   </xacro:macro>
-  <xacro:macro name="assemble" params="base parts slots:='' emit:=emit_part emit_slot:=part_slot">
+  <xacro:macro name="assemble"
+               params="base parts slots:='' emit:=emit_part emit_slot:=part_slot manifest:=true">
     <xacro:property name="base_name" value="${base.get('name', 'base_link')}"/>
     <xacro:property name="adhoc" value="${slots if slots else []}"/>
+    <!-- A bare `on:` key parses as the YAML boolean true; the key is `of:`. -->
+    <xacro:if value="${len([e for e in list(parts) + list(adhoc) if True in e]) > 0}">
+      <xacro:assembly_fail message="an entry has a bare 'on:' key, which YAML reads as true; the key is 'of:'"/>
+    </xacro:if>
     <xacro:property name="slot_entries" value="${[p for p in parts if 'slot' in p]}"/>
     <xacro:property name="free_entries" value="${[p for p in parts if 'slot' not in p]}"/>
     <xacro:part_info_of ptype="${base['type']}"/>
     <xacro:check_base_slots items="${slot_entries}"
-                            known="${list(part_info['slots'].keys()) + [s['name'] for s in adhoc if s.get('on', base_name) == base_name]}"/>
+                            known="${list(part_info['slots'].keys()) + [s['name'] for s in adhoc if s.get('of', base_name) == base_name]}"/>
     <xacro:place_part ptype="${base['type']}" name="${base_name}" parent="" xyz="0 0 0" rpy="0 0 0"
                       collision="${base.get('collision', True)}" joint="fixed" axis=""

File: bluerobotics_parts/urdf/basestation_antenna.urdf.xacro (robot description, xacro)
@@ -6,5 +6,5 @@
   Inertia: estimated from the delivered collision geometry at 1000 kg/m^3 (SDF auto inertia); replace with measured values.
   Contract (see parts.xacro): <part>_info exports the metadata (attach,
-  axis, slots, frames); <part> instantiates the link, its mounting joint
+  slots, frames, drive); <part> instantiates the link, its mounting joint
   and its slot / frame links.
 -->
@@ -13,5 +13,4 @@
     <xacro:property name="part_info" scope="parent" value="${dict(
         attach='0 0 0',
-        axis='1 0 0',
         slots=dict(
         ),

File: bluerobotics_parts/urdf/blueboat_antenna_mast.urdf.xacro (robot description, xacro)
@@ -6,5 +6,5 @@
   Inertia: estimated from the delivered collision geometry at 1000 kg/m^3 (SDF auto inertia); replace with measured values.
   Contract (see parts.xacro): <part>_info exports the metadata (attach,
-  axis, slots, frames); <part> instantiates the link, its mounting joint
+  slots, frames, drive); <part> instantiates the link, its mounting joint
   and its slot / frame links.
 -->
@@ -13,5 +13,4 @@
     <xacro:property name="part_info" scope="parent" value="${dict(
         attach='0 0 -0.331',
-        axis='1 0 0',
         slots=dict(
         ),

File: bluerobotics_parts/urdf/blueboat_chassis.urdf.xacro (robot description, xacro)
@@ -6,5 +6,5 @@
   Inertia: tensor shape estimated from the collision geometry, scaled from 68.139 kg at 1000 kg/m^3 to the stated 12 kg.
   Contract (see parts.xacro): <part>_info exports the metadata (attach,
-  axis, slots, frames); <part> instantiates the link, its mounting joint
+  slots, frames, drive); <part> instantiates the link, its mounting joint
   and its slot / frame links.
   Slots other parts fit into, as frames <name>_<slot>:
@@ -20,5 +20,4 @@
     <xacro:property name="part_info" scope="parent" value="${dict(
         attach='0 0 0',
-        axis='1 0 0',
         slots=dict(
             motor_port=dict(xyz='-0.52 0.301 -0.117', rpy='0 0 0', accepts=['m200_weedless_prop_ccw', 't200_prop_ccw'], default='m200_weedless_prop_ccw', joint='continuous'),
