Commit message: Fix the generation audit findings: of: instead of the YAML boolean on:, config driven thrusters, manifest backed config check, base name plumbing, no dead axis metadata
Assisted-by: Claude Fable 5 <noreply@anthropic.com>
Signed-off-by: Carlos Agüero <caguero@honurobotics.com>

File: bluerobotics_parts/urdf/blueboat_flag.urdf.xacro (robot description, xacro)
@@ -6,5 +6,5 @@
   Inertia: estimated from the delivered collision geometry at 1000 kg/m^3 (SDF auto inertia); replace with measured values.
   Contract (see parts.xacro): <part>_info exports the metadata (attach,
-  axis, slots, frames); <part> instantiates the link, its mounting joint
+  slots, frames, drive); <part> instantiates the link, its mounting joint
   and its slot / frame links.
 -->
@@ -13,5 +13,4 @@
     <xacro:property name="part_info" scope="parent" value="${dict(
         attach='0 0 -0.515',
-        axis='1 0 0',
         slots=dict(
         ),

File: bluerobotics_parts/urdf/blueboat_payload_bracket.urdf.xacro (robot description, xacro)
@@ -6,5 +6,5 @@
   Inertia: estimated from the delivered collision geometry at 1000 kg/m^3 (SDF auto inertia); replace with measured values.
   Contract (see parts.xacro): <part>_info exports the metadata (attach,
-  axis, slots, frames); <part> instantiates the link, its mounting joint
+  slots, frames, drive); <part> instantiates the link, its mounting joint
   and its slot / frame links.
 -->
@@ -13,5 +13,4 @@
     <xacro:property name="part_info" scope="parent" value="${dict(
         attach='0 0 0',
-        axis='1 0 0',
         slots=dict(
         ),

File: bluerobotics_parts/urdf/blueboat_ping_singlebeam_mount.urdf.xacro (robot description, xacro)
@@ -6,5 +6,5 @@
   Inertia: estimated from the delivered collision geometry at 1000 kg/m^3 (SDF auto inertia); replace with measured values.
   Contract (see parts.xacro): <part>_info exports the metadata (attach,
-  axis, slots, frames); <part> instantiates the link, its mounting joint
+  slots, frames, drive); <part> instantiates the link, its mounting joint
   and its slot / frame links.
   Slots other parts fit into, as frames <name>_<slot>:
@@ -15,5 +15,4 @@
     <xacro:property name="part_info" scope="parent" value="${dict(
         attach='0 0 0',
-        axis='1 0 0',
         slots=dict(
             ping=dict(xyz='0 0 -0.01', rpy='0 0 0', accepts=['ping_singlebeam'], default='ping_singlebeam'),

File: bluerobotics_parts/urdf/m200_weedless_prop_ccw.urdf.xacro (robot description, xacro)
@@ -5,6 +5,8 @@
   2026-08-21. This file is the part: maintain it by hand from here on.
   Inertia: estimated from the delivered collision geometry at 1000 kg/m^3 (SDF auto inertia); replace with measured values.
+  Drive: T200 16 V endpoints and prop diameter as placeholders for every
+  propeller option; replace with measured values for this prop.
   Contract (see parts.xacro): <part>_info exports the metadata (attach,
-  axis, slots, frames); <part> instantiates the link, its mounting joint
+  slots, frames, drive); <part> instantiates the link, its mounting joint
   and its slot / frame links.
 -->
@@ -13,9 +15,9 @@
     <xacro:property name="part_info" scope="parent" value="${dict(
         attach='0 0 0',
-        axis='1 0 0',
         slots=dict(
         ),
         frames=dict(
-        ))}"/>
+        ),
+        drive=dict(diameter=0.076, max_thrust=51.5, min_thrust=-40.2, rotation='ccw'))}"/>
   </xacro:macro>
   <xacro:macro name="m200_weedless_prop_ccw"

File: bluerobotics_parts/urdf/m200_weedless_prop_cw.urdf.xacro (robot description, xacro)
@@ -5,6 +5,8 @@
   2026-08-21. This file is the part: maintain it by hand from here on.
   Inertia: estimated from the delivered collision geometry at 1000 kg/m^3 (SDF auto inertia); replace with measured values.
+  Drive: T200 16 V endpoints and prop diameter as placeholders for every
+  propeller option; replace with measured values for this prop.
   Contract (see parts.xacro): <part>_info exports the metadata (attach,
-  axis, slots, frames); <part> instantiates the link, its mounting joint
+  slots, frames, drive); <part> instantiates the link, its mounting joint
   and its slot / frame links.
 -->
@@ -13,9 +15,9 @@
     <xacro:property name="part_info" scope="parent" value="${dict(
         attach='0 0 0',
-        axis='1 0 0',
         slots=dict(
         ),
         frames=dict(
-        ))}"/>
+        ),
+        drive=dict(diameter=0.076, max_thrust=51.5, min_thrust=-40.2, rotation='cw'))}"/>
   </xacro:macro>
   <xacro:macro name="m200_weedless_prop_cw"

File: bluerobotics_parts/urdf/omniscan_450_sidescan.urdf.xacro (robot description, xacro)
@@ -6,5 +6,5 @@
   Inertia: estimated from the delivered collision geometry at 1000 kg/m^3 (SDF auto inertia); replace with measured values.
   Contract (see parts.xacro): <part>_info exports the metadata (attach,
-  axis, slots, frames); <part> instantiates the link, its mounting joint
+  slots, frames, drive); <part> instantiates the link, its mounting joint
   and its slot / frame links.
 -->
@@ -13,5 +13,4 @@
     <xacro:property name="part_info" scope="parent" value="${dict(
         attach='0 0 0',
-        axis='1 0 0',
         slots=dict(
         ),

File: bluerobotics_parts/urdf/part_probe.urdf.xacro (robot description, xacro)
@@ -8,5 +8,5 @@
   actually break: instantiating at all, two instances without a name collision,
   collision:=false, and a part parented to another part rather than to the
-  chassis. See "Accepting a new part" in the package README.
+  chassis. See the site: how-to/add-part.
 -->
 <robot name="part_probe" xmlns:xacro="http://ros.org/wiki/xacro">

File: bluerobotics_parts/urdf/parts.xacro (robot description, xacro)
@@ -14,5 +14,4 @@
          attach   where the part bolts onto its parent, "x y z" in the part
                   frame (the mounting joint folds it in)
-         axis     spin axis in the part frame, for parts that turn
          slots    named mount points other parts fit into, each with
                     xyz / rpy   pose in the part frame
@@ -23,4 +22,14 @@
          frames   named reference frames (a sensor's beam origin, a lens),
                   each with xyz / rpy
+         drive    propellers only: what a simulator needs to drive the part
+                  as a thruster on its mounting joint
+                    diameter    propeller diameter, m
+                    max_thrust  forward thrust limit, N
+                    min_thrust  reverse thrust limit, N (negative)
+                    rotation    'ccw' or 'cw', seen from behind looking
+                                forward along the spin axis
+     Simulators read `frames` and `drive` (blueboat_gazebo places a
+     <sensor> at a sensor part's frame and a Thruster on a propeller's
+     joint); the URDF itself only turns `frames` into links.
   2. <part>: the macro that instantiates it, taking exactly
          name       link name for this instance; the joint is <name>_joint
@@ -29,10 +38,11 @@
          collision  false to instantiate the part without contact geometry
          joint      fixed (default), or continuous / revolute for parts that spin
-         axis       joint axis in the part frame, used when joint is not fixed
+         axis       joint axis in the part frame, used when joint is not
+                    fixed; the macro's default is the part's own spin axis
      and emitting one link (inertia, visual via part_visual, optional
-     collision), the mounting joint (part_joint), and its slots and frames as massless links
-     named <name>_<slot> / <name>_<frame> (part_slots, part_frames). They
-     show up in TF and are lumped away in Gazebo, where they survive as
-     frames of the same name.
+     collision), the mounting joint (part_joint), and its slots and frames as
+     massless links named <name>_<slot> / <name>_<frame> (part_slots,
+     part_frames). They show up in TF and are lumped away in Gazebo, where
+     they survive as frames of the same name.
   The URDF xacro is the part. It may be bootstrapped from a modeler's SDF
   with scripts/sdf_to_part.py or written by hand; nothing downstream knows
@@ -99,9 +109,6 @@
     </joint>
   </xacro:macro>
-  <xacro:macro name="part_frame" params="name parent xyz rpy:='0 0 0'">
-    <xacro:part_slot name="${name}" parent="${parent}" xyz="${xyz}" rpy="${rpy}"/>
-  </xacro:macro>
-  <!-- All of a part's slots / frames from its part_info tables (xacro has
-       no loop; recurse over list(table.items())). -->
+  <!-- All of a part's slots (or frames: same thing to the URDF) from its
+       part_info table (xacro has no loop; recurse over list(table.items())). -->
   <xacro:macro name="part_slots" params="name items">
     <xacro:if value="${len(items) > 0}">
@@ -112,9 +119,5 @@
   </xacro:macro>
   <xacro:macro name="part_frames" params="name items">
-    <xacro:if value="${len(items) > 0}">
-      <xacro:part_frame name="${name}_${items[0][0]}" parent="${name}"
-                        xyz="${items[0][1]['xyz']}" rpy="${items[0][1].get('rpy', '0 0 0')}"/>
-      <xacro:part_frames name="${name}" items="${items[1:]}"/>
-    </xacro:if>
+    <xacro:part_slots name="${name}" items="${items}"/>
   </xacro:macro>
   <!-- ===== catalog =====

File: bluerobotics_parts/urdf/ping_singlebeam.urdf.xacro (robot description, xacro)
@@ -6,5 +6,5 @@
   Inertia: estimated from the delivered collision geometry at 1000 kg/m^3 (SDF auto inertia); replace with measured values.
   Contract (see parts.xacro): <part>_info exports the metadata (attach,
-  axis, slots, frames); <part> instantiates the link, its mounting joint
+  slots, frames, drive); <part> instantiates the link, its mounting joint
   and its slot / frame links.
   Reference frames, as <name>_<frame>: beam
@@ -14,5 +14,4 @@
     <xacro:property name="part_info" scope="parent" value="${dict(
         attach='0 0 0',
-        axis='1 0 0',
         slots=dict(
         ),

File: bluerobotics_parts/urdf/surveyor_multibeam.urdf.xacro (robot description, xacro)
@@ -6,5 +6,5 @@
   Inertia: estimated from the delivered collision geometry at 1000 kg/m^3 (SDF auto inertia); replace with measured values.
   Contract (see parts.xacro): <part>_info exports the metadata (attach,
-  axis, slots, frames); <part> instantiates the link, its mounting joint
+  slots, frames, drive); <part> instantiates the link, its mounting joint
   and its slot / frame links.
 -->
@@ -13,5 +13,4 @@
     <xacro:property name="part_info" scope="parent" value="${dict(
         attach='0 0 0',
-        axis='1 0 0',
         slots=dict(
         ),

File: bluerobotics_parts/urdf/t200_prop_ccw.urdf.xacro (robot description, xacro)
@@ -5,6 +5,8 @@
   2026-08-21. This file is the part: maintain it by hand from here on.
   Inertia: estimated from the delivered collision geometry at 1000 kg/m^3 (SDF auto inertia); replace with measured values.
+  Drive: T200 16 V endpoints and prop diameter as placeholders for every
+  propeller option; replace with measured values for this prop.
   Contract (see parts.xacro): <part>_info exports the metadata (attach,
-  axis, slots, frames); <part> instantiates the link, its mounting joint
+  slots, frames, drive); <part> instantiates the link, its mounting joint
   and its slot / frame links.
 -->
@@ -13,9 +15,9 @@
     <xacro:property name="part_info" scope="parent" value="${dict(
         attach='0 0 0',
-        axis='1 0 0',
         slots=dict(
         ),
         frames=dict(
-        ))}"/>
+        ),
+        drive=dict(diameter=0.076, max_thrust=51.5, min_thrust=-40.2, rotation='ccw'))}"/>
   </xacro:macro>
   <xacro:macro name="t200_prop_ccw"

File: bluerobotics_parts/urdf/t200_prop_cw.urdf.xacro (robot description, xacro)
@@ -5,6 +5,8 @@
   2026-08-21. This file is the part: maintain it by hand from here on.
   Inertia: estimated from the delivered collision geometry at 1000 kg/m^3 (SDF auto inertia); replace with measured values.
+  Drive: T200 16 V endpoints and prop diameter as placeholders for every
+  propeller option; replace with measured values for this prop.
   Contract (see parts.xacro): <part>_info exports the metadata (attach,
-  axis, slots, frames); <part> instantiates the link, its mounting joint
+  slots, frames, drive); <part> instantiates the link, its mounting joint
   and its slot / frame links.
 -->
@@ -13,9 +15,9 @@
     <xacro:property name="part_info" scope="parent" value="${dict(
         attach='0 0 0',
-        axis='1 0 0',
         slots=dict(
         ),
         frames=dict(
-        ))}"/>
+        ),
+        drive=dict(diameter=0.076, max_thrust=51.5, min_thrust=-40.2, rotation='cw'))}"/>
   </xacro:macro>
   <xacro:macro name="t200_prop_cw"

File: bluerobotics_parts/urdf/t200_thruster.urdf.xacro (robot description, xacro)
@@ -6,5 +6,5 @@
   Inertia: tensor shape estimated from the collision geometry, scaled from 0.455 kg at 1000 kg/m^3 to the stated 0.344 kg.
   Contract (see parts.xacro): <part>_info exports the metadata (attach,
-  axis, slots, frames); <part> instantiates the link, its mounting joint
+  slots, frames, drive); <part> instantiates the link, its mounting joint
   and its slot / frame links.
 -->
@@ -13,5 +13,4 @@
     <xacro:property name="part_info" scope="parent" value="${dict(
         attach='0 0 0',
-        axis='1 0 0',
         slots=dict(
         ),

Commit message: Keep per part topic overrides under the instance namespace
Signed-off-by: Carlos Agüero <caguero@honurobotics.com>
Assisted-by: Claude Fable 5.1 <noreply@anthropic.com>

File: blueboat_gazebo/model.sdf.xacro (robot description, xacro)
@@ -33,6 +33,7 @@
   <!-- Topic namespace: every part topic is /<topic_namespace>/<part name>/...
        on both sides (a propeller's /thrust, the Ping's /range). Per part,
-       `gz_topic` / `topic` override the gz side base; the bridge config is
-       generated from the same yaml, so gz and ROS sides stay in sync. -->
+       `gz_topic` / `topic` override the gz side base, under the namespace
+       unless they start with a slash; the bridge config is generated from
+       the same yaml, so gz and ROS sides stay in sync. -->
   <xacro:property name="topic_ns" value="${cfg.get('topic_namespace', 'blueboat')}"/>
   <!-- The root link the assembly names (the config's base.name). -->
@@ -141,6 +142,7 @@
   <xacro:macro name="gz_part" params="ptype name parent xyz rpy collision joint axis info">
     <xacro:part_entry name="${name}"/>
+    <xacro:property name="topic_override" value="${entry.get('gz_topic', entry.get('topic', name))}"/>
     <xacro:property name="topic_base"
-                    value="${entry.get('gz_topic', entry.get('topic', topic_ns + '/' + name))}"/>
+                    value="${topic_override if topic_override.startswith('/') else topic_ns + '/' + topic_override}"/>
     <!-- A propeller on a fixed joint (a spare, say) is lumped away and
          drives nothing. -->

File: bluerov2_gazebo/model.sdf.xacro (robot description, xacro)
@@ -33,6 +33,7 @@
   <!-- Topic namespace: every part topic is /<topic_namespace>/<part name>/...
        on both sides (a camera's /image, a claw's /cmd_pos). Per part,
-       `gz_topic` / `topic` override the gz side base; the bridge config is
-       generated from the same yaml, so gz and ROS sides stay in sync. -->
+       `gz_topic` / `topic` override the gz side base, under the namespace
+       unless they start with a slash; the bridge config is generated from
+       the same yaml, so gz and ROS sides stay in sync. -->
   <xacro:property name="topic_ns" value="${cfg.get('topic_namespace', 'bluerov2')}"/>
   <!-- The root link the assembly names (the config's base.name). -->
@@ -224,6 +225,7 @@
   <xacro:macro name="gz_part" params="ptype name parent xyz rpy collision joint axis info">
     <xacro:part_entry name="${name}"/>
+    <xacro:property name="topic_override" value="${entry.get('gz_topic', entry.get('topic', name))}"/>
     <xacro:property name="topic_base"
-                    value="${entry.get('gz_topic', entry.get('topic', topic_ns + '/' + name))}"/>
+                    value="${topic_override if topic_override.startswith('/') else topic_ns + '/' + topic_override}"/>
     <!-- A propeller on a fixed joint (a spare, say) is lumped away and
          drives nothing. -->

Commit message: Keep per part topic overrides under the instance namespace
Signed-off-by: Carlos Agüero <caguero@honurobotics.com>
Assisted-by: Claude Fable 5.1 <noreply@anthropic.com>

File: blueboat_gazebo/model.sdf.xacro (robot description, xacro)
@@ -33,6 +33,7 @@
   <!-- Topic namespace: every part topic is /<topic_namespace>/<part name>/...
        on both sides (a propeller's /cmd, the Ping's /range). Per part,
-       `gz_topic` / `topic` override the gz side base; the bridge config is
-       generated from the same yaml, so gz and ROS sides stay in sync. -->
+       `gz_topic` / `topic` override the gz side base, under the namespace
+       unless they start with a slash; the bridge config is generated from
+       the same yaml, so gz and ROS sides stay in sync. -->
   <xacro:property name="topic_ns" value="${cfg.get('topic_namespace', 'blueboat')}"/>
   <!-- The root link the assembly names (the config's base.name). -->
@@ -149,6 +150,7 @@
   <xacro:macro name="gz_part" params="ptype name parent xyz rpy collision joint axis info">
     <xacro:part_entry name="${name}"/>
+    <xacro:property name="topic_override" value="${entry.get('gz_topic', entry.get('topic', name))}"/>
     <xacro:property name="topic_base"
-                    value="${entry.get('gz_topic', entry.get('topic', topic_ns + '/' + name))}"/>
+                    value="${topic_override if topic_override.startswith('/') else topic_ns + '/' + topic_override}"/>
     <!-- A propeller on a fixed joint (a spare, say) is lumped away and
          drives nothing. -->

File: bluerov2_gazebo/model.sdf.xacro (robot description, xacro)
@@ -33,6 +33,7 @@
   <!-- Topic namespace: every part topic is /<topic_namespace>/<part name>/...
        on both sides (a camera's /image, a claw's /cmd_pos). Per part,
-       `gz_topic` / `topic` override the gz side base; the bridge config is
-       generated from the same yaml, so gz and ROS sides stay in sync. -->
+       `gz_topic` / `topic` override the gz side base, under the namespace
+       unless they start with a slash; the bridge config is generated from
+       the same yaml, so gz and ROS sides stay in sync. -->
   <xacro:property name="topic_ns" value="${cfg.get('topic_namespace', 'bluerov2')}"/>
   <!-- The root link the assembly names (the config's base.name). -->
@@ -232,6 +233,7 @@
   <xacro:macro name="gz_part" params="ptype name parent xyz rpy collision joint axis info">
     <xacro:part_entry name="${name}"/>
+    <xacro:property name="topic_override" value="${entry.get('gz_topic', entry.get('topic', name))}"/>
     <xacro:property name="topic_base"
-                    value="${entry.get('gz_topic', entry.get('topic', topic_ns + '/' + name))}"/>
+                    value="${topic_override if topic_override.startswith('/') else topic_ns + '/' + topic_override}"/>
     <!-- A propeller on a fixed joint (a spare, say) is lumped away and
          drives nothing. -->
