Commit message: Name each vehicle instance once and spawn it at a full pose (#59)
Signed-off-by: Carlos Agüero <caguero@honurobotics.com>
Assisted-by: Claude Fable 5.1 <noreply@anthropic.com>

File: blueboat_gazebo/model.sdf.xacro (robot description, xacro)
@@ -33,6 +33,7 @@
   <!-- Topic namespace: every part topic is /<topic_namespace>/<part name>/...
        on both sides (a propeller's /cmd, the Ping's /range). Per part,
-       `gz_topic` / `topic` override the gz side base; the bridge config is
-       generated from the same yaml, so gz and ROS sides stay in sync. -->
+       `gz_topic` / `topic` override the gz side base, under the namespace
+       unless they start with a slash; the bridge config is generated from
+       the same yaml, so gz and ROS sides stay in sync. -->
   <xacro:property name="topic_ns" value="${cfg.get('topic_namespace', 'blueboat')}"/>
   <!-- The root link the assembly names (the config's base.name). -->
@@ -103,8 +104,15 @@
   </xacro:macro>
   <!-- One ArduPilotPlugin <control> block: a servo channel mapped onto a
-       thruster's command topic. -->
-  <xacro:macro name="ardupilot_control" params="channel joint topic">
+       motor's command topic, which is the topic that motor's Thruster
+       listens on: the part's gz_topic / topic override under the namespace,
+       or as given when it starts with a slash, exactly as gz_part resolves
+       it. -->
+  <xacro:macro name="ardupilot_control" params="channel motor">
+    <xacro:part_entry name="${motor}"/>
+    <xacro:property name="motor_override" value="${entry.get('gz_topic', entry.get('topic', motor))}"/>
+    <xacro:property name="motor_topic"
+                    value="${motor_override if motor_override.startswith('/') else '/' + topic_ns + '/' + motor_override}"/>
     <control channel="${channel}">
-      <jointName>${joint}</jointName>
+      <jointName>${motor}_joint</jointName>
       <servo_min>1100</servo_min>
       <servo_max>1900</servo_max>
@@ -112,5 +120,5 @@
       <multiplier>2</multiplier>
       <type>COMMAND</type>
-      <cmd_topic>${topic}</cmd_topic>
+      <cmd_topic>${motor_topic}/cmd</cmd_topic>
     </control>
   </xacro:macro>
@@ -123,6 +131,7 @@
              carries it (robot_state_publisher publishes the URDF links; the
              ${name}_sensor wrapper exists only here, and gz's derived id is
-             in neither). -->
-        <frame_id>${frame}</frame_id>
+             in neither), under the instance name, which is the prefix
+             robot_state_publisher puts on every frame of this instance. -->
+        <frame_id>${topic_ns}/${frame}</frame_id>
         <topic>${topic_base}/range</topic>
         <update_rate>10</update_rate>
@@ -149,6 +158,7 @@
   <xacro:macro name="gz_part" params="ptype name parent xyz rpy collision joint axis info">
     <xacro:part_entry name="${name}"/>
+    <xacro:property name="topic_override" value="${entry.get('gz_topic', entry.get('topic', name))}"/>
     <xacro:property name="topic_base"
-                    value="${entry.get('gz_topic', entry.get('topic', topic_ns + '/' + name))}"/>
+                    value="${topic_override if topic_override.startswith('/') else topic_ns + '/' + topic_override}"/>
     <!-- A propeller on a fixed joint (a spare, say) is lumped away and
          drives nothing. -->
@@ -209,5 +219,8 @@
     </joint>
   </xacro:macro>
-  <model name="blueboat">
+  <!-- Named after the instance (the config's topic_namespace, or the name option):
+       the model name, the topic namespace and, in the launch, the ROS
+       namespace are one name. A spawn may still rename it. -->
+  <model name="${topic_ns}">
     <include merge="true">
       <uri>$(arg urdf_uri)</uri>
@@ -287,8 +300,6 @@
           the newtons, including the asymmetry between ahead and astern.
         -->
-        <xacro:ardupilot_control channel="0" joint="motor_stbd_joint"
-                                 topic="/${topic_ns}/motor_stbd/cmd"/>
-        <xacro:ardupilot_control channel="2" joint="motor_port_joint"
-                                 topic="/${topic_ns}/motor_port/cmd"/>
+        <xacro:ardupilot_control channel="0" motor="motor_stbd"/>
+        <xacro:ardupilot_control channel="2" motor="motor_port"/>
       </plugin>
     </xacro:if>

File: bluerov2_gazebo/model.sdf.xacro (robot description, xacro)
@@ -33,6 +33,7 @@
   <!-- Topic namespace: every part topic is /<topic_namespace>/<part name>/...
        on both sides (a camera's /image, a claw's /cmd_pos). Per part,
-       `gz_topic` / `topic` override the gz side base; the bridge config is
-       generated from the same yaml, so gz and ROS sides stay in sync. -->
+       `gz_topic` / `topic` override the gz side base, under the namespace
+       unless they start with a slash; the bridge config is generated from
+       the same yaml, so gz and ROS sides stay in sync. -->
   <xacro:property name="topic_ns" value="${cfg.get('topic_namespace', 'bluerov2')}"/>
   <!-- The root link the assembly names (the config's base.name). -->
@@ -82,7 +83,8 @@
        down per <tilt>; tune each accessory's rpy for the intended view.
        FRAMES. Every sensor pins <frame_id> to a link the DESCRIPTION defines,
-       because that is the only name TF carries: robot_state_publisher publishes
-       the URDF's links, while the ${name}_sensor wrapper links below exist only
-       here. Left unset, gz derives the id from the SDF ('bluerov2/camera_sensor/
+       under the instance name (robot_state_publisher prefixes every frame of
+       an instance with it), because that is the only name TF carries:
+       robot_state_publisher publishes the URDF's links, while the
+       ${name}_sensor wrapper links below exist only here. Left unset, gz derives the id from the SDF ('bluerov2/camera_sensor/
        camera'), which is in neither the URDF nor TF, so a consumer doing
        lookup_transform(base_link, msg.header.frame_id) simply fails.
@@ -129,5 +131,5 @@
       <sensor name="${name}" type="camera">
         <!-- Body frame; see the FRAMES note above on the optical convention. -->
-        <frame_id>${name}</frame_id>
+        <frame_id>${topic_ns}/${name}</frame_id>
         <topic>${topic_base}/image</topic>
         <update_rate>20</update_rate>
@@ -151,5 +153,5 @@
     <xacro:sensor_link name="${name}" frame="${frame}">
       <sensor name="${name}" type="rgbd_camera">
-        <frame_id>${name}</frame_id>
+        <frame_id>${topic_ns}/${name}</frame_id>
         <topic>${topic_base}</topic>
         <update_rate>15</update_rate>
@@ -170,5 +172,5 @@
     <xacro:sensor_link name="${name}" frame="${frame}">
       <sensor name="${name}" type="gpu_lidar">
-        <frame_id>${name}</frame_id>
+        <frame_id>${topic_ns}/${name}</frame_id>
         <topic>${topic_base}/scan</topic>
         <update_rate>10</update_rate>
@@ -197,5 +199,5 @@
     <xacro:sensor_link name="${name}" frame="${frame}">
       <sensor name="${name}" type="custom" gz:type="dvl">
-        <frame_id>${name}</frame_id>
+        <frame_id>${topic_ns}/${name}</frame_id>
         <topic>${topic_base}/velocity</topic>
         <update_rate>8</update_rate>
@@ -232,6 +234,7 @@
   <xacro:macro name="gz_part" params="ptype name parent xyz rpy collision joint axis info">
     <xacro:part_entry name="${name}"/>
+    <xacro:property name="topic_override" value="${entry.get('gz_topic', entry.get('topic', name))}"/>
     <xacro:property name="topic_base"
-                    value="${entry.get('gz_topic', entry.get('topic', topic_ns + '/' + name))}"/>
+                    value="${topic_override if topic_override.startswith('/') else topic_ns + '/' + topic_override}"/>
     <!-- A propeller on a fixed joint (a spare, say) is lumped away and
          drives nothing. -->
@@ -266,5 +269,8 @@
     </plugin>
   </xacro:macro>
-  <model name="bluerov2">
+  <!-- Named after the instance (the config's topic_namespace, or the name option):
+       the model name, the topic namespace and, in the launch, the ROS
+       namespace are one name. A spawn may still rename it. -->
+  <model name="${topic_ns}">
     <include merge="true">
       <uri>$(arg urdf_uri)</uri>

Commit message: Mark one windage box per BlueBoat hull gz:wind="true"
Assisted-by: Claude Opus 5.5 <noreply@anthropic.com>
Signed-off-by: Carlos Agüero <caguero@honurobotics.com>

File: blueboat_gazebo/model.sdf.xacro (robot description, xacro)
@@ -187,5 +187,9 @@
        gz-maritime's gz_buoyancy) floats this link by them under whatever
        name the boat is spawned, with no <enable> list. Gazebo's stock
-       system ignores the attribute, so the worlds here are unchanged. -->
+       system ignores the attribute, so the worlds here are unchanged.
+       One windage box per hull, spanning the whole pontoon, carries
+       gz:wind="true" instead: a world with gz-maritime's wind system pushes
+       on the part of it above the waterline. Not the segments, which would
+       count a hull's frontal area once per segment in a head wind. -->
   <xacro:macro name="pontoon" params="hull side y n i:=0">
     <xacro:if value="${i != n}">
@@ -200,4 +204,13 @@
       <xacro:pontoon hull="${hull}" side="${side}" y="${y}" n="${n}" i="${i + 1}"/>
     </xacro:if>
+  </xacro:macro>
+  <xacro:macro name="windage" params="hull side y">
+    <collision name="windage_${side}" gz:wind="true">
+      <pose>${hull['x']} ${y} ${hull['z']} 0 0 0</pose>
+      <geometry>
+        <box><size>${hull['length']} ${hull['width']} ${hull['height']}</size></box>
+      </geometry>
+      <surface><contact><collide_bitmask>0x00</collide_bitmask></contact></surface>
+    </collision>
   </xacro:macro>
   <xacro:macro name="hull_displacement" params="hull">
@@ -213,4 +226,6 @@
       <xacro:pontoon hull="${hull}" side="port" y="${hull['y']}"  n="${hull['segments']}"/>
       <xacro:pontoon hull="${hull}" side="stbd" y="${-hull['y']}" n="${hull['segments']}"/>
+      <xacro:windage hull="${hull}" side="port" y="${hull['y']}"/>
+      <xacro:windage hull="${hull}" side="stbd" y="${-hull['y']}"/>
     </link>
     <joint name="hull_displacement_joint" type="fixed">

Commit message: Snapshot: surge drag identified, thrust and mass updated
Work in progress on phase 4, committed as a point to return to.

The surge damping is now linear-free with a quadratic term of -7.0, identified against the boat's response rather than carried over as a placeholder. The other axes keep their placeholder values and the comment no longer claims otherwise.

The M200 propeller parts carry measured endpoints - 40.22 N ahead, 20.1 N astern - and a 0.2 N deadband, which the model emits only when a part declares one. The chassis mass is 16.8 kg with a recomputed inertia tensor.

Also here: the parameters provenance page and the tuning walkthrough outline, both still outlines, and the reference spreadsheet and plot behind the drag identification.

Co-Authored-By: Claude Opus 5 (1M context) <noreply@anthropic.com>

File: blueboat_gazebo/model.sdf.xacro (robot description, xacro)
@@ -47,5 +47,5 @@
   </xacro:macro>
   <!-- A propeller part drives its mounting joint: one Thruster plugin per
-       propeller instance, with the limits and diameter the part declares in
+       propeller instance, with the thrust limits the part declares in
        its `drive` table. Counter rotating pairs (ccw to port, cw to
        starboard in the default configuration) get opposite coefficient signs so
@@ -74,4 +74,10 @@
       <max_thrust_cmd>${drive['max_thrust']}</max_thrust_cmd>
       <min_thrust_cmd>${drive['min_thrust']}</min_thrust_cmd>
+      <!-- Emitted only when the part declares one: the plugin enables the
+           deadband by the element's presence, so a zero would arm a cut that
+           never fires. -->
+      <xacro:if value="${'deadband' in drive and drive['deadband'] > 0}">
+        <deadband>${drive['deadband']}</deadband>
+      </xacro:if>
     </plugin>
   </xacro:macro>
@@ -229,20 +235,16 @@
       <xacro:hull_displacement hull="${cfg['hull_displacement']}"/>
     </xacro:if>
-    <!-- Hydrodynamic damping for the surface hull (Fossen). USV placeholder
-         coefficients: strong sway/yaw resistance, moderate surge, plus
-         heave/roll/pitch damping so the graded-buoyancy float settles instead of
-         bobbing. Tune against real BlueBoat response. -->
+    <!-- Hydrodynamic drag/damping coefficient (derivative terms)
+    -->
     <plugin filename="gz-sim-hydrodynamics-system"
             name="gz::sim::systems::Hydrodynamics">
       <link_name>${base_name}</link_name>
       <water_density>1025.0</water_density>
-      <xU>-20</xU>    <yV>-40</yV>    <zW>-30</zW>
-      <kP>-20</kP>    <mQ>-20</mQ>    <nR>-15</nR>
-      <xUabsU>-30</xUabsU>
-      <yVabsV>-90</yVabsV>
-      <zWabsW>-100</zWabsW>
-      <kPabsP>-40</kPabsP>
-      <mQabsQ>-40</mQabsQ>
-      <nRabsR>-30</nRabsR>
+      <xU>0</xU>    <xUabsU>-7.0</xUabsU>
+      <yV>-40</yV>    <yVabsV>-90</yVabsV>
+      <zW>-30</zW>    <zWabsW>-50</zWabsW>
+      <kP>-20</kP>    <kPabsP>-40</kPabsP>
+      <mQ>-20</mQ>    <mQabsQ>-40</mQabsQ>
+      <nR>-15</nR>    <nRabsR>-30</nRabsR>
     </plugin>
     <!-- Joint states for the propeller joints, so robot_state_publisher can

File: bluerobotics_parts/urdf/blueboat_chassis.urdf.xacro (robot description, xacro)
@@ -44,8 +44,8 @@
       <inertial>
         <origin xyz="0.0212659 0 0.0724998" rpy="0 0 0"/>
-        <mass value="12"/>
-        <inertia ixx="1.6043" ixy="-1.22202e-18" ixz="0.00372803"
-                 iyy="0.988314" iyz="4.88808e-18"
-                 izz="2.53089"/>
+        <mass value="16.8"/>
+        <inertia ixx="1.51" ixy="0" ixz="0"
+                 iyy="2.41" iyz="0"
+                 izz="3.23"/>
       </inertial>
       <xacro:part_visual mesh="package://bluerobotics_parts/models/blueboat_chassis/blueboat_chassis.visual.glb"/>

File: bluerobotics_parts/urdf/m200_weedless_prop_ccw.urdf.xacro (robot description, xacro)
@@ -1,13 +1,6 @@
 <?xml version="1.0"?>
 <!--
-  m200_weedless_prop_ccw part macro.
-  Bootstrapped from models/m200_weedless_prop_ccw/model.sdf by scripts/sdf_to_part.py on
-  2026-08-21. This file is the part: maintain it by hand from here on.
-  Inertia: estimated from the delivered collision geometry at 1000 kg/m^3 (SDF auto inertia); replace with measured values.
-  Drive: T200 16 V endpoints and prop diameter as placeholders for every
-  propeller option; replace with measured values for this prop.
-  Contract (see parts.xacro): <part>_info exports the metadata (attach,
-  slots, frames, drive); <part> instantiates the link, its mounting joint
-  and its slot / frame links.
+  m200_weedless_prop_ccw part macro for blueboat
+  Identical to m200_weedless_prop_cw.urdf.xacro - see documentation there.
 -->
 <robot xmlns:xacro="http://ros.org/wiki/xacro">
@@ -19,5 +12,10 @@
         frames=dict(
         ),
-        drive=dict(diameter=0.076, max_thrust=51.5, min_thrust=-40.2, rotation='ccw'))}"/>
+        drive=dict(
+          diameter=0.1,
+          max_thrust=40.22,
+          min_thrust=-20.1,
+          deadband=0.2,
+          rotation='ccw'))}"/>
   </xacro:macro>
   <xacro:macro name="m200_weedless_prop_ccw"

File: bluerobotics_parts/urdf/m200_weedless_prop_cw.urdf.xacro (robot description, xacro)
@@ -1,13 +1,8 @@
 <?xml version="1.0"?>
 <!--
-  m200_weedless_prop_cw part macro.
-  Bootstrapped from models/m200_weedless_prop_cw/model.sdf by scripts/sdf_to_part.py on
-  2026-08-21. This file is the part: maintain it by hand from here on.
-  Inertia: estimated from the delivered collision geometry at 1000 kg/m^3 (SDF auto inertia); replace with measured values.
-  Drive: T200 16 V endpoints and prop diameter as placeholders for every
-  propeller option; replace with measured values for this prop.
-  Contract (see parts.xacro): <part>_info exports the metadata (attach,
-  slots, frames, drive); <part> instantiates the link, its mounting joint
-  and its slot / frame links.
+  m200_weedless_prop_cw part macro for blueboat
+  Identical to m200_weedless_prop_ccw.urdf.xacro
+  Values derived according to src/bluerobotics_models/docs/vehicles/blueboat/parameters.md
+  For the `drive` dictionary, `max_thrust` and `min_thrust` are in Newtons, and `rotation` indicates the propeller rotation direction.  `diameter`, is a bit confusing because it controls both the visual representation (how fast the prop spins for a given command) and, in certain modes, how the command is interpreted.   Not really ideal, but it works for now.  We declare a physical diameter value here, but it does not dictate the size of the visual or how it affects physics, just with how fast the propeller rotation is animated.
 -->
 <robot xmlns:xacro="http://ros.org/wiki/xacro">
@@ -19,5 +14,10 @@
         frames=dict(
         ),
-        drive=dict(diameter=0.076, max_thrust=51.5, min_thrust=-40.2, rotation='cw'))}"/>
+        drive=dict(
+          diameter=0.1,
+          max_thrust=40.22,
+          min_thrust=-20.1,
+          deadband=0.2,
+          rotation='cw'))}"/>
   </xacro:macro>
   <xacro:macro name="m200_weedless_prop_cw"
@@ -27,5 +27,5 @@
       <inertial>
         <origin xyz="0.000336 3e-05 -5e-06" rpy="0 0 0"/>
-        <mass value="0.074472"/>
+        <mass value="0.01"/>
         <inertia ixx="1.41779e-05" ixy="0" ixz="-5.54437e-12"
                  iyy="3.11438e-05" iyz="0"

File: bluerobotics_parts/urdf/parts.xacro (robot description, xacro)
@@ -27,7 +27,12 @@
          drive    propellers only: what a simulator needs to drive the part
                   as a thruster on its mounting joint
-                    diameter    propeller diameter, m
+                    diameter    propeller diameter, m. Sets the spin
+                                rate the plugin commands, not the
+                                force on the hull
                     max_thrust  forward thrust limit, N
                     min_thrust  reverse thrust limit, N (negative)
+                    deadband    optional; thrust below which the thruster
+                                produces nothing, N. Omitted or 0 means
+                                none
                     rotation    'ccw' or 'cw', seen from behind looking
                                 forward along the spin axis

Commit message: BlueBoat windage marks (#70)
Assisted-by: Claude Opus 5.5 <noreply@anthropic.com>
Signed-off-by: Carlos Agüero <caguero@honurobotics.com>

File: blueboat_gazebo/model.sdf.xacro (robot description, xacro)
@@ -193,5 +193,8 @@
        gz-maritime's gz_buoyancy) floats this link by them under whatever
        name the boat is spawned, with no <enable> list. Gazebo's stock
-       system ignores the attribute, so the worlds here are unchanged. -->
+       system ignores the attribute, so the worlds here are unchanged.
+       Nothing but these boxes may live on this link: the stock system
+       floats every collision of the link it is enabled on. The wind sees
+       the hulls through a link of their own, windage, below. -->
   <xacro:macro name="pontoon" params="hull side y n i:=0">
     <xacro:if value="${i != n}">
@@ -206,4 +209,43 @@
       <xacro:pontoon hull="${hull}" side="${side}" y="${y}" n="${n}" i="${i + 1}"/>
     </xacro:if>
+  </xacro:macro>
+  <!-- ===================== Windage =====================
+       One box per hull, spanning the whole pontoon, marked gz:wind="true":
+       a world with gz-maritime's wind system pushes on the part of it above
+       the waterline, under whatever name the boat was spawned. One box, not
+       the buoyancy segments, which would count a hull's frontal area once
+       per segment in a head wind.
+       On a link of its own, fixed to the root link like hull_displacement,
+       and never on hull_displacement itself: the stock buoyancy system
+       floats every collision of the link it is enabled on, and a box with
+       the hull's full volume there would double the displacement. The boxes
+       collide with nothing (collide_bitmask 0x00) and carry no gz:buoyancy
+       mark, so they displace nothing in either buoyancy system. -->
+  <xacro:macro name="windage_box" params="hull side y">
+    <collision name="windage_${side}" gz:wind="true">
+      <pose>${hull['x']} ${y} ${hull['z']} 0 0 0</pose>
+      <geometry>
+        <box><size>${hull['length']} ${hull['width']} ${hull['height']}</size></box>
+      </geometry>
+      <surface><contact><collide_bitmask>0x00</collide_bitmask></contact></surface>
+    </collision>
+  </xacro:macro>
+  <xacro:macro name="windage" params="hull">
+    <link name="windage">
+      <pose relative_to="${base_name}">0 0 0 0 0 0</pose>
+      <inertial>
+        <mass>1e-5</mass>
+        <inertia>
+          <ixx>1e-8</ixx><ixy>0</ixy><ixz>0</ixz>
+          <iyy>1e-8</iyy><iyz>0</iyz><izz>1e-8</izz>
+        </inertia>
+      </inertial>
+      <xacro:windage_box hull="${hull}" side="port" y="${hull['y']}"/>
+      <xacro:windage_box hull="${hull}" side="stbd" y="${-hull['y']}"/>
+    </link>
+    <joint name="windage_joint" type="fixed">
+      <parent>${base_name}</parent>
+      <child>windage</child>
+    </joint>
   </xacro:macro>
   <xacro:macro name="hull_displacement" params="hull">
@@ -234,4 +276,5 @@
     <xacro:if value="${'hull_displacement' in cfg}">
       <xacro:hull_displacement hull="${cfg['hull_displacement']}"/>
+      <xacro:windage hull="${cfg['hull_displacement']}"/>
     </xacro:if>
     <!-- Hydrodynamic drag/damping coefficient (derivative terms)
