Commit message: Drive the BlueBoat with ArduRover in SITL
Phase 1 of the SITL roadmap: the boat driven by the same autopilot it runs
on the water, using the thruster interface exactly as it exists today. No
plugin work; this proves the plumbing and the channel mapping.

The ArduPilot variant is generated from model.sdf.xacro behind a flag that
defaults to false, so the model generated today is byte-identical and the
ROS 2 path is untouched. The roadmap proposed a hand-written wrapper
merge-including model://blueboat instead, which cannot work: merge-include
does not nest and the composed model already merge-includes its URDF, so
the frame name collides. SITL_DESIGN.md is amended rather than quietly
rewritten, so intent and implementation can be reviewed together.

The IMU is a frame on the chassis, not a part and not a Gazebo-only link.
Parts already declare frames for where they sense, so one line gives a
base_link_imu link in the URDF and therefore in TF, with the composition
hanging the sensor on it as it already does for the Ping's echosounder.

Parameters derive from Blue Robotics' hardware dump, not from ArduPilot's
rover-skid defaults and not from the community SITL_Models config, both of
which assign the throttles the other way round. Four deltas are marked in
the file: both trims to 1500, and SERVO3_REVERSED to 0, which compensates
for wiring that does not exist in simulation and would otherwise drive the
port thruster backwards.

The world loads gz-sim-imu-system. Without it the IMU sensor produces
nothing, ArduPilotPlugin has no attitude to report and never replies, and
SITL stalls resending servos. The existing worlds never needed it because
the boat had no IMU until now.

Verified headless: zero duplicate frames, MAVProxy detects the vehicle and
downloads 1275 parameters. The drive test itself needs an interactive
ground station and has not been run.

File: blueboat_gazebo/model.sdf.xacro (robot description, xacro)
@@ -24,4 +24,11 @@
        configs) a file:// URI of one generated from the same config. -->
   <xacro:arg name="urdf_uri" default="model://blueboat/blueboat.urdf"/>
+  <!-- ArduPilot SITL. False generates the model this repository has always
+       generated; true adds an IMU and the ArduPilotPlugin, so ArduRover can
+       drive the boat instead of ROS 2 topics. Two models come out of this one
+       source: model://blueboat and model://blueboat_with_ardupilot. See
+       docs how-to/verify-sitl. -->
+  <xacro:arg name="ardupilot" default="false"/>
+  <xacro:property name="ardupilot" value="${'$(arg ardupilot)'.lower() == 'true'}"/>
   <!-- Topic namespace: every part topic is /<topic_namespace>/<part name>/...
        on both sides (a propeller's /thrust, the Ping's /range). Per part,
@@ -86,4 +93,17 @@
       <child>${name}_sensor</child>
     </joint>
+  </xacro:macro>
+  <!-- One ArduPilotPlugin <control> block: a servo channel mapped onto a
+       thruster's command topic. -->
+  <xacro:macro name="ardupilot_control" params="channel joint topic">
+    <control channel="${channel}">
+      <jointName>${joint}</jointName>
+      <servo_min>1100</servo_min>
+      <servo_max>1900</servo_max>
+      <offset>-0.5</offset>
+      <multiplier>80.4</multiplier>
+      <type>COMMAND</type>
+      <cmd_topic>${topic}</cmd_topic>
+    </control>
   </xacro:macro>
   <!-- Ping2 single-beam echosounder: a 1-ray gpu_lidar pointing straight down
@@ -208,4 +228,53 @@
                     slots="${cfg.get('slots') or []}" emit="gz_part" emit_slot="gz_no_slot"
                     manifest="false"/>
+    <!-- ===================== ArduPilot SITL =====================
+         Only when ardupilot:=true. Everything above is unchanged, so the
+         default model and the ROS 2 path are untouched. -->
+    <xacro:if value="${ardupilot}">
+      <!-- Attitude source for ArduPilotPlugin, at the chassis's imu frame.
+           The frame is declared by the part, so it exists in the URDF and
+           therefore in TF; this hangs the Gazebo sensor on it, exactly as the
+           echosounder does for the Ping's beam frame. -->
+      <xacro:sensor_link name="imu" frame="${base_name}_imu">
+        <sensor name="imu_sensor" type="imu">
+          <always_on>1</always_on>
+          <update_rate>1000</update_rate>
+        </sensor>
+      </xacro:sensor_link>
+      <plugin name="ArduPilotPlugin" filename="ArduPilotPlugin">
+        <fdm_addr>127.0.0.1</fdm_addr>
+        <fdm_port_in>9002</fdm_port_in>
+        <connectionTimeoutMaxCount>5</connectionTimeoutMaxCount>
+        <lock_step>1</lock_step>
+        <!-- base_link is x forward, y left, z up (docs reference/frames), and
+             ArduPilot wants x forward, y right, z down: roll 180. The world
+             transform is the usual Gazebo-ENU to NED. Both are the standard
+             values because this model follows the ordinary convention - the
+             bow is at +X and the propeller joints are on axis 1 0 0. -->
+        <modelXYZToAirplaneXForwardZDown degrees="true">0 0 0 180 0 0</modelXYZToAirplaneXForwardZDown>
+        <gazeboXYZToNED degrees="true">0 0 0 180 0 90</gazeboXYZToNED>
+        <imuName>imu_sensor::imu_sensor</imuName>
+        <!--
+          Channels follow the shipped boat, not ArduPilot's rover-skid
+          defaults and not the BlueBoat in SITL_Models, both of which have
+          them the other way round. From BlueBoat120.params:
+              SERVO1_FUNCTION 74   ThrottleRight  ->  starboard
+              SERVO3_FUNCTION 73   ThrottleLeft   ->  port
+              SERVO1_MIN/MAX  1100 / 1900
+          channel= is zero-based, so channel 0 is SERVO1 and channel 2 is
+          SERVO3. These must agree with params/blueboat_sitl.params; nothing
+          checks that they do, and if they drift the boat steers backwards.
+          cmd = multiplier * (clamp((pwm - min)/(max - min)) + offset), so
+          offset -0.5 puts stop at mid-stick and multiplier is newtons at full
+          deflection. It is symmetric and a T200 is not (+51.5 N against
+          -40.2 N): the smaller magnitude is used for both, which under-drives
+          ahead but keeps the mapping linear. Phase 3's problem.
+        -->
+        <xacro:ardupilot_control channel="0" joint="motor_stbd_joint"
+                                 topic="/${topic_ns}/motor_stbd/thrust"/>
+        <xacro:ardupilot_control channel="2" joint="motor_port_joint"
+                                 topic="/${topic_ns}/motor_port/thrust"/>
+      </plugin>
+    </xacro:if>
   </model>
 </sdf>

File: bluerobotics_parts/urdf/blueboat_chassis.urdf.xacro (robot description, xacro)
@@ -17,4 +17,10 @@
 -->
 <robot xmlns:xacro="http://ros.org/wiki/xacro">
+  <!-- The imu frame is where the Navigator flight controller senses attitude.
+       Declared as a frame rather than a part because nothing about its mass or
+       appearance matters, but simulation and TF have to agree on where it is.
+       The position is a placeholder at the chassis origin: the real offset
+       inside the enclosure has not been measured, and the lever arm only starts
+       to matter once accelerations are compared against the real boat. -->
   <xacro:macro name="blueboat_chassis_info">
     <xacro:property name="part_info" scope="parent" value="${dict(
@@ -29,4 +35,5 @@
         ),
         frames=dict(
+            imu=dict(xyz='0 0 0', rpy='0 0 0'),
         ))}"/>
   </xacro:macro>

Commit message: Include bouyancy marks
Signed-off-by: Alejandro Hernandez Cordero <ahcorde@gmail.com>

File: blueboat_gazebo/model.sdf.xacro (robot description, xacro)
@@ -162,9 +162,14 @@
        hubs). Segmented so each box responds to its own local depth and a
        pitched waterplane restores properly. The boxes also give contact.
-       Fixed jointed to the root link: physics sees one rigid body. -->
+       Fixed jointed to the root link: physics sees one rigid body.
+       Each box is also marked gz:buoyancy="true": a world whose buoyancy
+       system reads marked collisions (gz-sim 229ec07e, carried by
+       gz-maritime's gz_buoyancy) floats this link by them under whatever
+       name the boat is spawned, with no <enable> list. Gazebo's stock
+       system ignores the attribute, so the worlds here are unchanged. -->
   <xacro:macro name="pontoon" params="hull side y n i:=0">
     <xacro:if value="${i != n}">
       <xacro:property name="seg_len" value="${hull['length'] / n}"/>
-      <collision name="pontoon_${side}_${i}">
+      <collision name="pontoon_${side}_${i}" gz:buoyancy="true">
         <pose>${hull['x'] - hull['length']/2.0 + seg_len*(i + 0.5)} ${y} ${hull['z']} 0 0 0</pose>
         <geometry>

File: bluerov2_gazebo/model.sdf.xacro (robot description, xacro)
@@ -268,5 +268,10 @@
        with the box centroid on the declared CoB (cob_offset from the CoM
        or from the root link). total_mass / com come from the assembled
-       URDF via generate_model.py. Fixed jointed: physics sees one body. -->
+       URDF via generate_model.py. Fixed jointed: physics sees one body.
+       The box is also marked gz:buoyancy="true": a world whose buoyancy
+       system reads marked collisions (gz-sim 229ec07e, carried by
+       gz-maritime's gz_buoyancy) floats this link by it under whatever
+       name the ROV is spawned, with no <enable> list. Gazebo's stock
+       system ignores the attribute, so the worlds here are unchanged. -->
     <xacro:property name="buoyancy_cfg" value="${cfg.get('buoyancy') or dict()}"/>
     <xacro:if value="${'$(arg total_mass)' == '' or '$(arg com)' == ''}">
@@ -298,5 +303,5 @@
         </inertia>
       </inertial>
-      <collision name="displacement">
+      <collision name="displacement" gz:buoyancy="true">
         <pose>${cob_target[0]} ${cob_target[1]} ${cob_target[2]} 0 0 0</pose>
         <geometry>

Commit message: Suggestions to #59
Signed-off-by: Alejandro Hernandez Cordero <ahcorde@gmail.com>

File: blueboat_gazebo/model.sdf.xacro (robot description, xacro)
@@ -96,8 +96,15 @@
   </xacro:macro>
   <!-- One ArduPilotPlugin <control> block: a servo channel mapped onto a
-       thruster's command topic. -->
-  <xacro:macro name="ardupilot_control" params="channel joint topic">
+       motor's command topic, which is the topic that motor's Thruster
+       listens on: the part's gz_topic / topic override under the namespace,
+       or as given when it starts with a slash, exactly as gz_part resolves
+       it. -->
+  <xacro:macro name="ardupilot_control" params="channel motor">
+    <xacro:part_entry name="${motor}"/>
+    <xacro:property name="motor_override" value="${entry.get('gz_topic', entry.get('topic', motor))}"/>
+    <xacro:property name="motor_topic"
+                    value="${motor_override if motor_override.startswith('/') else '/' + topic_ns + '/' + motor_override}"/>
     <control channel="${channel}">
-      <jointName>${joint}</jointName>
+      <jointName>${motor}_joint</jointName>
       <servo_min>1100</servo_min>
       <servo_max>1900</servo_max>
@@ -105,5 +112,5 @@
       <multiplier>80.4</multiplier>
       <type>COMMAND</type>
-      <cmd_topic>${topic}</cmd_topic>
+      <cmd_topic>${motor_topic}/thrust</cmd_topic>
     </control>
   </xacro:macro>
@@ -276,8 +283,6 @@
           ahead but keeps the mapping linear. Phase 3's problem.
         -->
-        <xacro:ardupilot_control channel="0" joint="motor_stbd_joint"
-                                 topic="/${topic_ns}/motor_stbd/thrust"/>
-        <xacro:ardupilot_control channel="2" joint="motor_port_joint"
-                                 topic="/${topic_ns}/motor_port/thrust"/>
+        <xacro:ardupilot_control channel="0" motor="motor_stbd"/>
+        <xacro:ardupilot_control channel="2" motor="motor_port"/>
       </plugin>
     </xacro:if>

Commit message: Validate the instance name and follow motor overrides in the ArduPilot block
Signed-off-by: Carlos Agüero <caguero@honurobotics.com>

File: blueboat_gazebo/model.sdf.xacro (robot description, xacro)
@@ -104,8 +104,15 @@
   </xacro:macro>
   <!-- One ArduPilotPlugin <control> block: a servo channel mapped onto a
-       thruster's command topic. -->
-  <xacro:macro name="ardupilot_control" params="channel joint topic">
+       motor's command topic, which is the topic that motor's Thruster
+       listens on: the part's gz_topic / topic override under the namespace,
+       or as given when it starts with a slash, exactly as gz_part resolves
+       it. -->
+  <xacro:macro name="ardupilot_control" params="channel motor">
+    <xacro:part_entry name="${motor}"/>
+    <xacro:property name="motor_override" value="${entry.get('gz_topic', entry.get('topic', motor))}"/>
+    <xacro:property name="motor_topic"
+                    value="${motor_override if motor_override.startswith('/') else '/' + topic_ns + '/' + motor_override}"/>
     <control channel="${channel}">
-      <jointName>${joint}</jointName>
+      <jointName>${motor}_joint</jointName>
       <servo_min>1100</servo_min>
       <servo_max>1900</servo_max>
@@ -113,5 +120,5 @@
       <multiplier>2</multiplier>
       <type>COMMAND</type>
-      <cmd_topic>${topic}</cmd_topic>
+      <cmd_topic>${motor_topic}/cmd</cmd_topic>
     </control>
   </xacro:macro>
@@ -285,8 +292,6 @@
           the newtons, including the asymmetry between ahead and astern.
         -->
-        <xacro:ardupilot_control channel="0" joint="motor_stbd_joint"
-                                 topic="/${topic_ns}/motor_stbd/cmd"/>
-        <xacro:ardupilot_control channel="2" joint="motor_port_joint"
-                                 topic="/${topic_ns}/motor_port/cmd"/>
+        <xacro:ardupilot_control channel="0" motor="motor_stbd"/>
+        <xacro:ardupilot_control channel="2" motor="motor_port"/>
       </plugin>
     </xacro:if>

Commit message: Mark the displacement collisions as buoyancy geometry (#57)
Signed-off-by: Alejandro Hernandez Cordero <ahcorde@gmail.com>

File: blueboat_gazebo/model.sdf.xacro (robot description, xacro)
@@ -169,14 +169,22 @@
        collision geometry (the modeler's hull cylinders, hatch boxes, prop
        hubs). Segmented so each box responds to its own local depth and a
-       pitched waterplane restores properly. The boxes also give contact.
-       Fixed jointed to the root link: physics sees one rigid body. -->
+       pitched waterplane restores properly. The boxes never collide
+       (collide_bitmask 0x00): they displace only, and contact stays with
+       the chassis collisions, which the boxes overlap.
+       Fixed jointed to the root link: physics sees one rigid body.
+       Each box is also marked gz:buoyancy="true": a world whose buoyancy
+       system reads marked collisions (gz-sim 229ec07e, carried by
+       gz-maritime's gz_buoyancy) floats this link by them under whatever
+       name the boat is spawned, with no <enable> list. Gazebo's stock
+       system ignores the attribute, so the worlds here are unchanged. -->
   <xacro:macro name="pontoon" params="hull side y n i:=0">
     <xacro:if value="${i != n}">
       <xacro:property name="seg_len" value="${hull['length'] / n}"/>
-      <collision name="pontoon_${side}_${i}">
+      <collision name="pontoon_${side}_${i}" gz:buoyancy="true">
         <pose>${hull['x'] - hull['length']/2.0 + seg_len*(i + 0.5)} ${y} ${hull['z']} 0 0 0</pose>
         <geometry>
           <box><size>${seg_len} ${hull['width']} ${hull['height']}</size></box>
         </geometry>
+        <surface><contact><collide_bitmask>0x00</collide_bitmask></contact></surface>
       </collision>
       <xacro:pontoon hull="${hull}" side="${side}" y="${y}" n="${n}" i="${i + 1}"/>

File: bluerov2_gazebo/model.sdf.xacro (robot description, xacro)
@@ -278,5 +278,12 @@
        with the box centroid on the declared CoB (cob_offset from the CoM
        or from the root link). total_mass / com come from the assembled
-       URDF via generate_model.py. Fixed jointed: physics sees one body. -->
+       URDF via generate_model.py. Fixed jointed: physics sees one body.
+       The box is also marked gz:buoyancy="true": a world whose buoyancy
+       system reads marked collisions (gz-sim 229ec07e, carried by
+       gz-maritime's gz_buoyancy) floats this link by it under whatever
+       name the ROV is spawned, with no <enable> list. Gazebo's stock
+       system ignores the attribute, so the worlds here are unchanged. The
+       box never collides (collide_bitmask 0x00): it displaces only, and
+       contact stays with the parts' collisions, which it overlaps. -->
     <xacro:property name="buoyancy_cfg" value="${cfg.get('buoyancy') or dict()}"/>
     <xacro:if value="${'$(arg total_mass)' == '' or '$(arg com)' == ''}">
@@ -308,9 +315,10 @@
         </inertia>
       </inertial>
-      <collision name="displacement">
+      <collision name="displacement" gz:buoyancy="true">
         <pose>${cob_target[0]} ${cob_target[1]} ${cob_target[2]} 0 0 0</pose>
         <geometry>
           <box><size>${footprint[0]} ${footprint[1]} ${box_height}</size></box>
         </geometry>
+        <surface><contact><collide_bitmask>0x00</collide_bitmask></contact></surface>
       </collision>
     </link>

Commit message: Suggestions #70
Signed-off-by: Alejandro Hernandez Cordero <ahcorde@gmail.com>

File: blueboat_gazebo/model.sdf.xacro (robot description, xacro)
@@ -188,8 +188,7 @@
        name the boat is spawned, with no <enable> list. Gazebo's stock
        system ignores the attribute, so the worlds here are unchanged.
-       One windage box per hull, spanning the whole pontoon, carries
-       gz:wind="true" instead: a world with gz-maritime's wind system pushes
-       on the part of it above the waterline. Not the segments, which would
-       count a hull's frontal area once per segment in a head wind. -->
+       Nothing but these boxes may live on this link: the stock system
+       floats every collision of the link it is enabled on. The wind sees
+       the hulls through a link of their own, windage, below. -->
   <xacro:macro name="pontoon" params="hull side y n i:=0">
     <xacro:if value="${i != n}">
@@ -205,5 +204,17 @@
     </xacro:if>
   </xacro:macro>
-  <xacro:macro name="windage" params="hull side y">
+  <!-- ===================== Windage =====================
+       One box per hull, spanning the whole pontoon, marked gz:wind="true":
+       a world with gz-maritime's wind system pushes on the part of it above
+       the waterline, under whatever name the boat was spawned. One box, not
+       the buoyancy segments, which would count a hull's frontal area once
+       per segment in a head wind.
+       On a link of its own, fixed to the root link like hull_displacement,
+       and never on hull_displacement itself: the stock buoyancy system
+       floats every collision of the link it is enabled on, and a box with
+       the hull's full volume there would double the displacement. The boxes
+       collide with nothing (collide_bitmask 0x00) and carry no gz:buoyancy
+       mark, so they displace nothing in either buoyancy system. -->
+  <xacro:macro name="windage_box" params="hull side y">
     <collision name="windage_${side}" gz:wind="true">
       <pose>${hull['x']} ${y} ${hull['z']} 0 0 0</pose>
@@ -213,4 +224,22 @@
       <surface><contact><collide_bitmask>0x00</collide_bitmask></contact></surface>
     </collision>
+  </xacro:macro>
+  <xacro:macro name="windage" params="hull">
+    <link name="windage">
+      <pose relative_to="${base_name}">0 0 0 0 0 0</pose>
+      <inertial>
+        <mass>1e-5</mass>
+        <inertia>
+          <ixx>1e-8</ixx><ixy>0</ixy><ixz>0</ixz>
+          <iyy>1e-8</iyy><iyz>0</iyz><izz>1e-8</izz>
+        </inertia>
+      </inertial>
+      <xacro:windage_box hull="${hull}" side="port" y="${hull['y']}"/>
+      <xacro:windage_box hull="${hull}" side="stbd" y="${-hull['y']}"/>
+    </link>
+    <joint name="windage_joint" type="fixed">
+      <parent>${base_name}</parent>
+      <child>windage</child>
+    </joint>
   </xacro:macro>
   <xacro:macro name="hull_displacement" params="hull">
@@ -243,4 +272,5 @@
     <xacro:if value="${'hull_displacement' in cfg}">
       <xacro:hull_displacement hull="${cfg['hull_displacement']}"/>
+      <xacro:windage hull="${cfg['hull_displacement']}"/>
     </xacro:if>
     <!-- Hydrodynamic damping for the surface hull (Fossen). USV placeholder
