Commit message: Suggestions #70 (#74)
* Suggestions #70

Signed-off-by: Alejandro Hernandez Cordero <ahcorde@gmail.com>

File: blueboat_gazebo/model.sdf.xacro (robot description, xacro)
@@ -188,8 +188,7 @@
        name the boat is spawned, with no <enable> list. Gazebo's stock
        system ignores the attribute, so the worlds here are unchanged.
-       One windage box per hull, spanning the whole pontoon, carries
-       gz:wind="true" instead: a world with gz-maritime's wind system pushes
-       on the part of it above the waterline. Not the segments, which would
-       count a hull's frontal area once per segment in a head wind. -->
+       Nothing but these boxes may live on this link: the stock system
+       floats every collision of the link it is enabled on. The wind sees
+       the hulls through a link of their own, windage, below. -->
   <xacro:macro name="pontoon" params="hull side y n i:=0">
     <xacro:if value="${i != n}">
@@ -205,5 +204,17 @@
     </xacro:if>
   </xacro:macro>
-  <xacro:macro name="windage" params="hull side y">
+  <!-- ===================== Windage =====================
+       One box per hull, spanning the whole pontoon, marked gz:wind="true":
+       a world with gz-maritime's wind system pushes on the part of it above
+       the waterline, under whatever name the boat was spawned. One box, not
+       the buoyancy segments, which would count a hull's frontal area once
+       per segment in a head wind.
+       On a link of its own, fixed to the root link like hull_displacement,
+       and never on hull_displacement itself: the stock buoyancy system
+       floats every collision of the link it is enabled on, and a box with
+       the hull's full volume there would double the displacement. The boxes
+       collide with nothing (collide_bitmask 0x00) and carry no gz:buoyancy
+       mark, so they displace nothing in either buoyancy system. -->
+  <xacro:macro name="windage_box" params="hull side y">
     <collision name="windage_${side}" gz:wind="true">
       <pose>${hull['x']} ${y} ${hull['z']} 0 0 0</pose>
@@ -213,4 +224,22 @@
       <surface><contact><collide_bitmask>0x00</collide_bitmask></contact></surface>
     </collision>
+  </xacro:macro>
+  <xacro:macro name="windage" params="hull">
+    <link name="windage">
+      <pose relative_to="${base_name}">0 0 0 0 0 0</pose>
+      <inertial>
+        <mass>1e-5</mass>
+        <inertia>
+          <ixx>1e-8</ixx><ixy>0</ixy><ixz>0</ixz>
+          <iyy>1e-8</iyy><iyz>0</iyz><izz>1e-8</izz>
+        </inertia>
+      </inertial>
+      <xacro:windage_box hull="${hull}" side="port" y="${hull['y']}"/>
+      <xacro:windage_box hull="${hull}" side="stbd" y="${-hull['y']}"/>
+    </link>
+    <joint name="windage_joint" type="fixed">
+      <parent>${base_name}</parent>
+      <child>windage</child>
+    </joint>
   </xacro:macro>
   <xacro:macro name="hull_displacement" params="hull">
@@ -226,6 +255,4 @@
       <xacro:pontoon hull="${hull}" side="port" y="${hull['y']}"  n="${hull['segments']}"/>
       <xacro:pontoon hull="${hull}" side="stbd" y="${-hull['y']}" n="${hull['segments']}"/>
-      <xacro:windage hull="${hull}" side="port" y="${hull['y']}"/>
-      <xacro:windage hull="${hull}" side="stbd" y="${-hull['y']}"/>
     </link>
     <joint name="hull_displacement_joint" type="fixed">
@@ -243,4 +270,5 @@
     <xacro:if value="${'hull_displacement' in cfg}">
       <xacro:hull_displacement hull="${cfg['hull_displacement']}"/>
+      <xacro:windage hull="${cfg['hull_displacement']}"/>
     </xacro:if>
     <!-- Hydrodynamic damping for the surface hull (Fossen). USV placeholder

Commit message: BlueBoat and BlueROV2 drift with the ocean current
Signed-off-by: Alejandro Hernandez Cordero <ahcorde@gmail.com>

File: blueboat_gazebo/model.sdf.xacro (robot description, xacro)
@@ -210,10 +210,20 @@
     </xacro:if>
   </xacro:macro>
-  <!-- ===================== Windage =====================
+  <!-- ===================== Windage and water drag =====================
        One box per hull, spanning the whole pontoon, marked gz:wind="true":
        a world with gz-maritime's wind system pushes on the part of it above
        the waterline, under whatever name the boat was spawned. One box, not
        the buoyancy segments, which would count a hull's frontal area once
-       per segment in a head wind.
+       per segment in a head wind (or a head current).
+       The same box is marked gz:ocean_current="true": gz-maritime's ocean
+       current system drags the part below the waterline against the water,
+       along every axis, so the boat drifts with the world's current. That
+       is the boat's surge, sway and heave damping, which the Hydrodynamics
+       plugin below therefore leaves out. Its drag coefficient is set so the
+       marks reproduce the identified surge coefficient (xUabsU = -7.0, PR
+       #72): the 12.3 kg boat floats at a draft of 3.2 cm, the two hull ends
+       show the water 2 * 0.18 * 0.032 = 0.0114 m^2, and
+       7.0 / (0.5 * 1025 * 0.0114) is about 1.19. Sway and heave follow from
+       the same coefficient on the hulls' side and bottom areas.
        On a link of its own, fixed to the root link like hull_displacement,
        and never on hull_displacement itself: the stock buoyancy system
@@ -222,6 +232,8 @@
        collide with nothing (collide_bitmask 0x00) and carry no gz:buoyancy
        mark, so they displace nothing in either buoyancy system. -->
+  <xacro:property name="ocean_current_cd" value="1.19"/>
   <xacro:macro name="windage_box" params="hull side y">
-    <collision name="windage_${side}" gz:wind="true">
+    <collision name="windage_${side}" gz:wind="true"
+               gz:ocean_current="true" gz:ocean_current_cd="${ocean_current_cd}">
       <pose>${hull['x']} ${y} ${hull['z']} 0 0 0</pose>
       <geometry>
@@ -278,7 +290,13 @@
       <xacro:windage hull="${cfg['hull_displacement']}"/>
     </xacro:if>
-    <!-- Hydrodynamic drag/damping coefficient (derivative terms)
-          Surge and yaw coefficients are identified in PR #72.
-          The remainder are still placeholders - see Issue #73.
+    <!-- Hydrodynamic drag/damping coefficients (derivative terms), for the
+         motions the hull boxes' gz:ocean_current marks do not cover: roll,
+         pitch and yaw. Surge, sway and heave come from the marks, against the
+         water, with the identified surge (xUabsU = -7.0, PR #72) carried by
+         their drag coefficient (see Windage and water drag). Fossen surge,
+         sway or heave here as well would damp the boat against the ground
+         too, hold it back in a current, and damp heave twice. The yaw
+         coefficient is identified in PR #72; roll and pitch are still
+         placeholders - see Issue #73.
     -->
     <plugin filename="gz-sim-hydrodynamics-system"
@@ -286,7 +304,4 @@
       <link_name>${base_name}</link_name>
       <water_density>1025.0</water_density>
-      <xU>0</xU>    <xUabsU>-7.0</xUabsU>
-      <yV>-40</yV>    <yVabsV>-90</yVabsV>
-      <zW>-30</zW>    <zWabsW>-50</zWabsW>
       <kP>-20</kP>    <kPabsP>-40</kPabsP>
       <mQ>-20</mQ>    <mQabsQ>-40</mQabsQ>

File: bluerov2_gazebo/model.sdf.xacro (robot description, xacro)
@@ -394,5 +394,50 @@
               name="gz::sim::systems::DopplerVelocityLogSystem"/>
     </xacro:if>
-    <!-- Hydrodynamic damping (Fossen quadratic drag, reference BlueROV2).
+    <!-- ===================== Water drag =====================
+         The ROV's translational drag, surge, sway and heave, against the
+         water: one box marked gz:ocean_current="true", which gz-maritime's
+         ocean current system drags along every axis, relative to the water,
+         so the ROV drifts with the world's current. Its sides are sized so
+         that, with a drag coefficient of one, the box reproduces the
+         reference BlueROV2 quadratic coefficients exactly: a face of area A
+         across a flow gives 0.5 * rho * A * u^2, so the faces normal to x, y
+         and z are X / q, Y / q and Z / q, q = 0.5 * rho, and the box is
+         sqrt(Y Z / (X q)) by sqrt(X Z / (Y q)) by sqrt(X Y / (Z q)), about
+         0.48 by 0.30 by 0.22 m, close to the ROV's own envelope. Centred on
+         the centre of mass, so translation puts no moment on it.
+         On a link of its own, never on buoyancy_displacement: the stock
+         buoyancy system floats every collision of the link it is enabled
+         on. The box collides with nothing and carries no gz:buoyancy mark,
+         so it displaces nothing in either buoyancy system. -->
+    <xacro:property name="drag_x" value="33.732"/>
+    <xacro:property name="drag_y" value="54.16"/>
+    <xacro:property name="drag_z" value="73.225"/>
+    <xacro:property name="drag_q" value="${0.5 * water_density}"/>
+    <link name="water_drag">
+      <pose relative_to="${base_name}">0 0 0 0 0 0</pose>
+      <inertial>
+        <mass>1e-5</mass>
+        <inertia>
+          <ixx>1e-8</ixx><ixy>0</ixy><ixz>0</ixz>
+          <iyy>1e-8</iyy><iyz>0</iyz><izz>1e-8</izz>
+        </inertia>
+      </inertial>
+      <collision name="water_drag" gz:ocean_current="true">
+        <pose>${com[0]} ${com[1]} ${com[2]} 0 0 0</pose>
+        <geometry>
+          <box><size>${sqrt(drag_y * drag_z / (drag_x * drag_q))} ${sqrt(drag_x * drag_z / (drag_y * drag_q))} ${sqrt(drag_x * drag_y / (drag_z * drag_q))}</size></box>
+        </geometry>
+        <surface><contact><collide_bitmask>0x00</collide_bitmask></contact></surface>
+      </collision>
+    </link>
+    <joint name="water_drag_joint" type="fixed">
+      <parent>${base_name}</parent>
+      <child>water_drag</child>
+    </joint>
+    <!-- Hydrodynamic damping (Fossen quadratic drag, reference BlueROV2), for
+         the motions the water drag box does not cover: roll, pitch and yaw.
+         Surge, sway and heave come from the box, against the water; Fossen
+         terms on those axes as well would damp the ROV against the ground
+         too, hold it back in a current, and damp heave twice.
          Added mass (xDotU etc., e.g. von Benzon 2022) is intentionally left at
          zero: the plugin applies it as explicit acceleration feedback, which
@@ -404,9 +449,5 @@
       <link_name>${base_name}</link_name>
       <water_density>1025.0</water_density>
-      <xU>0</xU>   <yV>0</yV>   <zW>0</zW>
       <kP>0</kP>   <mQ>0</mQ>   <nR>0</nR>
-      <xUabsU>-33.732</xUabsU>
-      <yVabsV>-54.16</yVabsV>
-      <zWabsW>-73.225</zWabsW>
       <kPabsP>-3.992</kPabsP>
       <mQabsQ>-3.992</mQabsQ>

File: bluerov2_gazebo/worlds/bluerov2_pool.sdf.xacro (robot description, xacro)
@@ -222,4 +222,16 @@
       </graded_buoyancy>
       <enable>bluerov2::buoyancy_displacement</enable>
+    </plugin>
+    <!-- gz-maritime's ocean current (gz_ocean_current): slack water here,
+         <speed> in m/s and the <direction> it sets towards, in degrees
+         clockwise from north. It also drags the vehicle's collisions marked
+         gz:ocean_current="true" against the water, which is the vehicle's
+         surge, sway and heave damping, so it runs even with no current. The
+         density matches the buoyancy's water. -->
+    <plugin filename="gz-maritime-ocean-current-system"
+            name="gz::sim::maritime::OceanCurrent">
+      <speed>0</speed>
+      <direction>0</direction>
+      <water_density>1025</water_density>
     </plugin>
     <light type="directional" name="sun">
