Commit message: Apply review fixes: ament hook, RViz durability, xacro deps, sensor mass, docs
Assisted-by: Claude Fable 5 <noreply@anthropic.com>
Signed-off-by: Carlos Aguero <caguero@honurobotics.com>

File: bluerov2_gazebo/model.sdf.xacro (robot description, xacro)
@@ -47,15 +47,17 @@
        a camera looks +X, a gpu_lidar scans the sensor XY plane, DVL beams point
        down per <tilt>; tune each accessory's rpy for the intended view. -->
-  <!-- Wrapper: a massless sensor link fixed to base_link at `pose`, holding the
-       <sensor> block passed in. Mass is negligible (the accessory's real mass/
-       geometry already live in base_link via the description). -->
+  <!-- Wrapper: a near-massless sensor link fixed to base_link at `pose`, holding
+       the <sensor> block passed in. The accessory's real mass/geometry already
+       live in base_link via the description; 1e-5 kg keeps each wrapper under
+       0.5% of the 0.02% buoyancy margin, so a full sensor loadout cannot tip
+       the trim negative. -->
   <xacro:macro name="sensor_link" params="name pose *sensor">
     <link name="${name}_sensor">
       <pose relative_to="base_link">${pose}</pose>
       <inertial>
-        <mass>0.001</mass>
+        <mass>1e-5</mass>
         <inertia>
-          <ixx>1e-6</ixx><ixy>0</ixy><ixz>0</ixz>
-          <iyy>1e-6</iyy><iyz>0</iyz><izz>1e-6</izz>
+          <ixx>1e-8</ixx><ixy>0</ixy><ixz>0</ixz>
+          <iyy>1e-8</iyy><iyz>0</iyz><izz>1e-8</izz>
         </inertia>
       </inertial>
@@ -208,5 +210,10 @@
       <uri>package://bluerov2_description/urdf/bluerov2.urdf</uri>
     </include>
-    <!-- Hydrodynamic damping (Fossen quadratic drag, reference BlueROV2). -->
+    <!-- Hydrodynamic damping (Fossen quadratic drag, reference BlueROV2).
+         Added mass (xDotU etc., e.g. von Benzon 2022) is intentionally left at
+         zero: the plugin applies it as explicit acceleration feedback, which
+         diverges when added mass exceeds rigid mass (heave: 18.68 vs 11.5 kg).
+         The stable path is SDF <fluid_added_mass>, pending build time URDF
+         conversion so base_link's inertial can carry it. -->
     <plugin filename="gz-sim-hydrodynamics-system"
             name="gz::sim::systems::Hydrodynamics">

Commit message: Generate a BlueROV2 model ArduSub can drive
The same model.sdf.xacro behind an `ardupilot` flag, as the BlueBoat does:
false generates what this repository always generated, true adds an IMU and
the ArduPilotPlugin. A second model rather than a wrapper, because
<include merge="true"> does not nest and the composed model already
merge-includes its URDF.

The <control> blocks are emitted rather than written. A second pass of the
assembly dispatcher inside the plugin element gives one per propeller, with
the command topic coming from the same `topic_base` the Thruster uses, so
the two cannot drift apart. Six or eight then follows from the chassis
rather than from an edit here.

The channel is the thruster's number minus one, and that is a claim about
geometry rather than a choice: ArduSub assigns SERVO1..6 to Motor1..6 from
FRAME_CONFIG, so what has to be true is that thruster_N sits where the
Vectored frame expects Motor N.

Unlike the boat, the ROV's model goes through generate_model.py, because
the buoyancy solve needs mass properties xacro cannot read from the URDF;
the flag is passed through rather than around it.

Co-Authored-By: Claude Opus 5 <noreply@anthropic.com>

File: bluerov2_gazebo/model.sdf.xacro (robot description, xacro)
@@ -31,4 +31,11 @@
   <xacro:arg name="total_mass" default=""/>
   <xacro:arg name="com" default=""/>
+  <!-- ArduPilot SITL. False generates the model this repository has always
+       generated; true adds an IMU and the ArduPilotPlugin, so ArduSub can
+       drive the ROV instead of ROS 2 topics. Two models come out of this one
+       source: model://bluerov2 and model://bluerov2_with_ardupilot. See
+       docs how-to/verify-sitl-rov. -->
+  <xacro:arg name="ardupilot" default="false"/>
+  <xacro:property name="ardupilot" value="${'$(arg ardupilot)'.lower() == 'true'}"/>
   <!-- Topic namespace: every part topic is /<topic_namespace>/<part name>/...
        on both sides (a camera's /image, a claw's /cmd_pos). Per part,
@@ -224,4 +231,45 @@
     </xacro:sensor_link>
   </xacro:macro>
+  <!-- One ArduPilotPlugin <control> block: a servo channel mapped onto a
+       thruster's command topic.
+       cmd = multiplier * (clamp((pwm - min)/(max - min)) + offset), so
+       offset -0.5 puts stop at mid-stick and multiplier 2 spans [-1, 1].
+       That is the whole of it: no thrust limits, no vehicle physics, just
+       the servo band converted to a normalized command. The thruster owns
+       the newtons, including the asymmetry between ahead and astern.
+       ArduSub parks disarmed motors at 1500 rather than at MIN, which this
+       mapping turns into a zero command. -->
+  <xacro:macro name="ardupilot_control" params="channel joint topic">
+    <control channel="${channel}">
+      <jointName>${joint}</jointName>
+      <servo_min>1100</servo_min>
+      <servo_max>1900</servo_max>
+      <offset>-0.5</offset>
+      <multiplier>2</multiplier>
+      <type>COMMAND</type>
+      <cmd_topic>${topic}</cmd_topic>
+    </control>
+  </xacro:macro>
+  <!-- A second pass of the assembly dispatcher, inside the plugin element:
+       one <control> per propeller instance, emitted by the same iteration
+       that emits the Thrusters so the command topic cannot drift between
+       them - both come from `topic_base`.
+       The channel is the thruster's own number minus one, and that is a
+       claim about geometry rather than a choice. ArduSub assigns
+       SERVO1..6 to Motor1..6 automatically from FRAME_CONFIG, and our
+       thruster_N slots sit where ArduSub's Vectored frame expects Motor N
+       (AP_Motors6DOF.cpp, SUB_FRAME_VECTORED). test_ardusub_frame.py
+       asserts that correspondence; if a slot moves, it fails there rather
+       than as a vehicle that swims sideways. -->
+  <xacro:macro name="ap_control" params="ptype name parent xyz rpy collision joint axis info">
+    <xacro:if value="${'drive' in info and joint != 'fixed'}">
+      <xacro:part_entry name="${name}"/>
+      <xacro:property name="topic_base"
+                      value="${entry.get('gz_topic', entry.get('topic', topic_ns + '/' + name))}"/>
+      <xacro:ardupilot_control channel="${int(name.split('_')[-1]) - 1}"
+                               joint="${name}_joint"
+                               topic="/${topic_base}/cmd"/>
+    </xacro:if>
+  </xacro:macro>
   <!-- Emitters for the assembly dispatcher. Per resolved part instance: a
        propeller (a part with a `drive` table) gets a Thruster on its joint,
@@ -357,4 +405,45 @@
                     slots="${cfg.get('slots') or []}" emit="gz_part" emit_slot="gz_no_slot"
                     manifest="false"/>
+    <!-- ===================== ArduPilot SITL =====================
+         Only when ardupilot:=true. Everything above is unchanged, so the
+         default model and the ROS 2 path are untouched. -->
+    <xacro:if value="${ardupilot}">
+      <!-- Attitude source for ArduPilotPlugin, at the chassis's imu frame.
+           The frame is declared by the part, so it exists in the URDF and
+           therefore in TF; this hangs the Gazebo sensor on it, exactly as the
+           sonar does for the Ping360's beam frame. -->
+      <xacro:sensor_link name="imu" frame="${base_name}_imu">
+        <sensor name="imu_sensor" type="imu">
+          <always_on>1</always_on>
+          <update_rate>1000</update_rate>
+        </sensor>
+      </xacro:sensor_link>
+      <plugin name="ArduPilotPlugin" filename="ArduPilotPlugin">
+        <fdm_addr>127.0.0.1</fdm_addr>
+        <fdm_port_in>9002</fdm_port_in>
+        <connectionTimeoutMaxCount>5</connectionTimeoutMaxCount>
+        <lock_step>1</lock_step>
+        <!-- base_link is x forward, y left, z up (docs reference/frames), and
+             ArduPilot wants x forward, y right, z down: roll 180. The world
+             transform is the usual Gazebo-ENU to NED. Both are the standard
+             values because this model follows the ordinary convention - the
+             bow is at +X and the propeller joints are on axis 1 0 0. -->
+        <modelXYZToAirplaneXForwardZDown degrees="true">0 0 0 180 0 0</modelXYZToAirplaneXForwardZDown>
+        <gazeboXYZToNED degrees="true">0 0 0 180 0 90</gazeboXYZToNED>
+        <imuName>imu_sensor::imu_sensor</imuName>
+        <!--
+          Depth needs no sensor here. The JSON protocol carries no pressure
+          field at all (SIM_JSON.h, the sensor keytable), and ArduSub does
+          not want one: AP_Baro_SITL uses BARO_TYPE_WATER and synthesizes
+          pressure from the altitude this plugin already reports.
+          The <control> blocks are emitted below rather than written out,
+          one per propeller the assembly resolved, so a different loadout
+          gets correct blocks with no edit here.
+        -->
+        <xacro:assemble base="${cfg['base']}" parts="${cfg.get('parts') or []}"
+                        slots="${cfg.get('slots') or []}" emit="ap_control"
+                        emit_slot="gz_no_slot" manifest="false"/>
+      </plugin>
+    </xacro:if>
   </model>
 </sdf>

Commit message: Generate a BlueROV2 model ArduSub can drive
The same model.sdf.xacro behind an `ardupilot` flag, as the BlueBoat does:
false generates what this repository always generated, true adds an IMU and
the ArduPilotPlugin. A second model rather than a wrapper, because
<include merge="true"> does not nest and the composed model already
merge-includes its URDF.

The <control> blocks are emitted rather than written. A second pass of the
assembly dispatcher inside the plugin element gives one per propeller, with
the command topic coming from the same `topic_base` the Thruster uses, so
the two cannot drift apart. Six or eight then follows from the chassis
rather than from an edit here.

The channel is the thruster's number minus one, and that is a claim about
geometry rather than a choice: ArduSub assigns SERVO1..6 to Motor1..6 from
FRAME_CONFIG, so what has to be true is that thruster_N sits where the
Vectored frame expects Motor N.

Unlike the boat, the ROV's model goes through generate_model.py, because
the buoyancy solve needs mass properties xacro cannot read from the URDF;
the flag is passed through rather than around it.

Co-Authored-By: Claude Opus 5 <noreply@anthropic.com>

File: bluerov2_gazebo/model.sdf.xacro (robot description, xacro)
@@ -31,4 +31,11 @@
   <xacro:arg name="total_mass" default=""/>
   <xacro:arg name="com" default=""/>
+  <!-- ArduPilot SITL. False generates the model this repository has always
+       generated; true adds an IMU and the ArduPilotPlugin, so ArduSub can
+       drive the ROV instead of ROS 2 topics. Two models come out of this one
+       source: model://bluerov2 and model://bluerov2_with_ardupilot. See
+       docs how-to/verify-sitl-rov. -->
+  <xacro:arg name="ardupilot" default="false"/>
+  <xacro:property name="ardupilot" value="${'$(arg ardupilot)'.lower() == 'true'}"/>
   <!-- Topic namespace: every part topic is /<topic_namespace>/<part name>/...
        on both sides (a camera's /image, a claw's /cmd_pos). Per part,
@@ -226,4 +233,45 @@
     </xacro:sensor_link>
   </xacro:macro>
+  <!-- One ArduPilotPlugin <control> block: a servo channel mapped onto a
+       thruster's command topic.
+       cmd = multiplier * (clamp((pwm - min)/(max - min)) + offset), so
+       offset -0.5 puts stop at mid-stick and multiplier 2 spans [-1, 1].
+       That is the whole of it: no thrust limits, no vehicle physics, just
+       the servo band converted to a normalized command. The thruster owns
+       the newtons, including the asymmetry between ahead and astern.
+       ArduSub parks disarmed motors at 1500 rather than at MIN, which this
+       mapping turns into a zero command. -->
+  <xacro:macro name="ardupilot_control" params="channel joint topic">
+    <control channel="${channel}">
+      <jointName>${joint}</jointName>
+      <servo_min>1100</servo_min>
+      <servo_max>1900</servo_max>
+      <offset>-0.5</offset>
+      <multiplier>2</multiplier>
+      <type>COMMAND</type>
+      <cmd_topic>${topic}</cmd_topic>
+    </control>
+  </xacro:macro>
+  <!-- A second pass of the assembly dispatcher, inside the plugin element:
+       one <control> per propeller instance, emitted by the same iteration
+       that emits the Thrusters so the command topic cannot drift between
+       them - both come from `topic_base`.
+       The channel is the thruster's own number minus one, and that is a
+       claim about geometry rather than a choice. ArduSub assigns
+       SERVO1..6 to Motor1..6 automatically from FRAME_CONFIG, and our
+       thruster_N slots sit where ArduSub's Vectored frame expects Motor N
+       (AP_Motors6DOF.cpp, SUB_FRAME_VECTORED). test_ardusub_frame.py
+       asserts that correspondence; if a slot moves, it fails there rather
+       than as a vehicle that swims sideways. -->
+  <xacro:macro name="ap_control" params="ptype name parent xyz rpy collision joint axis info">
+    <xacro:if value="${'drive' in info and joint != 'fixed'}">
+      <xacro:part_entry name="${name}"/>
+      <xacro:property name="topic_base"
+                      value="${entry.get('gz_topic', entry.get('topic', topic_ns + '/' + name))}"/>
+      <xacro:ardupilot_control channel="${int(name.split('_')[-1]) - 1}"
+                               joint="${name}_joint"
+                               topic="/${topic_base}/cmd"/>
+    </xacro:if>
+  </xacro:macro>
   <!-- Emitters for the assembly dispatcher. Per resolved part instance: a
        propeller (a part with a `drive` table) gets a Thruster on its joint,
@@ -371,4 +419,45 @@
                     slots="${cfg.get('slots') or []}" emit="gz_part" emit_slot="gz_no_slot"
                     manifest="false"/>
+    <!-- ===================== ArduPilot SITL =====================
+         Only when ardupilot:=true. Everything above is unchanged, so the
+         default model and the ROS 2 path are untouched. -->
+    <xacro:if value="${ardupilot}">
+      <!-- Attitude source for ArduPilotPlugin, at the chassis's imu frame.
+           The frame is declared by the part, so it exists in the URDF and
+           therefore in TF; this hangs the Gazebo sensor on it, exactly as the
+           sonar does for the Ping360's beam frame. -->
+      <xacro:sensor_link name="imu" frame="${base_name}_imu">
+        <sensor name="imu_sensor" type="imu">
+          <always_on>1</always_on>
+          <update_rate>1000</update_rate>
+        </sensor>
+      </xacro:sensor_link>
+      <plugin name="ArduPilotPlugin" filename="ArduPilotPlugin">
+        <fdm_addr>127.0.0.1</fdm_addr>
+        <fdm_port_in>9002</fdm_port_in>
+        <connectionTimeoutMaxCount>5</connectionTimeoutMaxCount>
+        <lock_step>1</lock_step>
+        <!-- base_link is x forward, y left, z up (docs reference/frames), and
+             ArduPilot wants x forward, y right, z down: roll 180. The world
+             transform is the usual Gazebo-ENU to NED. Both are the standard
+             values because this model follows the ordinary convention - the
+             bow is at +X and the propeller joints are on axis 1 0 0. -->
+        <modelXYZToAirplaneXForwardZDown degrees="true">0 0 0 180 0 0</modelXYZToAirplaneXForwardZDown>
+        <gazeboXYZToNED degrees="true">0 0 0 180 0 90</gazeboXYZToNED>
+        <imuName>imu_sensor::imu_sensor</imuName>
+        <!--
+          Depth needs no sensor here. The JSON protocol carries no pressure
+          field at all (SIM_JSON.h, the sensor keytable), and ArduSub does
+          not want one: AP_Baro_SITL uses BARO_TYPE_WATER and synthesizes
+          pressure from the altitude this plugin already reports.
+          The <control> blocks are emitted below rather than written out,
+          one per propeller the assembly resolved, so a different loadout
+          gets correct blocks with no edit here.
+        -->
+        <xacro:assemble base="${cfg['base']}" parts="${cfg.get('parts') or []}"
+                        slots="${cfg.get('slots') or []}" emit="ap_control"
+                        emit_slot="gz_no_slot" manifest="false"/>
+      </plugin>
+    </xacro:if>
   </model>
 </sdf>

Commit message: Snapshot: ROV thrust from published data, and an axis test
Intermediate commit. The T200 parts now carry Blue Robotics' bench thrust
at the 14.8 V pack and the ESC dead zone, and the BlueROV2 model scales
them by an installation factor taken from the published bollard pull for
the assembled vehicle. The derivation, and the correction of the earlier
60-65% estimate, are in the parameters page; the comments point there
rather than repeating the figures.

The heave and surge launch tests are replaced by one test that commands
0.5 on each of surge, sway, heave and yaw in both directions, and checks
the motion lies within 20 degrees of the commanded axis and within a
factor of ten of an expected speed. The expected speeds come from the
vehicle's published performance and engineering judgement, not from the
model, whose hydrodynamic coefficients are still being identified. The
allocation is the teleop mixer's, so the test says nothing about
ArduSub's Vectored frame. A table of each case against its limits is
printed at the end of the run.

Hydrodynamic identification and the closed-loop checks are still open.

Co-Authored-By: Claude Opus 5.5 <noreply@anthropic.com>

File: bluerov2_gazebo/model.sdf.xacro (robot description, xacro)
@@ -60,5 +60,12 @@
        the plugin prefixes a custom <topic> with its <namespace> (the model
        name unless given), so the namespace is emptied and the topic follows
-       the config like every other part topic, not the spawn name. -->
+       the config like every other part topic, not the spawn name.
+       The ROV spec declares bollard pull force values.  These values not consistent
+       with the bench thrust values of the individual thrusters.
+       So we introduce a derived factor to correct for this as a
+       multiplier on the bench thrust. The Heavy
+       has no published bollard figures and takes the same factor as an
+       assumption. Derivation: docs/vehicles/bluerov2/parameters.md. -->
+  <xacro:property name="thrust_install_factor" value="0.74"/>
   <xacro:macro name="prop_thruster" params="name drive topic_base">
     <plugin filename="gz-maritime-thruster-system"
@@ -78,6 +85,12 @@
       <propeller_diameter>${drive['diameter']}</propeller_diameter>
       <velocity_control>true</velocity_control>
-      <max_thrust_cmd>${drive['max_thrust']}</max_thrust_cmd>
-      <min_thrust_cmd>${drive['min_thrust']}</min_thrust_cmd>
+      <max_thrust_cmd>${drive['max_thrust'] * thrust_install_factor}</max_thrust_cmd>
+      <min_thrust_cmd>${drive['min_thrust'] * thrust_install_factor}</min_thrust_cmd>
+      <!-- Emitted only when the part declares one: the plugin enables the
+           deadband by the element's presence, so a zero would arm a cut that
+           never fires. -->
+      <xacro:if value="${'deadband' in drive and drive['deadband'] > 0}">
+        <deadband>${drive['deadband'] * thrust_install_factor}</deadband>
+      </xacro:if>
     </plugin>
   </xacro:macro>
